File: pcbs/Register with Reset/resetlogic.kicad_sch (KiCad schematic)
At the start: 12 parts, among them U401 74HC08, U402 74HC14

Commit message: Addressing clock blocking issue
Connections:
- net GND: no longer U401.4, U401.5
- net ~{RESET}: now also U401.4
- net CLK_{Out}: now reaches U401.6
- new net CLK_{in}: U401.5
Other:
- moved on the sheet: U401B
Changed lines of the file:
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@@
+		(color 0 0 0 0)
+	)
+	(junction
+		(at 53.34 76.2)
+		(diameter 0)
 		(color 0 0 0 0)
 	)
@@
 	(wire
 		(pts
+			(xy 53.34 76.2) (xy 55.88 76.2)
+		)
+		(stroke
+			(width 0)
+			(type default)
+		)
+	)
+	(wire
+		(pts
 			(xy 144.78 55.88) (xy 152.4 55.88)
 		)
@@
 	(wire
 		(pts
+			(xy 53.34 90.17) (xy 57.15 90.17)
+		)
+		(stroke
+			(width 0)
+			(type default)
+		)
+	)
+	(wire
+		(pts
 			(xy 21.59 144.78) (xy 24.13 144.78)
 		)
@@
 	(wire
 		(pts
+			(xy 50.8 95.25) (xy 57.15 95.25)
+		)
+		(stroke
+			(width 0)
+			(type default)
+		)
+	)
+	(wire
+		(pts
 			(xy 195.58 67.31) (xy 195.58 69.85)
 		)
@@
 	(wire
 		(pts
+			(xy 72.39 92.71) (xy 80.01 92.71)
+		)
+		(stroke
+			(width 0)
+			(type default)
+		)
+	)
+	(wire
+		(pts
 			(xy 267.97 148.59) (xy 267.97 152.4)
 		)
@@
 	(wire
 		(pts
+			(xy 53.34 76.2) (xy 53.34 90.17)
+		)
+		(stroke
+			(width 0)
+			(type default)
+		)
+	)
+	(wire
+		(pts
 			(xy 21.59 165.1) (xy 21.59 160.02)
 		)
@@
 	(wire
 		(pts
-			(xy 50.8 76.2) (xy 55.88 76.2)
+			(xy 50.8 76.2) (xy 53.34 76.2)
 		)
 		(stroke
@@
 		(shape output)
 		(at 254 55.88 0)
+		(fields_autoplaced yes)
+		(effects
+			(font
+				(size 1.27 1.27)
+			)
+			(justify left)
+		)
+	)
+	(hierarchical_label "CLK_{in}"
+		(shape input)
+		(at 50.8 95.25 180)
+		(fields_autoplaced yes)
+		(effects
+			(font
+				(size 1.27 1.27)
+			)
+			(justify right)
+		)
+	)
+	(hierarchical_label "CLK_{Out}"
+		(shape output)
+		(at 80.01 92.71 0)
 		(fields_autoplaced yes)
 		(effects
@@
 	(symbol
 		(lib_id "74xx:74LS08")
-		(at 31.75 147.32 0)
+		(at 64.77 92.71 0)
 		(unit 2)
 		(exclude_from_sim no)
@@
 		(fields_autoplaced yes)
 		(property "Reference" "U401"
-			(at 31.7417 138.43 0)
+			(at 64.7617 83.82 0)
 			(effects
 				(font
@@
 		)
 		(property "Value" "74HC08"
-			(at 31.7417 140.97 0)
+			(at 64.7617 86.36 0)
 			(effects
 				(font
@@
 		)
 		(property "Footprint" "Package_SO:SOIC-14_3.9x8.7mm_P1.27mm"
-			(at 31.75 147.32 0)
+			(at 64.77 92.71 0)
 			(effects
 				(font
@@
 		)
 		(property "Datasheet" "https://wmsc.lcsc.com/wmsc/upload/file/pdf/v2/lcsc/2304140030_Nexperia-74HC08D-653_C5593.pdf"
-			(at 31.75 147.32 0)
+			(at 64.77 92.71 0)
 			(effects
 				(font
@@
 		)
 		(property "Description" "Quad And2"
-			(at 31.75 147.32 0)
+			(at 64.77 92.71 0)
 			(effects
 				(font
@@
 		)
 		(property "LCSC" "C5593"
-			(at 31.75 147.32 0)
-			(effects
-				(font
+			(at 64.77 92.71 0)
+			(effects
+				(font

Commit message: Starting to redo layout
Connections:
- no-connect marks 5 -> 4
Changed lines of the file:
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@@
-	)
-	(junction
-		(at 21.59 160.02)
-		(diameter 0)
-		(color 0 0 0 0)
 	)
 	(junction
@@
 	(junction
 		(at 21.59 179.07)
-		(diameter 0)
-		(color 0 0 0 0)
-	)
-	(junction
-		(at 21.59 149.86)
 		(diameter 0)
 		(color 0 0 0 0)
@@
 	)
 	(no_connect
-		(at 39.37 147.32)
-	)
-	(no_connect
 		(at 39.37 176.53)
 	)
@@
 	(wire
 		(pts
-			(xy 21.59 160.02) (xy 21.59 149.86)
-		)
-		(stroke
-			(width 0)
-			(type default)
-		)
-	)
-	(wire
-		(pts
 			(xy 25.4 67.31) (xy 25.4 72.39)
 		)
@@
 	(wire
 		(pts
-			(xy 21.59 149.86) (xy 24.13 149.86)
-		)
-		(stroke
-			(width 0)
-			(type default)
-		)
-	)
-	(wire
-		(pts
 			(xy 67.31 76.2) (xy 72.39 76.2)
 		)
@@
 	(wire
 		(pts
-			(xy 21.59 144.78) (xy 24.13 144.78)
-		)
-		(stroke
-			(width 0)
-			(type default)
-		)
-	)
-	(wire
-		(pts
 			(xy 144.78 67.31) (xy 144.78 69.85)
 		)
@@
 		)
 		(stroke
-			(width 0)
-			(type default)
-		)
-	)
-	(wire
-		(pts
-			(xy 21.59 149.86) (xy 21.59 144.78)
-		)
-		(stroke
