File: pcbs/Register with Reset/Register with Reset.kicad_pcb (KiCad board)
At the start: 2 copper layers, 101.6 x 114.3 mm, 76 parts, among them J101 Conn_02x20_Odd_Even, U201 74HC245, U202 74HCT574, U203 74HC245, U301 74HC245, U302 74HCT574, U303 74HC245, U401 74HC08, U402 74HC14

Commit message: Addressing clock blocking issue
Parts:
- removed H101, H102, H103, H104: MountingHole, MountingHole:MountingHole_2.7mm_M2.5
Connections:
- D102 pad 2: /CLK -> /ResetLogic/CLK_{Out}
- U401 pad 4: GND -> /~{RESET}
- U401 pad 5: GND -> /CLK
- U401 pad 6: unconnected-(U401-Pad6) -> /ResetLogic/CLK_{Out}

Commit message: Starting to redo layout
Parts:
- J101: value Conn_02x20_Odd_Even -> ~; footprint Connector_IDC:IDC-Header_2x20_P2.54mm_Vertical -> BoardEdgeConnectors:TE-5530843-4-Edge
- moved D101 28.6 mm to (116.2, 99.1)
- moved D102 28.6 mm to (116.2, 101.6)
- moved R101 27.9 mm to (120.7, 99.1)
- moved J101 10.2 mm to (58.4, 101.6), turned to -90 degrees
- moved R302 7.62 mm to (123.2, 124.5)
- moved R303 7.62 mm to (123.2, 127.0)
- moved R304 7.62 mm to (123.2, 129.5)
- moved R306 7.62 mm to (123.2, 134.6)
- moved R307 7.62 mm to (123.2, 137.2)
- moved R308 7.62 mm to (123.2, 139.7)
- moved U301 7.62 mm to (109.2, 129.5)
- moved U302 7.62 mm to (127.0, 119.4)
- moved U303 7.62 mm to (130.8, 152.4)
- moved R301 7.62 mm to (123.2, 121.9)
- moved R305 7.62 mm to (123.2, 132.1)
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Routing:
- net /~{OE}: track 121.2 -> 3.64 mm, vias 2 -> 0
- net Net-(U202-Q0): track 89.3 -> 1.71 mm, vias 1 -> 0
- net Net-(U202-Q1): track 83.9 -> 1.68 mm, vias 1 -> 0
- net /Reg1.Out0: track 80.3 -> 0.00 mm, vias 2 -> 0
- net Net-(U202-Q2): track 78.8 -> 1.71 mm, vias 1 -> 0
- net /Reg1.Out2: track 75.3 -> 0.00 mm, vias 2 -> 0
- net /Reg1.Out1: track 74.7 -> 0.00 mm, vias 2 -> 0
- net Net-(U202-Q3): track 73.7 -> 1.68 mm, vias 1 -> 0
- net Net-(U302-Q0): track 73.7 -> 1.71 mm, vias 1 -> 0
- net /Reg1.Out4: track 70.2 -> 0.00 mm, vias 2 -> 0
- net /Reg1.Out3: track 69.6 -> 0.00 mm, vias 2 -> 0
- net Net-(U302-Q1): track 68.6 -> 1.71 mm, vias 1 -> 0
- net Net-(U202-Q4): track 68.6 -> 1.71 mm, vias 1 -> 0
- net /Reg1.Out6: track 65.1 -> 0.00 mm, vias 2 -> 0
- net /Reg1.Out5: track 64.6 -> 0.00 mm, vias 2 -> 0
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
Commit message: A little more editing
Routing:
- net /Reg0.Out7: track 64.6 -> 18.8 mm, vias 1 -> 0
- net /Reg0.Out6: track 62.0 -> 18.2 mm, vias 1 -> 0
- net /Reg0.Out5: track 59.5 -> 17.6 mm, vias 1 -> 0
- net /Reg0.Out3: track 54.4 -> 16.3 mm, vias 1 -> 0
- net /Reg0.Out2: track 51.9 -> 15.7 mm, vias 1 -> 0
- net /Reg0.Out1: track 49.3 -> 15.0 mm, vias 1 -> 0
- net /Reg0.Out0: track 46.8 -> 14.4 mm, vias 1 -> 0
- net /Reg0.Out4: track 56.9 -> 43.0 mm, vias 1 -> 0
Changed lines of the file:
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@@
 		(tags "capacitor")
 		(property "Reference" "C201"
-			(at 0 -1.43 360)
+			(at 0 -1.43 0)
 			(layer "F.SilkS")
 			(hide yes)
@@
 		)
 		(property "Value" "C"
-			(at 0 1.43 360)
+			(at 0 1.43 0)
 			(layer "F.Fab")
 			(effects
@@
 		)
 		(fp_text user "${REFERENCE}"
-			(at 0 0 360)
+			(at 0 0 0)
 			(layer "F.Fab")
 			(effects
@@
 		(tags "capacitor")
 		(property "Reference" "C301"
-			(at 0 -1.43 360)
+			(at 0 -1.43 0)
 			(layer "F.SilkS")
 			(hide yes)
@@
 		)
 		(property "Value" "C"
-			(at 0 1.43 360)
+			(at 0 1.43 0)
 			(layer "F.Fab")
 			(effects
@@
 		)
 		(fp_text user "${REFERENCE}"
-			(at 0 0 360)
+			(at 0 0 0)
 			(layer "F.Fab")
 			(effects
@@
 		(net 77)
 	)
-	(via
-		(at 107.315 104.775)
-		(size 0.45)
-		(drill 0.3)
-		(layers "F.Cu" "B.Cu")
-		(net 77)
-	)
-	(segment
-		(start 107.315 104.775)
-		(end 107.315 150.495)
-		(width 0.127)
-		(layer "B.Cu")
-		(net 77)
-	)
 	(segment
 		(start 126.16 108.585)
@@
 		(net 80)
 	)
-	(via
-		(at 109.22 108.585)
-		(size 0.45)
-		(drill 0.3)
-		(layers "F.Cu" "B.Cu")
-		(net 80)
-	)
 	(segment
 		(start 109.22 122.555)
@@
 	)
 	(segment
-		(start 109.22 108.585)
-		(end 109.22 122.555)
-		(width 0.127)
-		(layer "B.Cu")
-		(net 80)
-	)
-	(segment
 		(start 126.16 107.315)
 		(end 108.585 107.315)
@@
 		(net 81)
 	)
-	(via
-		(at 108.585 107.315)
-		(size 0.45)
-		(drill 0.3)
-		(layers "F.Cu" "B.Cu")
-		(net 81)
-	)
-	(segment
-		(start 108.585 107.315)
-		(end 108.585 149.225)
-		(width 0.127)
-		(layer "B.Cu")
-		(net 81)
-	)
 	(segment
 		(start 126.16 113.665)
@@
 		(net 82)
 	)
-	(via
-		(at 111.76 113.665)
-		(size 0.45)
-		(drill 0.3)
-		(layers "F.Cu" "B.Cu")
-		(net 82)
-	)
-	(segment
-		(start 111.76 113.665)
-		(end 111.76 146.05)
-		(width 0.127)
-		(layer "B.Cu")
-		(net 82)
-	)
 	(segment
 		(start 126.16 111.125)
@@
 		(net 87)
 	)
-	(via
-		(at 110.49 111.125)
-		(size 0.45)
-		(drill 0.3)
-		(layers "F.Cu" "B.Cu")
-		(net 87)
-	)
-	(segment
-		(start 110.49 115.57)
-		(end 110.49 147.32)
-		(width 0.127)
-		(layer "B.Cu")
-		(net 87)
-	)
-	(segment
-		(start 110.49 111.125)
-		(end 110.49 115.57)
-		(width 0.127)
-		(layer "B.Cu")
-		(net 87)
-	)
 	(segment
 		(start 126.16 109.855)
@@
 		(net 89)
 	)
-	(via
-		(at 109.855 109.855)
-		(size 0.45)
-		(drill 0.3)
-		(layers "F.Cu" "B.Cu")
-		(net 89)
-	)
-	(segment
-		(start 109.855 111.76)
-		(end 109.855 147.955)
-		(width 0.127)
-		(layer "B.Cu")
-		(net 89)
-	)
-	(segment
-		(start 109.855 109.855)
-		(end 109.855 111.76)
-		(width 0.127)
-		(layer "B.Cu")
-		(net 89)
-	)
 	(segment
 		(start 126.16 106.045)
@@
 		(net 90)
 	)
-	(via
-		(at 107.95 106.045)
-		(size 0.45)
-		(drill 0.3)
-		(layers "F.Cu" "B.Cu")
-		(net 90)
-	)
-	(segment
-		(start 107.95 106.045)
-		(end 107.95 149.86)
-		(width 0.127)
-		(layer "B.Cu")
-		(net 90)
-	)
 	(segment
 		(start 126.16 112.395)
@@
 		(net 92)
 	)
-	(via
-		(at 111.125 112.395)
-		(size 0.45)
-		(drill 0.3)
-		(layers "F.Cu" "B.Cu")
-		(net 92)
-	)
-	(segment
-		(start 111.125 112.395)
-		(end 111.125 146.685)
-		(width 0.127)
-		(layer "B.Cu")
-		(net 92)
-	)

Commit message: Get buses routed
Parts:
- moved R403 74.8 mm to (91.7, 148.6)
- moved R401 74.0 mm to (91.1, 153.0)
- moved C401 74.0 mm to (95.5, 149.2)
- moved R402 72.4 mm to (96.3, 152.4)
- moved U401 63.0 mm to (95.2, 141.0)
- moved U402 24.8 mm to (103.5, 98.4)
- moved R404 23.7 mm to (108.6, 95.9)
- moved R406 23.5 mm to (108.6, 99.2)
- moved C402 23.1 mm to (110.5, 95.9)
- moved C403 22.8 mm to (110.5, 99.2)
- moved R405 22.5 mm to (112.4, 95.9)
- moved R407 22.2 mm to (112.4, 99.2)
- moved J101 17.8 mm to (76.2, 102.9)
Connections:
- U203 pad 11: Net-(U202-Q0) -> Net-(U202-Q7)
- U203 pad 12: Net-(U202-Q1) -> Net-(U202-Q6)
- U203 pad 13: Net-(U202-Q2) -> Net-(U202-Q5)
- U203 pad 14: Net-(U202-Q3) -> Net-(U202-Q4)
- U203 pad 15: Net-(U202-Q4) -> Net-(U202-Q3)
- U203 pad 16: Net-(U202-Q5) -> Net-(U202-Q2)
- U203 pad 17: Net-(U202-Q6) -> Net-(U202-Q1)
- U203 pad 18: Net-(U202-Q7) -> Net-(U202-Q0)
- U203 pad 2: /Reg0.Out7 -> /Reg0.Out0
- U203 pad 3: /Reg0.Out6 -> /Reg0.Out1
- U203 pad 4: /Reg0.Out5 -> /Reg0.Out2
- U203 pad 5: /Reg0.Out4 -> /Reg0.Out3
- U203 pad 6: /Reg0.Out3 -> /Reg0.Out4
- U203 pad 7: /Reg0.Out2 -> /Reg0.Out5
- U203 pad 8: /Reg0.Out1 -> /Reg0.Out6
- U203 pad 9: /Reg0.Out0 -> /Reg0.Out7
- U303 pad 11: Net-(U302-Q0) -> Net-(U302-Q7)
- U303 pad 12: Net-(U302-Q1) -> Net-(U302-Q6)
- U303 pad 13: Net-(U302-Q2) -> Net-(U302-Q5)
- U303 pad 14: Net-(U302-Q3) -> Net-(U302-Q4)
- U303 pad 15: Net-(U302-Q4) -> Net-(U302-Q3)
- U303 pad 16: Net-(U302-Q5) -> Net-(U302-Q2)
- U303 pad 17: Net-(U302-Q6) -> Net-(U302-Q1)
- U303 pad 18: Net-(U302-Q7) -> Net-(U302-Q0)
- U303 pad 2: /Reg1.Out7 -> /Reg1.Out0
- U303 pad 3: /Reg1.Out6 -> /Reg1.Out1
- U303 pad 4: /Reg1.Out5 -> /Reg1.Out2
- U303 pad 5: /Reg1.Out4 -> /Reg1.Out3
- U303 pad 6: /Reg1.Out3 -> /Reg1.Out4
- U303 pad 7: /Reg1.Out2 -> /Reg1.Out5
- U303 pad 8: /Reg1.Out1 -> /Reg1.Out6
- U303 pad 9: /Reg1.Out0 -> /Reg1.Out7
Routing:
- net /Reg1.Out7: track 0.00 -> 58.8 mm, vias 0 -> 1
- net /Reg1.Out6: track 0.00 -> 58.2 mm, vias 0 -> 1
- net /Reg1.Out5: track 0.00 -> 57.6 mm, vias 0 -> 1
- net /Reg1.Out4: track 0.00 -> 56.9 mm, vias 0 -> 1
- net /Reg1.Out3: track 0.00 -> 52.5 mm, vias 0 -> 1
- net /Reg1.Out2: track 0.00 -> 51.9 mm, vias 0 -> 1
- net /Reg1.In0: track 0.00 -> 51.9 mm, vias 0 -> 2
- net /~{OE}: track 3.64 -> 55.0 mm, vias 0 -> 2
- net /Reg1.Out1: track 0.00 -> 49.3 mm, vias 0 -> 1
- net /Reg1.Out0: track 0.00 -> 48.7 mm, vias 0 -> 1
- net /Reg1.In7: track 0.00 -> 48.3 mm, vias 0 -> 1
- net /Reg1.In5: track 0.00 -> 47.0 mm, vias 0 -> 1
- net /Reg1.In6: track 0.00 -> 46.2 mm, vias 0 -> 2
- net /Reg1.In3: track 0.00 -> 45.8 mm, vias 0 -> 1
- net /Reg1.In4: track 0.00 -> 44.9 mm, vias 0 -> 2
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Other:
- board size 101.6 x 114.3 mm -> 83.8 x 101.6 mm

Commit message: Doing some tweaking
Parts:
- moved R209 24.1 mm to (141.0, 78.7)
- moved R210 23.9 mm to (141.6, 81.3)
- moved R211 23.7 mm to (142.2, 83.8)
- moved R212 23.5 mm to (142.9, 86.4)
- moved R213 23.4 mm to (143.5, 88.9)
- moved R214 23.3 mm to (144.1, 91.4)
- moved R215 23.2 mm to (144.8, 94.0)
- moved R216 23.1 mm to (145.4, 96.5)
- moved D203 22.9 mm to (152.4, 83.8)
- moved D305 22.9 mm to (152.4, 109.2)
- moved D201 22.9 mm to (152.4, 78.7)
- moved D202 22.9 mm to (152.4, 81.3)
- moved D204 22.9 mm to (152.4, 86.4)
- moved D205 22.9 mm to (152.4, 88.9)
- moved D206 22.9 mm to (152.4, 91.4)
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Connections:
- U402 pad 3: Net-(U401-Pad3) -> GND
- U402 pad 4: /Register 0/ZeroInput -> unconnected-(U402-Pad4)
- U402 pad 5: GND -> Net-(U401-Pad3)
- U402 pad 6: unconnected-(U402-Pad6) -> /Register 0/ZeroInput
Routing:
- net /ResetLogic/CLK_{Out}: track 0.00 -> 64.3 mm, vias 0 -> 2
- net Net-(U401-Pad3): track 0.00 -> 55.4 mm, vias 0 -> 3
- net /Register 0/ZeroInput: track 59.5 -> 91.0 mm, vias 2 -> 5
- net Net-(D301-A): track 2.20 -> 27.6 mm
- net Net-(D302-A): track 2.20 -> 27.0 mm
- net Net-(D306-A): track 2.20 -> 25.1 mm
- net Net-(D307-A): track 2.20 -> 25.1 mm
- net Net-(D303-A): track 2.20 -> 25.1 mm
- net Net-(D304-A): track 2.20 -> 25.1 mm
- net Net-(D305-A): track 2.20 -> 25.1 mm
- net Net-(D308-A): track 2.20 -> 25.1 mm
- net Net-(U202-Q7): track 13.8 -> 35.4 mm, vias 0 -> 2
- net /Reg1.Out0: track 48.7 -> 67.1 mm, vias 1 -> 2
- net /Reg1.Out1: track 49.3 -> 67.1 mm, vias 1 -> 2
- net /Reg1.Out2: track 51.9 -> 67.1 mm, vias 1 -> 2
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
Commit message: Everything connected
Parts:
- moved J101 10.2 mm to (86.4, 102.9)
- moved D201 2.54 mm to (149.9, 78.7)
- moved D202 2.54 mm to (149.9, 81.3)
- moved D203 2.54 mm to (149.9, 83.8)
- moved D204 2.54 mm to (149.9, 86.4)
- moved D205 2.54 mm to (149.9, 88.9)
- moved D206 2.54 mm to (149.9, 91.4)
- moved D207 2.54 mm to (149.9, 94.0)
- moved D208 2.54 mm to (149.9, 96.5)
- moved D301 2.54 mm to (149.9, 99.1)
- moved D302 2.54 mm to (149.9, 101.6)
- moved D303 2.54 mm to (149.9, 104.1)
- moved D304 2.54 mm to (149.9, 106.7)
- moved D305 2.54 mm to (149.9, 109.2)
- moved D306 2.54 mm to (149.9, 111.8)
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Routing:
- net /CLK: track 0.00 -> 58.8 mm, vias 0 -> 1
- net /~{RESET}: track 14.9 -> 64.5 mm, vias 0 -> 1
- net /~{OE}: track 55.0 -> 104.6 mm, vias 2 -> 4
- net +5V: track 21.0 -> 41.1 mm, vias 6 -> 8
- net /Reg0.In0: track 6.67 -> 20.5 mm
- net /Reg0.In1: track 8.31 -> 22.2 mm
- net /Reg0.In5: track 9.58 -> 22.2 mm
- net /Reg0.In2: track 8.58 -> 20.5 mm
- net /Reg1.In2: track 43.6 -> 54.3 mm
- net /Reg1.In1: track 44.5 -> 55.2 mm
- net /Reg0.In3: track 11.5 -> 22.2 mm
- net /Reg0.In4: track 10.5 -> 20.5 mm
- net /Reg0.In6: track 11.1 -> 20.5 mm
- net /Reg1.In4: track 44.9 -> 54.3 mm
- net /Reg1.In3: track 45.8 -> 55.2 mm
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Other:
- board size 83.8 x 101.6 mm -> 63.5 x 96.5 mm
- board text added: "RGE2024"
