File: pcbs/Incrementer/Incrementer.kicad_pcb (KiCad board)
At the start: 2 copper layers, 8.9 x 64.8 mm, 43 parts, among them U201 74HC283, U202 74HC245, U203 74HC283, U301 74HC283, U302 74HC245, U303 74HC283

Commit message: Basic routing
Parts:
- moved R208 8.13 mm to (85.7, 74.9)
- moved R302 8.13 mm to (85.7, 80.0)
- moved R304 8.13 mm to (85.7, 85.1)
- moved R306 8.13 mm to (85.7, 90.2)
- moved R201 8.13 mm to (85.7, 57.1)
- moved R205 8.13 mm to (85.7, 67.3)
- moved R202 8.13 mm to (85.7, 59.7)
- moved R203 8.13 mm to (85.7, 62.2)
- moved R204 8.13 mm to (85.7, 64.8)
- moved R206 8.13 mm to (85.7, 69.8)
- moved R207 8.13 mm to (85.7, 72.4)
- moved R301 8.13 mm to (85.7, 77.5)
- moved R303 8.13 mm to (85.7, 82.5)
- moved R305 8.13 mm to (85.7, 87.6)
- moved R307 8.13 mm to (85.7, 92.7)
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Routing:
- net /~{OE}: track 0.00 -> 103.6 mm, vias 0 -> 6
- net /Incremented1.Out1: track 7.41 -> 85.7 mm, vias 0 -> 3
- net /Incremented1.Out3: track 8.69 -> 85.7 mm, vias 0 -> 3
- net /Incremented1.Out2: track 8.05 -> 84.8 mm, vias 0 -> 2
- net /Incremented1.Out5: track 9.95 -> 85.7 mm, vias 0 -> 3
- net /Incremented1.Out4: track 9.32 -> 84.8 mm, vias 0 -> 2
- net /Incremented1.Out6: track 10.6 -> 84.8 mm, vias 0 -> 2
- net /Increment 8 Bits (Lower)/C_{Out}: track 0.00 -> 72.4 mm, vias 0 -> 3
- net /Incremented0.Out1: track 2.34 -> 50.1 mm, vias 1 -> 3
- net /Incremented0.Out3: track 3.61 -> 50.1 mm, vias 1 -> 3
- net /Incremented0.Out2: track 2.97 -> 49.2 mm, vias 1 -> 2
- net /Incremented0.Out5: track 4.88 -> 50.1 mm, vias 1 -> 3
- net /Incremented0.Out4: track 4.24 -> 49.2 mm, vias 1 -> 2
- net /Incremented0.Out6: track 11.2 -> 49.2 mm, vias 1 -> 2
- net /Increment 8 Bits (Upper)/Sum6: track 51.5 -> 84.0 mm, vias 2 -> 3
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- added copper zone on B.Cu, net +5V
- added copper zone on F.Cu, net GND
Other:
- board size 8.9 x 64.8 mm -> 67.3 x 95.2 mm
- board text added: "0"
- board text added: "10"
- board text added: "12"
- board text added: "14"
- board text added: "2"
- board text added: "4"
- board text added: "6"
- board text added: "8"
- board text added: "Incrementer"
- board text added: "JLCJLCJLCJLC"
- board text added: "RGE2024"
