File: pcbs/Barrel Shifter/shiftblock0.kicad_sch (KiCad schematic)
At the start: 1 part, among them U201 74HC138

Commit message: Starting to tidy up the LEDs
Parts:
- added C201: C, Capacitor_SMD:C_0603_1608Metric, symbol Device:C
Connections:
- net +5V: now also C201.1
- net GND: now also C201.2
- net ~{Enable}: now reaches U201.5 (~{E1})
