File: pcbs/Barrel Shifter/Barrel Shifter.kicad_sch (KiCad schematic)
At the start: 0 parts

Commit message: Second row
Other:
- added sheet Shift Block 1 (shiftblock1.kicad_sch)
- sheet Shift Block 0 ports: added A[0..15], Out[0..15]; removed none
Changed lines of the file:
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@@
 	(generator_version "8.0")
 	(paper "A4")
+	(bus
+		(pts
+			(xy 132.08 52.07) (xy 138.43 52.07)
+		)
+		(stroke
+			(width 0)
+			(type default)
+		)
+	)
+	(bus
+		(pts
+			(xy 132.08 80.01) (xy 138.43 80.01)
+		)
+		(stroke
+			(width 0)
+			(type default)
+		)
+	)
+	(bus
+		(pts
+			(xy 95.25 36.83) (xy 106.68 36.83)
+		)
+		(stroke
+			(width 0)
+			(type default)
+		)
+	)
+	(bus
+		(pts
+			(xy 138.43 52.07) (xy 138.43 80.01)
+		)
+		(stroke
+			(width 0)
+			(type default)
+		)
+	)
+	(bus
+		(pts
+			(xy 95.25 68.58) (xy 95.25 36.83)
+		)
+		(stroke
+			(width 0)
+			(type default)
+		)
+	)
+	(bus
+		(pts
+			(xy 106.68 68.58) (xy 95.25 68.58)
+		)
+		(stroke
+			(width 0)
+			(type default)
+		)
+	)
 	(sheet
-		(at 63.5 92.075)
-		(size 62.23 48.895)
+		(at 106.68 31.75)
+		(size 25.4 24.765)
 		(fields_autoplaced yes)
 		(stroke
@@
 		)
 		(property "Sheetname" "Shift Block 0"
-			(at 63.5 91.3634 0)
+			(at 106.68 31.0384 0)
 			(effects
 				(font
@@
 		)
 		(property "Sheetfile" "shiftblock0.kicad_sch"
-			(at 63.5 141.5546 0)
+			(at 106.68 57.0996 0)
 			(effects
 				(font
@@
 				)
 				(justify left top)
+			)
+		)
+		(pin "Out[0..15]" tri_state
+			(at 132.08 52.07 0)
+			(effects
+				(font
+					(size 1.27 1.27)
+				)
+				(justify right)
+			)
+		)
+		(pin "A[0..15]" input
+			(at 106.68 36.83 180)
+			(effects
+				(font
+					(size 1.27 1.27)
+				)
+				(justify left)
 			)
 		)
@@
 				)
 			)
+		)
+	)
+	(sheet
+		(at 106.68 62.865)
+		(size 25.4 23.495)
+		(fields_autoplaced yes)
+		(stroke
+			(width 0.1524)
+			(type solid)
+		)
+		(fill
+			(color 0 0 0 0.0000)
+		)
+		(property "Sheetname" "Shift Block 1"
+			(at 106.68 62.1534 0)
+			(effects
+				(font
+					(size 1.27 1.27)
+				)
+				(justify left bottom)
+			)
+		)
+		(property "Sheetfile" "shiftblock1.kicad_sch"
+			(at 106.68 86.9446 0)
+			(effects
+				(font
+					(size 1.27 1.27)
+				)
+				(justify left top)
+			)
+		)
+		(pin "Out[0..15]" tri_state
+			(at 132.08 80.01 0)
+			(effects
+				(font
+					(size 1.27 1.27)
+				)
+				(justify right)
+			)
+		)
+		(pin "A[0..15]" input
+			(at 106.68 68.58 180)
+			(effects
+				(font
+					(size 1.27 1.27)
+				)
+				(justify left)
+			)
+		)
+		(instances
+			(project "Barrel Shifter"
+				(path "/f9807743-2893-4e61-9d6a-d5b530ea0d07"
+					(page "2")
+				)
+			)

Commit message: Significant rethinking
Parts:
- added C101: C, Capacitor_SMD:C_0603_1608Metric, symbol Device:C
- added U101: 74HC138, Package_DIP:DIP-16_W7.62mm_Socket, symbol 74xx:74HC138
Connections:
- new net +5V: C101.1, U101.16 (VCC)
- new net GND: C101.2, U101.8 (GND)
- new net ~{Enable}: U101.5 (~{E1})
- new net ~{Y0}: U101.15 (~{Y0})
- new net ~{Y1}: U101.14 (~{Y1})
- new net ~{Y2}: U101.13 (~{Y2})
- new net ~{Y3}: U101.12 (~{Y3})
- new net ~{Y4}: U101.11 (~{Y4})
- new net ~{Y5}: U101.10 (~{Y5})
- new net ~{Y6}: U101.9 (~{Y6})
- new net ~{Y7}: U101.7 (~{Y7})
Other:
- removed sheet Shift Block 0
- removed sheet Shift Block 1
- added sheet Shifter 0 (shifter.kicad_sch)
- added sheet Shifter 1 (shifter.kicad_sch)
- added sheet Shifter 2 (shifter.kicad_sch)
- added sheet Shifter 3 (shifter.kicad_sch)
- added sheet Shifter 4 (shifter.kicad_sch)
- added sheet Shifter 5 (shifter.kicad_sch)
- added sheet Shifter 6 (shifter.kicad_sch)
- added sheet Shifter 7 (shifter.kicad_sch)

Commit message: Almost there...
Parts:
- added J101: ~, BoardEdgeConnectors:TE-5530843-4-Edge, symbol BoardEdgeConnectors:TE-5530843-4
Connections:
- net +5V: now also U101.6 (E2), J101.B1
- net A0: now also J101.A2
- net A1: now also J101.B2
- net A10: now also J101.A7
- net A11: now also J101.B7
- net A12: now also J101.A8
- net A13: now also J101.B8
- net A14: now also J101.A9
- net A15: now also J101.B9
- net A2: now also J101.A3
- net A3: now also J101.B3
- net A4: now also J101.A4
- net A5: now also J101.B4
- net A6: now also J101.A5
- net A7: now also J101.B5
- net A8: now also J101.A6
- net A9: now also J101.B6
- net GND: now also J101.A22
- net B_0: now reaches U101.1 (A0)
- net B_0: now also J101.A11
- net B_1: now reaches U101.2 (A1)
- net B_1: now also J101.B11
- net B_2: now reaches U101.3 (A2)
- net B_2: now also J101.A12
- net B_3: now reaches U101.4 (~{E0})
- net B_3: now also J101.B12
- net ~{Enable} renamed ~{OE}
- net ~{OE}: now also J101.A13
- new net C0: J101.A14
- new net C1: J101.B14
- new net C10: J101.A19
- new net C11: J101.B19
- new net C12: J101.A20
- new net C13: J101.B20
- new net C14: J101.A21
- new net C15: J101.B21
- new net C2: J101.A15
- new net C3: J101.B15
- new net C4: J101.A16
- new net C5: J101.B16
- new net C6: J101.A17
- new net C7: J101.B17
- new net C8: J101.A18
- new net C9: J101.B18
- no-connect marks 0 -> 5
