File: pcbs/Barrel Shifter/shifter.kicad_sch (KiCad schematic)
At the start: 4 parts, among them U301 74HC245, U302 74HC245

Commit message: Second row
Parts:
- renumbered D301 to D601, R301 to R601, U301 to U601, U302 to U602

Commit message: Significant rethinking
Parts:
- renumbered D601 to D201, R601 to R201, U601 to U201, U602 to U202

Commit message: Almost there...
Parts:
- renumbered D201 to D901, R201 to R901, U201 to U901, U202 to U902
Changed lines of the file:
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@@
 		(dnp no)
 		(fields_autoplaced yes)
-		(property "Reference" "R201"
+		(property "Reference" "R901"
 			(at 34.29 78.74 90)
 			(effects
@@
 		(dnp no)
 		(fields_autoplaced yes)
-		(property "Reference" "#PWR0207"
+		(property "Reference" "#PWR0907"
 			(at 77.47 146.05 0)
 			(effects
@@
 		(dnp no)
 		(fields_autoplaced yes)
-		(property "Reference" "#PWR0202"
+		(property "Reference" "#PWR0902"
 			(at 62.23 68.58 0)
 			(effects
@@
 		(on_board yes)
 		(dnp no)
-		(property "Reference" "D201"
+		(property "Reference" "D901"
 			(at 46.0375 78.105 0)
 			(effects
@@
 		(dnp no)
 		(fields_autoplaced yes)
-		(property "Reference" "#PWR0201"
+		(property "Reference" "#PWR0901"
 			(at 30.48 85.09 0)
 			(effects
@@
 		(dnp no)
 		(fields_autoplaced yes)
-		(property "Reference" "#PWR0205"
+		(property "Reference" "#PWR0905"
 			(at 77.47 86.36 0)
 			(effects
@@
 		(dnp no)
 		(fields_autoplaced yes)
-		(property "Reference" "#PWR0204"
+		(property "Reference" "#PWR0904"
 			(at 77.47 39.37 0)
 			(effects
@@
 		(dnp no)
 		(fields_autoplaced yes)
-		(property "Reference" "#PWR0203"
+		(property "Reference" "#PWR0903"
 			(at 62.23 128.27 0)
 			(effects
@@
 		(dnp no)
 		(fields_autoplaced yes)
-		(property "Reference" "U202"
+		(property "Reference" "U902"
 			(at 79.4894 97.79 0)
 			(effects
@@
 		(dnp no)
 		(fields_autoplaced yes)
-		(property "Reference" "U201"
+		(property "Reference" "U901"
 			(at 79.4894 38.1 0)
 			(effects
@@
 		(dnp no)
 		(fields_autoplaced yes)
-		(property "Reference" "#PWR0206"
+		(property "Reference" "#PWR0906"
 			(at 77.47 99.06 0)
 			(effects
