File: pcbs/Register File/Register File.kicad_pcb (KiCad board)
At the start: 2 copper layers, 222 parts, among them U1003 74HC138, U1004 74HC540, U1005 74HC138, U1006 74HC138, U201 74HCT574, U202 74HC245, U203 74HC245, U301 74HCT574, U302 74HC245, U303 74HC245, U401 74HCT574, U402 74HC245, U403 74HC245, U501 74HCT574, U502 74HC245, U503 74HC245, U601 74HCT574, U602 74HC245, U603 74HC245, U701 74HCT574, U702 74HC245, U703 74HC245, U801 74HCT574, U802 74HC245, U803 74HC245, U901 74HCT574, U902 74HC245, U903 74HC245

Commit message: Roughing out some layout
Parts:
- moved D906 354.9 mm to (294.5, 24.6)
- moved D907 354.9 mm to (294.5, 27.2)
- moved D908 354.9 mm to (294.5, 29.7)
- moved D909 354.9 mm to (294.5, 32.3)
- moved D910 354.9 mm to (294.5, 34.9)
- moved C901 354.9 mm to (282.4, 24.5)
- moved D901 354.9 mm to (290.4, 24.6)
- moved D902 354.9 mm to (290.4, 27.2)
- moved D903 354.9 mm to (290.4, 29.7)
- moved D904 354.9 mm to (290.4, 32.3)
- moved D905 354.9 mm to (290.4, 34.9)
- moved R901 354.9 mm to (282.4, 27.0)
- moved R902 354.9 mm to (282.4, 29.5)
- moved R903 354.9 mm to (282.4, 32.1)
- moved R904 354.9 mm to (282.4, 34.6)
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Connections:
- net /Selectors/C_{Write}1 renamed /Selectors/CW1
- net /Selectors/C_{Write}2 renamed /Selectors/CW2
- net /Selectors/C_{Write}3 renamed /Selectors/CW3
- net /Selectors/C_{Write}4 renamed /Selectors/CW4
- net /Selectors/C_{Write}5 renamed /Selectors/CW5
- net /Selectors/C_{Write}6 renamed /Selectors/CW6
- net /Selectors/C_{Write}7 renamed /Selectors/CW7
- net /Selectors/~{A_{select}}1 renamed /Selectors/~{AS}1
- net /Selectors/~{A_{select}}2 renamed /Selectors/~{AS}2
- net /Selectors/~{A_{select}}3 renamed /Selectors/~{AS}3
- net /Selectors/~{A_{select}}4 renamed /Selectors/~{AS}4
- net /Selectors/~{A_{select}}5 renamed /Selectors/~{AS}5
- net /Selectors/~{A_{select}}6 renamed /Selectors/~{AS}6
- net /Selectors/~{A_{select}}7 renamed /Selectors/~{AS}7
- net /Selectors/~{B_{select}}1 renamed /Selectors/~{BS}1
- net /Selectors/~{B_{select}}2 renamed /Selectors/~{BS}2
- net /Selectors/~{B_{select}}3 renamed /Selectors/~{BS}3
- net /Selectors/~{B_{select}}4 renamed /Selectors/~{BS}4
- net /Selectors/~{B_{select}}5 renamed /Selectors/~{BS}5
- net /Selectors/~{B_{select}}6 renamed /Selectors/~{BS}6
- net /Selectors/~{B_{select}}7 renamed /Selectors/~{BS}7
- D209 pad 1: /Register 0/~{A_{Enable}} -> /Selectors/~{AS}0
- D211 pad 1: /Register 0/~{B_{Enable}} -> /Selectors/~{BS}0
- R1001 pad 1: /Selectors/C_{Write}0 -> /Selectors/CW0
- U1004 pad 18: /Selectors/C_{Write}0 -> /Selectors/CW0
- U1005 pad 15: /Selectors/~{A_{select}}0 -> /Selectors/~{AS}0
- U1006 pad 15: /Selectors/~{B_{select}}0 -> /Selectors/~{BS}0
- U201 pad 11: /Register 0/C_{write} -> /Selectors/CW0
- U202 pad 19: /Register 0/~{A_{Enable}} -> /Selectors/~{AS}0
- U203 pad 19: /Register 0/~{B_{Enable}} -> /Selectors/~{BS}0
- U302 pad 11: /Register 1/A7 -> /Register 0/A7
- U302 pad 12: /Register 1/A6 -> /Register 0/A6
- U302 pad 13: /Register 1/A5 -> /Register 0/A5
- U302 pad 14: /Register 1/A4 -> /Register 0/A4
- U302 pad 15: /Register 1/A3 -> /Register 0/A3
- U302 pad 16: /Register 1/A2 -> /Register 0/A2
- U302 pad 17: /Register 1/A1 -> /Register 0/A1
- U302 pad 18: /Register 1/A0 -> /Register 0/A0
- U303 pad 11: /Register 1/B7 -> /Register 0/B7
- U303 pad 12: /Register 1/B6 -> /Register 0/B6
- U303 pad 13: /Register 1/B5 -> /Register 0/B5
- U303 pad 14: /Register 1/B4 -> /Register 0/B4
- U303 pad 15: /Register 1/B3 -> /Register 0/B3
- U303 pad 16: /Register 1/B2 -> /Register 0/B2
- U303 pad 17: /Register 1/B1 -> /Register 0/B1
- U303 pad 18: /Register 1/B0 -> /Register 0/B0
- U401 pad 2: /Register 2/C0 -> /Register 0/C0
- U401 pad 3: /Register 2/C1 -> /Register 0/C1
- U401 pad 4: /Register 2/C2 -> /Register 0/C2
- U401 pad 5: /Register 2/C3 -> /Register 0/C3
- U401 pad 6: /Register 2/C4 -> /Register 0/C4
- U401 pad 7: /Register 2/C5 -> /Register 0/C5
- U401 pad 8: /Register 2/C6 -> /Register 0/C6
- U401 pad 9: /Register 2/C7 -> /Register 0/C7
- U402 pad 11: /Register 2/A7 -> /Register 0/A7
- U402 pad 12: /Register 2/A6 -> /Register 0/A6
- U402 pad 13: /Register 2/A5 -> /Register 0/A5
- U402 pad 14: /Register 2/A4 -> /Register 0/A4
- U402 pad 15: /Register 2/A3 -> /Register 0/A3
- U402 pad 16: /Register 2/A2 -> /Register 0/A2
- U402 pad 17: /Register 2/A1 -> /Register 0/A1
- U402 pad 18: /Register 2/A0 -> /Register 0/A0
- U403 pad 11: /Register 2/B7 -> /Register 0/B7
- U403 pad 12: /Register 2/B6 -> /Register 0/B6
- U403 pad 13: /Register 2/B5 -> /Register 0/B5
- U403 pad 14: /Register 2/B4 -> /Register 0/B4
- U403 pad 15: /Register 2/B3 -> /Register 0/B3
- U403 pad 16: /Register 2/B2 -> /Register 0/B2
- U403 pad 17: /Register 2/B1 -> /Register 0/B1
- U403 pad 18: /Register 2/B0 -> /Register 0/B0
- U501 pad 2: /Register 3/C0 -> /Register 0/C0
- U501 pad 3: /Register 3/C1 -> /Register 0/C1
- U501 pad 4: /Register 3/C2 -> /Register 0/C2
- U501 pad 5: /Register 3/C3 -> /Register 0/C3
- U501 pad 6: /Register 3/C4 -> /Register 0/C4
- U501 pad 7: /Register 3/C5 -> /Register 0/C5
- U501 pad 8: /Register 3/C6 -> /Register 0/C6
- U501 pad 9: /Register 3/C7 -> /Register 0/C7
- U502 pad 11: /Register 3/A7 -> /Register 0/A7
- U502 pad 12: /Register 3/A6 -> /Register 0/A6
- U502 pad 13: /Register 3/A5 -> /Register 0/A5
- U502 pad 14: /Register 3/A4 -> /Register 0/A4
- U502 pad 15: /Register 3/A3 -> /Register 0/A3
- U502 pad 16: /Register 3/A2 -> /Register 0/A2
- U502 pad 17: /Register 3/A1 -> /Register 0/A1
- U502 pad 18: /Register 3/A0 -> /Register 0/A0
- U503 pad 11: /Register 3/B7 -> /Register 0/B7
- U503 pad 12: /Register 3/B6 -> /Register 0/B6
- U503 pad 13: /Register 3/B5 -> /Register 0/B5
- U503 pad 14: /Register 3/B4 -> /Register 0/B4
- U503 pad 15: /Register 3/B3 -> /Register 0/B3
- U503 pad 16: /Register 3/B2 -> /Register 0/B2
- U503 pad 17: /Register 3/B1 -> /Register 0/B1
- U503 pad 18: /Register 3/B0 -> /Register 0/B0
- U601 pad 2: /Register 4/C0 -> /Register 0/C0
- U601 pad 3: /Register 4/C1 -> /Register 0/C1
- U601 pad 4: /Register 4/C2 -> /Register 0/C2
- U601 pad 5: /Register 4/C3 -> /Register 0/C3
- U601 pad 6: /Register 4/C4 -> /Register 0/C4
- U601 pad 7: /Register 4/C5 -> /Register 0/C5
- U601 pad 8: /Register 4/C6 -> /Register 0/C6
- U601 pad 9: /Register 4/C7 -> /Register 0/C7
- U602 pad 11: /Register 4/A7 -> /Register 0/A7
- U602 pad 12: /Register 4/A6 -> /Register 0/A6
- U602 pad 13: /Register 4/A5 -> /Register 0/A5
- U602 pad 14: /Register 4/A4 -> /Register 0/A4
- U602 pad 15: /Register 4/A3 -> /Register 0/A3
- U602 pad 16: /Register 4/A2 -> /Register 0/A2
- U602 pad 17: /Register 4/A1 -> /Register 0/A1
- U602 pad 18: /Register 4/A0 -> /Register 0/A0
- U603 pad 11: /Register 4/B7 -> /Register 0/B7
- U603 pad 12: /Register 4/B6 -> /Register 0/B6
- U603 pad 13: /Register 4/B5 -> /Register 0/B5
- U603 pad 14: /Register 4/B4 -> /Register 0/B4
- U603 pad 15: /Register 4/B3 -> /Register 0/B3
- U603 pad 16: /Register 4/B2 -> /Register 0/B2
- U603 pad 17: /Register 4/B1 -> /Register 0/B1
- U603 pad 18: /Register 4/B0 -> /Register 0/B0
- U701 pad 2: /Register 5/C0 -> /Register 0/C0
- U701 pad 3: /Register 5/C1 -> /Register 0/C1
- U701 pad 4: /Register 5/C2 -> /Register 0/C2
- U701 pad 5: /Register 5/C3 -> /Register 0/C3
- U701 pad 6: /Register 5/C4 -> /Register 0/C4
- U701 pad 7: /Register 5/C5 -> /Register 0/C5
- U701 pad 8: /Register 5/C6 -> /Register 0/C6
- U701 pad 9: /Register 5/C7 -> /Register 0/C7
- U702 pad 11: /Register 5/A7 -> /Register 0/A7
- U702 pad 12: /Register 5/A6 -> /Register 0/A6
- U702 pad 13: /Register 5/A5 -> /Register 0/A5
- U702 pad 14: /Register 5/A4 -> /Register 0/A4
- U702 pad 15: /Register 5/A3 -> /Register 0/A3
- U702 pad 16: /Register 5/A2 -> /Register 0/A2
- U702 pad 17: /Register 5/A1 -> /Register 0/A1
- U702 pad 18: /Register 5/A0 -> /Register 0/A0
- U703 pad 11: /Register 5/B7 -> /Register 0/B7
- U703 pad 12: /Register 5/B6 -> /Register 0/B6
- U703 pad 13: /Register 5/B5 -> /Register 0/B5
- U703 pad 14: /Register 5/B4 -> /Register 0/B4
- U703 pad 15: /Register 5/B3 -> /Register 0/B3
- U703 pad 16: /Register 5/B2 -> /Register 0/B2
- U703 pad 17: /Register 5/B1 -> /Register 0/B1
- U703 pad 18: /Register 5/B0 -> /Register 0/B0
- U801 pad 2: /Register 6/C0 -> /Register 0/C0
- U801 pad 3: /Register 6/C1 -> /Register 0/C1
- U801 pad 4: /Register 6/C2 -> /Register 0/C2
- U801 pad 5: /Register 6/C3 -> /Register 0/C3
- U801 pad 6: /Register 6/C4 -> /Register 0/C4
- U801 pad 7: /Register 6/C5 -> /Register 0/C5
- U801 pad 8: /Register 6/C6 -> /Register 0/C6
- U801 pad 9: /Register 6/C7 -> /Register 0/C7
- U802 pad 11: /Register 6/A7 -> /Register 0/A7
- U802 pad 12: /Register 6/A6 -> /Register 0/A6
- U802 pad 13: /Register 6/A5 -> /Register 0/A5
- U802 pad 14: /Register 6/A4 -> /Register 0/A4
- U802 pad 15: /Register 6/A3 -> /Register 0/A3
- U802 pad 16: /Register 6/A2 -> /Register 0/A2
- U802 pad 17: /Register 6/A1 -> /Register 0/A1
- U802 pad 18: /Register 6/A0 -> /Register 0/A0
- U803 pad 11: /Register 6/B7 -> /Register 0/B7
- U803 pad 12: /Register 6/B6 -> /Register 0/B6
- U803 pad 13: /Register 6/B5 -> /Register 0/B5
- U803 pad 14: /Register 6/B4 -> /Register 0/B4
- U803 pad 15: /Register 6/B3 -> /Register 0/B3
- U803 pad 16: /Register 6/B2 -> /Register 0/B2
- U803 pad 17: /Register 6/B1 -> /Register 0/B1
- U803 pad 18: /Register 6/B0 -> /Register 0/B0
- U901 pad 2: /Register 7/C0 -> /Register 0/C0
- U901 pad 3: /Register 7/C1 -> /Register 0/C1
- U901 pad 4: /Register 7/C2 -> /Register 0/C2
- U901 pad 5: /Register 7/C3 -> /Register 0/C3
- U901 pad 6: /Register 7/C4 -> /Register 0/C4
- U901 pad 7: /Register 7/C5 -> /Register 0/C5
- U901 pad 8: /Register 7/C6 -> /Register 0/C6
- U901 pad 9: /Register 7/C7 -> /Register 0/C7
- U902 pad 11: /Register 7/A7 -> /Register 0/A7
- U902 pad 12: /Register 7/A6 -> /Register 0/A6
- U902 pad 13: /Register 7/A5 -> /Register 0/A5
- U902 pad 14: /Register 7/A4 -> /Register 0/A4
- U902 pad 15: /Register 7/A3 -> /Register 0/A3
- U902 pad 16: /Register 7/A2 -> /Register 0/A2
- U902 pad 17: /Register 7/A1 -> /Register 0/A1
- U902 pad 18: /Register 7/A0 -> /Register 0/A0
- U903 pad 11: /Register 7/B7 -> /Register 0/B7
- U903 pad 12: /Register 7/B6 -> /Register 0/B6
- U903 pad 13: /Register 7/B5 -> /Register 0/B5
- U903 pad 14: /Register 7/B4 -> /Register 0/B4
- U903 pad 15: /Register 7/B3 -> /Register 0/B3
- U903 pad 16: /Register 7/B2 -> /Register 0/B2
- U903 pad 17: /Register 7/B1 -> /Register 0/B1
- U903 pad 18: /Register 7/B0 -> /Register 0/B0
Routing:
- net /Register 1/r0: track 0.00 -> 76.5 mm
- net /Register 1/r1: track 0.00 -> 70.7 mm
- net /Register 1/r2: track 0.00 -> 68.8 mm
- net /Register 1/r3: track 0.00 -> 66.9 mm
- net /Register 1/r4: track 0.00 -> 65.0 mm
- net /Register 1/r5: track 0.00 -> 63.1 mm
- net /Register 1/r6: track 0.00 -> 61.2 mm
- net /Register 0/r6: track 17.0 -> 76.9 mm, vias 1 -> 0
- net /Register 1/r7: track 0.00 -> 59.3 mm
- net /Register 0/r7: track 13.8 -> 62.3 mm, vias 1 -> 0
- net /Register 0/r3: track 26.5 -> 74.4 mm, vias 1 -> 0
- net /Register 0/r1: track 32.9 -> 80.1 mm, vias 1 -> 0
- net /Register 0/r5: track 20.2 -> 66.2 mm, vias 1 -> 0
- net /Register 0/r4: track 23.3 -> 68.1 mm, vias 1 -> 0
- net /Register 0/r2: track 29.7 -> 71.9 mm, vias 1 -> 0
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
Commit message: Lots of thinking and routing
Parts:
- moved D1005 159.0 mm to (210.8, 47.6)
- moved R1013 134.7 mm to (203.2, 47.6)
- moved D1004 134.1 mm to (185.4, 47.6)
- moved R1012 111.4 mm to (177.8, 47.6)
- moved D1003 109.4 mm to (160.0, 47.8)
- moved R1003 108.0 mm to (169.7, 48.8), turned to 180 degrees
- moved R1011 86.4 mm to (152.4, 47.8)
- moved D1002 85.3 mm to (134.6, 47.8)
- moved R1002 83.3 mm to (144.1, 48.3), turned to 180 degrees
- moved D510 78.4 mm to (196.2, 116.8), turned to 180 degrees
- moved R510 77.9 mm to (196.2, 114.9)
- moved R1010 62.0 mm to (127.0, 47.8)
- moved R509 50.7 mm to (196.2, 84.5)
- moved D509 50.6 mm to (196.2, 86.4), turned to 180 degrees
- moved R508 39.5 mm to (193.0, 71.1), turned to 180 degrees
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Connections:
- D309 pad 1: /Register 1/~{A_{Enable}} -> /Selectors/~{AS}1
- D310 pad 1: /Register 1/~{B_{Enable}} -> /Selectors/~{BS}1
- D409 pad 1: /Register 2/~{A_{Enable}} -> /Selectors/~{AS}2
- D410 pad 1: /Register 2/~{B_{Enable}} -> /Selectors/~{BS}2
- D509 pad 1: /Register 3/~{A_{Enable}} -> /Selectors/~{AS}3
- D510 pad 1: /Register 3/~{B_{Enable}} -> /Selectors/~{BS}3
- U301 pad 11: /Register 1/C_{write} -> /Selectors/CW1
- U302 pad 19: /Register 1/~{A_{Enable}} -> /Selectors/~{AS}1
- U303 pad 19: /Register 1/~{B_{Enable}} -> /Selectors/~{BS}1
- U401 pad 11: /Register 2/C_{write} -> /Selectors/CW2
- U402 pad 19: /Register 2/~{A_{Enable}} -> /Selectors/~{AS}2
- U403 pad 19: /Register 2/~{B_{Enable}} -> /Selectors/~{BS}2
- U501 pad 11: /Register 3/C_{write} -> /Selectors/CW3
- U501 pad 2: /Register 0/C0 -> /Register 3/C0
- U501 pad 3: /Register 0/C1 -> /Register 3/C1
- U501 pad 4: /Register 0/C2 -> /Register 3/C2
- U501 pad 5: /Register 0/C3 -> /Register 3/C3
- U501 pad 6: /Register 0/C4 -> /Register 3/C4
- U501 pad 7: /Register 0/C5 -> /Register 3/C5
- U501 pad 8: /Register 0/C6 -> /Register 3/C6
- U501 pad 9: /Register 0/C7 -> /Register 3/C7
- U502 pad 19: /Register 3/~{A_{Enable}} -> /Selectors/~{AS}3
- U503 pad 19: /Register 3/~{B_{Enable}} -> /Selectors/~{BS}3
Routing:
- net /Selectors/CW3: track 0.00 -> 130.4 mm, vias 0 -> 2
- net /Selectors/CW2: track 0.00 -> 127.9 mm, vias 0 -> 2
- net /Selectors/CW1: track 0.00 -> 120.5 mm, vias 0 -> 2
- net /Selectors/~{BS}3: track 0.00 -> 112.2 mm, vias 0 -> 2
- net /Selectors/CW7: track 0.00 -> 106.7 mm, vias 0 -> 2
- net /Selectors/~{AS}3: track 0.00 -> 105.2 mm, vias 0 -> 2
- net /Selectors/CW6: track 0.00 -> 102.9 mm, vias 0 -> 2
- net /Selectors/CW5: track 0.00 -> 99.1 mm, vias 0 -> 2
- net /Selectors/CW4: track 0.00 -> 95.2 mm, vias 0 -> 2
- net /Register 2/r0: track 0.00 -> 88.8 mm, vias 0 -> 2
- net /Register 3/r0: track 0.00 -> 88.8 mm, vias 0 -> 2
- net /Selectors/~{BS}2: track 0.00 -> 86.2 mm, vias 0 -> 2
- net /Register 2/r1: track 0.00 -> 85.6 mm, vias 0 -> 2
- net /Register 3/r1: track 0.00 -> 85.6 mm, vias 0 -> 2
- net /Register 2/r2: track 0.00 -> 82.4 mm, vias 0 -> 2
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
Commit message: Lots of routing
Parts:
- moved D1008 235.1 mm to (287.0, 47.6)
- moved R1008 229.9 mm to (295.9, 47.6), turned to 180 degrees
- moved D1007 209.8 mm to (261.6, 47.6)
- moved R1016 209.2 mm to (279.4, 47.6)
- moved R1007 204.9 mm to (270.5, 47.6), turned to 180 degrees
- moved D1006 184.6 mm to (236.2, 47.6)
- moved R1015 184.2 mm to (254.0, 47.6)
- moved R1006 180.0 mm to (245.1, 47.6), turned to 180 degrees
- moved R1014 159.3 mm to (228.6, 47.6)
- moved R1005 157.1 mm to (219.7, 47.6), turned to 180 degrees
- moved R1004 132.0 mm to (194.3, 47.6), turned to 180 degrees
- moved D910 82.0 mm to (297.8, 116.8), turned to 180 degrees
- moved D710 81.7 mm to (247.0, 116.8), turned to 180 degrees
- moved R710 81.4 mm to (247.0, 114.9)
- moved R910 81.2 mm to (297.8, 114.9), turned to 180 degrees
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Connections:
- D609 pad 1: /Register 4/~{A_{Enable}} -> /Selectors/~{AS}4
- D610 pad 1: /Register 4/~{B_{Enable}} -> /Selectors/~{BS}4
- D709 pad 1: /Register 5/~{A_{Enable}} -> /Selectors/~{AS}5
- D710 pad 1: /Register 5/~{B_{Enable}} -> /Selectors/~{BS}5
- D809 pad 1: /Register 6/~{A_{Enable}} -> /Selectors/~{AS}6
- D810 pad 1: /Register 6/~{B_{Enable}} -> /Selectors/~{BS}6
- D909 pad 1: /Register 7/~{A_{Enable}} -> /Selectors/~{AS}7
- D910 pad 1: /Register 7/~{B_{Enable}} -> /Selectors/~{BS}7
- U601 pad 11: /Register 4/C_{write} -> /Selectors/CW4
- U602 pad 19: /Register 4/~{A_{Enable}} -> /Selectors/~{AS}4
- U603 pad 19: /Register 4/~{B_{Enable}} -> /Selectors/~{BS}4
- U701 pad 11: /Register 5/C_{write} -> /Selectors/CW5
- U702 pad 19: /Register 5/~{A_{Enable}} -> /Selectors/~{AS}5
- U703 pad 19: /Register 5/~{B_{Enable}} -> /Selectors/~{BS}5
- U801 pad 11: /Register 6/C_{write} -> /Selectors/CW6
- U802 pad 19: /Register 6/~{A_{Enable}} -> /Selectors/~{AS}6
- U803 pad 19: /Register 6/~{B_{Enable}} -> /Selectors/~{BS}6
- U901 pad 11: /Register 7/C_{write} -> /Selectors/CW7
- U902 pad 19: /Register 7/~{A_{Enable}} -> /Selectors/~{AS}7
- U903 pad 19: /Register 7/~{B_{Enable}} -> /Selectors/~{BS}7
Routing:
- net /Selectors/W7: track 0.00 -> 258.7 mm, vias 0 -> 2
- net /Selectors/~{BS}6: track 0.00 -> 227.1 mm, vias 0 -> 2
- net /Selectors/W6: track 0.00 -> 218.1 mm, vias 0 -> 2
- net /Selectors/~{BS}7: track 0.00 -> 216.3 mm, vias 0 -> 2
- net /Selectors/~{AS}7: track 0.00 -> 209.3 mm, vias 0 -> 2
- net /Selectors/W5: track 0.00 -> 201.0 mm, vias 0 -> 2
- net /Selectors/CW7: track 106.7 -> 307.0 mm, vias 2 -> 3
- net /Selectors/~{BS}4: track 0.00 -> 190.3 mm, vias 0 -> 2
- net /Selectors/~{AS}6: track 0.00 -> 183.3 mm, vias 0 -> 2
- net /Selectors/CW6: track 102.9 -> 276.5 mm, vias 2 -> 3
- net /Selectors/~{AS}5: track 0.00 -> 171.2 mm, vias 0 -> 2
- net /Selectors/~{BS}5: track 0.00 -> 164.3 mm, vias 0 -> 2
- net /Selectors/W4: track 0.00 -> 161.0 mm, vias 0 -> 2
- net /Register 0/A0: track 77.8 -> 230.6 mm, vias 0 -> 1
- net /Register 0/A1: track 77.8 -> 228.0 mm, vias 0 -> 1
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
Commit message: Compaction
Parts:
- moved U1006 17.0 mm to (94.0, 106.7), turned to -90 degrees
- moved U1005 15.2 mm to (94.0, 86.4), turned to -90 degrees
- moved R810 14.0 mm to (263.5, 104.1), turned to 180 degrees
- moved R510 14.0 mm to (187.3, 104.1), turned to 180 degrees
- moved R610 14.0 mm to (212.7, 104.1), turned to 180 degrees
- moved R310 14.0 mm to (136.5, 104.1), turned to 180 degrees
- moved R410 14.0 mm to (161.9, 104.1), turned to 180 degrees
- moved R710 14.0 mm to (238.1, 104.1), turned to 180 degrees
- moved R910 14.0 mm to (288.9, 104.1)
- moved R211 13.9 mm to (111.1, 104.1), turned to 180 degrees
- moved D410 12.7 mm to (170.8, 104.1)
- moved D211 12.7 mm to (120.0, 104.1)
- moved D310 12.7 mm to (145.4, 104.1)
- moved D510 12.7 mm to (196.2, 104.1)
- moved D610 12.7 mm to (221.6, 104.1)
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Routing:
- net /Register 0/A0: track 230.6 -> 0.00 mm, vias 1 -> 0
- net /Register 0/A1: track 228.0 -> 0.00 mm, vias 1 -> 0
- net /Register 0/A2: track 225.5 -> 0.00 mm, vias 1 -> 0
- net /Register 0/A3: track 223.0 -> 0.00 mm, vias 1 -> 0
- net /Register 0/A4: track 219.6 -> 0.00 mm, vias 1 -> 0
- net /Register 0/A5: track 218.3 -> 0.00 mm, vias 1 -> 0
- net /Register 0/A6: track 217.0 -> 0.00 mm, vias 1 -> 0
- net /Register 0/A7: track 215.8 -> 0.00 mm, vias 1 -> 0
- net /Register 0/B0: track 194.2 -> 0.00 mm, vias 1 -> 0
- net /Register 0/B1: track 192.9 -> 0.00 mm, vias 1 -> 0
- net /Register 0/B2: track 192.7 -> 0.00 mm, vias 1 -> 0
- net /Register 0/B3: track 190.4 -> 0.00 mm, vias 1 -> 0
- net /Register 0/B4: track 189.1 -> 0.00 mm, vias 1 -> 0
- net /Register 0/B5: track 187.8 -> 0.00 mm, vias 1 -> 0
- net /Register 0/B6: track 186.6 -> 0.00 mm, vias 1 -> 0
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
Commit message: Thinking, scheming, plotting
Parts:
- added J101: ~, BoardEdgeConnectors:TE-5530843-4-Edge, F.Cu at (165.1, 144.9)
- added U1001: 74HC14, Package_SO:SOIC-14_3.9x8.7mm_P1.27mm, F.Cu at (64.8, 40.6)
- moved U1005 5.68 mm to (88.9, 83.8)
- moved U1006 5.24 mm to (88.9, 105.4)
Connections:
- net /Selectors/~{Execute} renamed Net-(U1004-G1)
- U1003 pad 1: /Selectors/R_{C}0 -> /R_{C}0
- U1003 pad 2: /Selectors/R_{C}1 -> /R_{C}1
- U1003 pad 3: /Selectors/R_{C}2 -> /R_{C}2
- U1003 pad 4: /Selectors/~{Active} -> /R_{C}3
- U1003 pad 5: GND -> /Selectors/~{Active}
- U1003 pad 6: unconnected-(U1003-E2-Pad6) -> +5V
- U1005 pad 1: /Selectors/R_{A}0 -> /R_{A}0
- U1005 pad 2: /Selectors/R_{A}1 -> /R_{A}1
- U1005 pad 3: /Selectors/R_{A}2 -> /R_{A}2
- U1005 pad 4: /Selectors/~{Active} -> /R_{A}3
- U1005 pad 5: GND -> /Selectors/~{Active}
- U1006 pad 1: /Selectors/R_{B}0 -> /R_{B}0
- U1006 pad 2: /Selectors/R_{B}1 -> /R_{B}1
- U1006 pad 3: /Selectors/R_{B}2 -> /R_{B}2
- U1006 pad 4: /Selectors/~{Active} -> /R_{B}3
- U1006 pad 5: GND -> /Selectors/~{Active}
- U501 pad 2: /Register 3/C0 -> /Register 0/C0
- U501 pad 3: /Register 3/C1 -> /Register 0/C1
- U501 pad 4: /Register 3/C2 -> /Register 0/C2
- U501 pad 5: /Register 3/C3 -> /Register 0/C3
- U501 pad 6: /Register 3/C4 -> /Register 0/C4
- U501 pad 7: /Register 3/C5 -> /Register 0/C5
- U501 pad 8: /Register 3/C6 -> /Register 0/C6
- U501 pad 9: /Register 3/C7 -> /Register 0/C7
Routing:
- net /Register 0/B4: track 0.00 -> 243.6 mm, vias 0 -> 1
- net /Register 0/B5: track 0.00 -> 241.7 mm, vias 0 -> 1
- net /Register 0/B6: track 0.00 -> 240.4 mm, vias 0 -> 1
- net /Register 0/B7: track 0.00 -> 238.5 mm, vias 0 -> 1
- net /Register 0/A5: track 0.00 -> 233.4 mm, vias 0 -> 1
- net /Register 0/B0: track 0.00 -> 232.8 mm, vias 0 -> 1
- net /Register 0/A0: track 0.00 -> 230.3 mm, vias 0 -> 1
- net /Register 0/A4: track 0.00 -> 230.3 mm, vias 0 -> 1
- net /Register 0/C0: track 185.2 -> 415.2 mm, vias 0 -> 2
- net /Register 0/A1: track 0.00 -> 229.6 mm, vias 0 -> 1
- net /Register 0/A2: track 0.00 -> 228.4 mm, vias 0 -> 1
- net /Register 0/A3: track 0.00 -> 227.7 mm, vias 0 -> 1
- net /Register 0/C1: track 185.2 -> 412.6 mm, vias 0 -> 2
- net /Register 0/A6: track 0.00 -> 227.1 mm, vias 0 -> 1
- net /Register 0/B1: track 0.00 -> 226.5 mm, vias 0 -> 1
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Other:
- board outline added: 64.8 x 8.9 mm

Commit message: Routing, routing, routing
Parts:
- moved J101 23.4 mm to (142.2, 149.9)
Connections:
- J101 pad A10: /R_{B}2 -> /Register 0/A0
- J101 pad A11: /Register 0/B0 -> /Register 0/A2
- J101 pad A12: /Register 0/B2 -> /Register 0/A4
- J101 pad A13: /Register 0/B4 -> /Register 0/A6
- J101 pad A14: /Register 0/B6 -> /Register 0/B0
- J101 pad A15: /R_{C}0 -> /Register 0/B2
- J101 pad A16: /R_{C}2 -> /Register 0/B4
- J101 pad A17: /Register 0/C0 -> /Register 0/B6
- J101 pad A18: /Register 0/C2 -> /Register 0/C0
- J101 pad A19: /Register 0/C4 -> /Register 0/C2
- J101 pad A20: /Register 0/C6 -> /Register 0/C4
- J101 pad A21: unconnected-(J101-PadA21) -> /Register 0/C6
- J101 pad A5: /Register 0/A0 -> /R_{B}0
- J101 pad A6: /Register 0/A2 -> /R_{B}2
- J101 pad A7: /Register 0/A4 -> /R_{C}0
- J101 pad A8: /Register 0/A6 -> /R_{C}2
- J101 pad A9: /R_{B}0 -> unconnected-(J101-PadA9)
- J101 pad B10: /R_{B}3 -> /Register 0/A1
- J101 pad B11: /Register 0/B1 -> /Register 0/A3
- J101 pad B12: /Register 0/B3 -> /Register 0/A5
- J101 pad B13: /Register 0/B5 -> /Register 0/A7
- J101 pad B14: /Register 0/B7 -> /Register 0/B1
- J101 pad B15: /R_{C}1 -> /Register 0/B3
- J101 pad B16: /R_{C}3 -> /Register 0/B5
- J101 pad B17: /Register 0/C1 -> /Register 0/B7
- J101 pad B18: /Register 0/C3 -> /Register 0/C1
- J101 pad B19: /Register 0/C5 -> /Register 0/C3
- J101 pad B20: /Register 0/C7 -> /Register 0/C5
- J101 pad B21: unconnected-(J101-PadB21) -> /Register 0/C7
- J101 pad B5: /Register 0/A1 -> /R_{B}1
- J101 pad B6: /Register 0/A3 -> /R_{B}3
- J101 pad B7: /Register 0/A5 -> /R_{C}1
- J101 pad B8: /Register 0/A7 -> /R_{C}3
- J101 pad B9: /R_{B}1 -> unconnected-(J101-PadB9)
Routing:
- net /Register 0/C1: track 412.6 -> 277.1 mm
- net /Register 0/C2: track 410.1 -> 275.9 mm
- net /Register 0/C3: track 407.6 -> 274.6 mm
- net /Register 0/C4: track 405.0 -> 273.3 mm, vias 2 -> 1
- net /Register 0/C5: track 402.5 -> 272.1 mm, vias 2 -> 1
- net /Register 0/C6: track 399.9 -> 270.8 mm, vias 2 -> 1
- net /Register 0/C7: track 397.4 -> 269.5 mm, vias 2 -> 1
- net /R_{B}3: track 149.1 -> 42.8 mm
- net /R_{C}3: track 200.6 -> 105.7 mm
- net /R_{B}1: track 156.7 -> 62.5 mm
- net /R_{B}2: track 152.9 -> 59.3 mm
- net /R_{C}2: track 198.6 -> 105.7 mm
- net /R_{B}0: track 160.5 -> 67.6 mm
- net /R_{C}1: track 201.2 -> 110.1 mm
- net /R_{C}0: track 203.7 -> 114.6 mm
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- added copper zone on B.Cu, net +5V
- added copper zone on F.Cu, net GND
Other:
- board size 64.8 x 8.9 mm -> 269.2 x 116.8 mm

Commit message: Routing.... first draft?
Parts:
- moved J101 16.5 mm to (142.2, 133.3)
- moved U1005 3.81 mm to (88.9, 87.6)
- moved U1006 3.81 mm to (88.9, 109.2)
Connections:
- J101 pad A1: /Selectors/CLK -> unconnected-(J101-PadA1)
- J101 pad A2: /Selectors/~{Active} -> /R_{C}0
- J101 pad A3: /R_{A}0 -> /R_{C}2
- J101 pad A4: /R_{A}2 -> /Selectors/~{Active}
- J101 pad A7: /R_{C}0 -> /R_{A}0
- J101 pad A8: /R_{C}2 -> /R_{A}2
- J101 pad B2: unconnected-(J101-PadB2) -> /R_{C}1
- J101 pad B3: /R_{A}1 -> /R_{C}3
- J101 pad B4: /R_{A}3 -> /Selectors/CLK
- J101 pad B7: /R_{C}1 -> /R_{A}1
- J101 pad B8: /R_{C}3 -> /R_{A}3
Routing:
- net +5V: track 0.00 -> 196.0 mm, vias 0 -> 33
- net /Register 0/C7: track 269.5 -> 408.4 mm
- net /Register 0/C6: track 270.8 -> 408.4 mm, vias 1 -> 2
- net /Register 0/C0: track 434.8 -> 334.4 mm, vias 2 -> 1
- net /Register 0/C4: track 273.3 -> 369.4 mm
- net /Register 0/C5: track 272.1 -> 366.8 mm, vias 1 -> 0
- net /Register 0/C2: track 275.9 -> 351.6 mm, vias 2 -> 1
- net /Register 0/C3: track 274.6 -> 349.0 mm, vias 2 -> 0
- net /Register 0/C1: track 277.1 -> 331.3 mm, vias 2 -> 0
- net /R_{C}0: track 114.6 -> 154.2 mm
- net /R_{C}2: track 105.7 -> 141.5 mm
- net /R_{B}3: track 42.8 -> 77.2 mm, vias 2 -> 0
- net /R_{C}1: track 110.1 -> 142.8 mm, vias 1 -> 0
- net /R_{C}3: track 105.7 -> 137.7 mm, vias 1 -> 0
- net /R_{A}3: track 80.3 -> 103.8 mm, vias 2 -> 0
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Other:
- board size 269.2 x 116.8 mm -> 254 x 101.6 mm
- board text added: "RGE2024"
- board text added: "Register File"

Commit message: Deal with islands
Routing:
- net GND: track 5.61 -> 163.0 mm, vias 0 -> 49
Other:
- board text added: "JLCJLCJLCJLC"
