File: pcbs/Register File/Register File.kicad_sch (KiCad schematic)
At the start: 1 part

Commit message: Roughing out some layout
Other:
- sheet Selectors ports: added CW[0..7], R_{A}[0..2], R_{B}[0..2], R_{C}[0..2], ~{AS}[0..7], ~{BS}[0..7]; removed none

Commit message: Lots of thinking and routing
Other:
- moved on the sheet: J101

Commit message: Thinking, scheming, plotting
Parts:
- J101: footprint (none) -> BoardEdgeConnectors:TE-5530843-4-Edge
Connections:
- net Selectors/CLK: now reaches J101.A1
- net R_{B}2: now reaches J101.A10
- net B0: now reaches J101.A11
- net B2: now reaches J101.A12
- net B4: now reaches J101.A13
- net B6: now reaches J101.A14
- net R_{C}0: now reaches J101.A15
- net R_{C}2: now reaches J101.A16
- net C0: now reaches J101.A17
- net C2: now reaches J101.A18
- net C4: now reaches J101.A19
- net Selectors/~{Active}: now reaches J101.A2
- net C6: now reaches J101.A20
- net R_{A}0: now reaches J101.A3
- net R_{A}2: now reaches J101.A4
- net A0: now reaches J101.A5
- net A2: now reaches J101.A6
- net A4: now reaches J101.A7
- net A6: now reaches J101.A8
- net R_{B}0: now reaches J101.A9
- net R_{B}3: now reaches J101.B10
- net B1: now reaches J101.B11
- net B3: now reaches J101.B12
- net B5: now reaches J101.B13
- net B7: now reaches J101.B14
- net R_{C}1: now reaches J101.B15
- net R_{C}3: now reaches J101.B16
- net C1: now reaches J101.B17
- net C3: now reaches J101.B18
- net C5: now reaches J101.B19
- net C7: now reaches J101.B20
- net R_{A}1: now reaches J101.B3
- net R_{A}3: now reaches J101.B4
- net A1: now reaches J101.B5
- net A3: now reaches J101.B6
- net A5: now reaches J101.B7
- net A7: now reaches J101.B8
- net R_{B}1: now reaches J101.B9
- no-connect marks 0 -> 4
Other:
- sheet Selectors ports: added CLK, R_{A}[0..3], R_{B}[0..3], R_{C}[0..3], ~{Active}; removed R_{A}[0..2], R_{B}[0..2], R_{C}[0..2]

Commit message: Routing, routing, routing
Connections:
- net A0: now also J101.A10; no longer J101.A5
- net A1: now also J101.B10; no longer J101.B5
- net A2: now also J101.A11; no longer J101.A6
- net A3: now also J101.B11; no longer J101.B6
- net A4: now also J101.A12; no longer J101.A7
- net A5: now also J101.B12; no longer J101.B7
- net A6: now also J101.A13; no longer J101.A8
- net A7: now also J101.B13; no longer J101.B8
- net B0: now also J101.A14; no longer J101.A11
- net B1: now also J101.B14; no longer J101.B11
- net B2: now also J101.A15; no longer J101.A12
- net B3: now also J101.B15; no longer J101.B12
- net B4: now also J101.A16; no longer J101.A13
- net B5: now also J101.B16; no longer J101.B13
- net B6: now also J101.A17; no longer J101.A14
- net B7: now also J101.B17; no longer J101.B14
- net C0: now also J101.A18; no longer J101.A17
- net C1: now also J101.B18; no longer J101.B17
- net C2: now also J101.A19; no longer J101.A18
- net C3: now also J101.B19; no longer J101.B18
- net C4: now also J101.A20; no longer J101.A19
- net C5: now also J101.B20; no longer J101.B19
- net C6: now also J101.A21; no longer J101.A20
- net C7: now also J101.B21; no longer J101.B20
- net R_{B}0: now also J101.A5; no longer J101.A9
- net R_{B}1: now also J101.B5; no longer J101.B9
- net R_{B}2: now also J101.A6; no longer J101.A10
- net R_{B}3: now also J101.B6; no longer J101.B10
- net R_{C}0: now also J101.A7; no longer J101.A15
- net R_{C}1: now also J101.B7; no longer J101.B15
- net R_{C}2: now also J101.A8; no longer J101.A16
- net R_{C}3: now also J101.B8; no longer J101.B16

Commit message: Routing.... first draft?
Connections:
- net R_{A}0: now also J101.A7; no longer J101.A3
- net R_{A}1: now also J101.B7; no longer J101.B3
- net R_{A}2: now also J101.A8; no longer J101.A4
- net R_{A}3: now also J101.B8; no longer J101.B4
- net R_{C}0: now also J101.A2; no longer J101.A7
- net R_{C}1: now also J101.B2; no longer J101.B7
- net R_{C}2: now also J101.A3; no longer J101.A8
- net R_{C}3: now also J101.B3; no longer J101.B8
- net Selectors/CLK: now also J101.B4; no longer J101.A1
- net Selectors/~{Active}: now also J101.A4; no longer J101.A2

Commit message: Working on exclude from BOM etc.
Parts:
- J101: now left out of the parts list
Changed lines of the file:
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@@
 		(unit 1)
 		(exclude_from_sim no)
-		(in_bom yes)
+		(in_bom no)
 		(on_board yes)
 		(dnp no)
