File: pcbs/Register File/selectors.kicad_sch (KiCad schematic)
At the start: 30 parts, among them U1003 74HC138, U1004 74HC540, U1005 74HC138, U1006 74HC138

Commit message: Roughing out some layout
Connections:
- net C_{Write}0 renamed CW0
- net C_{Write}1 renamed CW1
- net C_{Write}2 renamed CW2
- net C_{Write}3 renamed CW3
- net C_{Write}4 renamed CW4
- net C_{Write}5 renamed CW5
- net C_{Write}6 renamed CW6
- net C_{Write}7 renamed CW7
- net ~{A_{select}}0 renamed ~{AS}0
- net ~{A_{select}}1 renamed ~{AS}1
- net ~{A_{select}}2 renamed ~{AS}2
- net ~{A_{select}}3 renamed ~{AS}3
- net ~{A_{select}}4 renamed ~{AS}4
- net ~{A_{select}}5 renamed ~{AS}5
- net ~{A_{select}}6 renamed ~{AS}6
- net ~{A_{select}}7 renamed ~{AS}7
- net ~{B_{select}}0 renamed ~{BS}0
- net ~{B_{select}}1 renamed ~{BS}1
- net ~{B_{select}}2 renamed ~{BS}2
- net ~{B_{select}}3 renamed ~{BS}3
- net ~{B_{select}}4 renamed ~{BS}4
- net ~{B_{select}}5 renamed ~{BS}5
- net ~{B_{select}}6 renamed ~{BS}6
- net ~{B_{select}}7 renamed ~{BS}7
Changed lines of the file:
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@@
 		)
 	)
-	(label "~{B_{select}}1"
+	(label "~{AS}2"
+		(at 242.57 39.37 0)
+		(fields_autoplaced yes)
+		(effects
+			(font
+				(size 1.27 1.27)
+			)
+			(justify left bottom)
+		)
+	)
+	(label "~{BS}1"
 		(at 242.57 86.36 0)
 		(fields_autoplaced yes)
@@
 		)
 	)
-	(label "~{B_{select}}2"
+	(label "~{BS}2"
 		(at 242.57 88.9 0)
 		(fields_autoplaced yes)
@@
 		)
 	)
-	(label "C_{Write}7"
+	(label "CW7"
 		(at 116.84 86.36 0)
 		(fields_autoplaced yes)
@@
 		)
 	)
+	(label "~{AS}1"
+		(at 242.57 36.83 0)
+		(fields_autoplaced yes)
+		(effects
+			(font
+				(size 1.27 1.27)
+			)
+			(justify left bottom)
+		)
+	)
 	(label "R_{B}2"
 		(at 212.09 88.9 0)
@@
 		)
 	)
-	(label "C_{Write}0"
+	(label "CW0"
 		(at 116.84 68.58 0)
 		(fields_autoplaced yes)
@@
 		)
 	)
+	(label "~{AS}3"
+		(at 242.57 41.91 0)
+		(fields_autoplaced yes)
+		(effects
+			(font
+				(size 1.27 1.27)
+			)
+			(justify left bottom)
+		)
+	)
 	(label "W1"
 		(at 181.61 82.55 0)
@@
 		)
 	)
-	(label "C_{Write}2"
+	(label "CW2"
 		(at 116.84 73.66 0)
 		(fields_autoplaced yes)
@@
 		)
 	)
-	(label "C_{Write}3"
+	(label "CW3"
 		(at 116.84 76.2 0)
 		(fields_autoplaced yes)
@@
 		)
 	)
-	(label "~{A_{select}}7"
-		(at 242.57 52.07 0)
-		(fields_autoplaced yes)
-		(effects
-			(font
-				(size 1.27 1.27)
-			)
-			(justify left bottom)
-		)
-	)
-	(label "C_{Write}6"
+	(label "CW6"
 		(at 116.84 83.82 0)
 		(fields_autoplaced yes)
@@
 		)
 	)
-	(label "~{A_{select}}3"
-		(at 242.57 41.91 0)
-		(fields_autoplaced yes)
-		(effects
-			(font
-				(size 1.27 1.27)
-			)
-			(justify left bottom)
-		)
-	)
-	(label "~{B_{select}}5"
+	(label "~{BS}5"
 		(at 242.57 96.52 0)
 		(fields_autoplaced yes)
@@
 		)
 	)
-	(label "~{B_{select}}3"
+	(label "~{BS}3"
 		(at 242.57 91.44 0)
 		(fields_autoplaced yes)
@@
 		)
 	)
-	(label "~{B_{select}}7"
+	(label "~{BS}7"
 		(at 242.57 101.6 0)
-		(fields_autoplaced yes)
-		(effects
-			(font
-				(size 1.27 1.27)
-			)
-			(justify left bottom)
-		)
-	)
-	(label "~{A_{select}}4"
-		(at 242.57 44.45 0)
 		(fields_autoplaced yes)
 		(effects
@@
 		)
 	)
-	(label "~{A_{select}}2"
-		(at 242.57 39.37 0)
-		(fields_autoplaced yes)
-		(effects
-			(font
-				(size 1.27 1.27)
-			)
-			(justify left bottom)
-		)
-	)
-	(label "~{B_{select}}0"
+	(label "~{AS}5"
+		(at 242.57 46.99 0)
+		(fields_autoplaced yes)
+		(effects
+			(font
+				(size 1.27 1.27)
+			)
+			(justify left bottom)
+		)
+	)
+	(label "~{BS}0"
 		(at 242.57 83.82 0)
 		(fields_autoplaced yes)
@@
 		)
 	)
-	(label "C_{Write}5"
+	(label "CW5"
 		(at 116.84 81.28 0)
 		(fields_autoplaced yes)
@@
 		)
 	)
-	(label "~{B_{select}}6"
+	(label "~{BS}6"
 		(at 242.57 99.06 0)
 		(fields_autoplaced yes)
@@
 		)
 	)
-	(label "~{A_{select}}0"
+	(label "~{AS}0"
 		(at 242.57 34.29 0)
 		(fields_autoplaced yes)
@@
 		)
 	)
-	(label "C_{Write}4"
+	(label "CW4"
 		(at 116.84 78.74 0)
 		(fields_autoplaced yes)
@@
 		)
 	)
-	(label "~{B_{select}}4"
+	(label "~{BS}4"
 		(at 242.57 93.98 0)
 		(fields_autoplaced yes)
@@
 		)
 	)
-	(label "C_{Write}1"
+	(label "CW1"
 		(at 116.84 71.12 0)
 		(fields_autoplaced yes)
@@
 		)
 	)
-	(label "~{A_{select}}6"
-		(at 242.57 49.53 0)
+	(label "~{AS}7"
+		(at 242.57 52.07 0)
 		(fields_autoplaced yes)
 		(effects
@@
 		)
 	)
-	(label "~{A_{select}}5"
-		(at 242.57 46.99 0)
-		(fields_autoplaced yes)
-		(effects
-			(font
-				(size 1.27 1.27)
-			)
-			(justify left bottom)
-		)
-	)
 	(label "R_{A}2"
 		(at 212.09 39.37 0)
@@
 		)
 	)
+	(label "~{AS}4"
+		(at 242.57 44.45 0)
+		(fields_autoplaced yes)
+		(effects
+			(font
+				(size 1.27 1.27)
+			)
+			(justify left bottom)
+		)
+	)
 	(label "W7"
 		(at 81.28 86.36 0)
@@
 		)
 	)
+	(label "~{AS}6"
+		(at 242.57 49.53 0)
+		(fields_autoplaced yes)
+		(effects
+			(font
+				(size 1.27 1.27)
+			)
+			(justify left bottom)
+		)
+	)
 	(label "W4"
 		(at 81.28 78.74 0)
-		(fields_autoplaced yes)
-		(effects
-			(font
-				(size 1.27 1.27)
-			)
-			(justify left bottom)
-		)
-	)
-	(label "~{A_{select}}1"
-		(at 242.57 36.83 0)
 		(fields_autoplaced yes)
 		(effects
@@
 		)
 	)
-	(hierarchical_label "~{B_{select}}[0..7]"
+	(hierarchical_label "~{BS}[0..7]"
 		(shape output)
 		(at 270.51 80.01 0)
@@
 		)
 	)
-	(hierarchical_label "~{A_{select}}[0..7]"
+	(hierarchical_label "~{AS}[0..7]"
 		(shape output)
 		(at 270.51 30.48 0)
@@
 		)
 	)
-	(hierarchical_label "C_{Write}[0..7]"
+	(hierarchical_label "CW[0..7]"
 		(shape output)
 		(at 157.48 59.69 0)

Commit message: Thinking, scheming, plotting
Parts:
- added U1001: 74HC14, Package_SO:SOIC-14_3.9x8.7mm_P1.27mm, symbol 74xx:74HC14
Connections:
- net +5V: now also U1003.6 (E2), U1001.14 (VCC)
- net GND: now also U1001.1, U1001.11, U1001.3, U1001.5, U1001.7 (GND), U1001.9; no longer U1003.5 (~{E1}), U1005.5 (~{E1}), U1006.5 (~{E1})
- net ~{Active}: now also U1003.5 (~{E1}), U1005.5 (~{E1}), U1006.5 (~{E1}); no longer U1003.4 (~{E0}), U1005.4 (~{E0}), U1006.4 (~{E0})
- net ~{Execute}: no longer names the net of U1004.1 (G1), U1004.19 (G2)
- net ~{Execute}: now also U1001.12
- new net CLK: U1001.13
- new net R_{A}3: U1005.4 (~{E0})
- new net R_{B}3: U1006.4 (~{E0})
- new net R_{C}3: U1003.4 (~{E0})
- no-connect marks 0 -> 5

Commit message: Working on exclude from BOM etc.
Parts:
- U1003, U1005, U1006: now left out of the parts list
Changed lines of the file:
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@@
 	)
 	(symbol
-		(lib_name "GND_2")
 		(lib_id "power:GND")
 		(at 107.95 189.23 0)
@@
 			)
 		)
-		(property "Description" ""
+		(property "Description" "Power symbol creates a global label with name \"+5V\""
 			(at 215.9 105.41 0)
 			(effects
@@
 			)
 		)
-		(property "Description" ""
+		(property "Description" "Power symbol creates a global label with name \"GND\" , ground"
 			(at 104.14 106.68 0)
 			(effects
@@
 			)
 		)
-		(property "Description" ""
+		(property "Description" "Power symbol creates a global label with name \"+5V\""
 			(at 104.14 57.15 0)
 			(effects
@@
 			)
 		)
-		(property "Description" ""
+		(property "Description" "Power symbol creates a global label with name \"GND\" , ground"
 			(at 232.41 62.23 0)
 			(effects
@@
 	)
 	(symbol
-		(lib_name "+5V_2")
 		(lib_id "power:+5V")
 		(at 48.26 148.59 0)
@@
 			)
 		)
-		(property "Description" ""
+		(property "Description" "Power symbol creates a global label with name \"GND\" , ground"
 			(at 232.41 111.76 0)
 			(effects
@@
 			)
 		)
-		(property "Description" ""
+		(property "Description" "Power symbol creates a global label with name \"GND\" , ground"
 			(at 64.77 96.52 0)
 			(effects
@@
 			)
 		)
-		(property "Description" ""
+		(property "Description" "Power symbol creates a global label with name \"GND\" , ground"
 			(at 34.29 39.37 0)
 			(effects
@@
 			)
 		)
-		(property "Description" ""
+		(property "Description" "Power symbol creates a global label with name \"GND\" , ground"
 			(at 125.73 26.67 0)
 			(effects
@@
 			)
 		)
-		(property "Description" ""
+		(property "Description" "Power symbol creates a global label with name \"+5V\""
 			(at 215.9 55.88 0)
 			(effects
@@
 			)
 		)
-		(property "Description" ""
+		(property "Description" "Power symbol creates a global label with name \"+5V\""
 			(at 34.29 26.67 0)
 			(effects
@@
 		(unit 1)
 		(exclude_from_sim no)
-		(in_bom yes)
+		(in_bom no)
 		(on_board yes)
 		(dnp no)
@@
 			)
 		)
-		(property "Description" ""
+		(property "Description" "Power symbol creates a global label with name \"+5V\""
 			(at 232.41 25.4 0)
 			(effects
@@
 		(unit 1)
 		(exclude_from_sim no)
-		(in_bom yes)
+		(in_bom no)
 		(on_board yes)
 		(dnp no)
@@
 			)
 		)
-		(property "Description" ""
+		(property "Description" "Power symbol creates a global label with name \"+5V\""
 			(at 232.41 74.93 0)
 			(effects
@@
 	)
 	(symbol
-		(lib_name "GND_1")
 		(lib_id "power:GND")
 		(at 48.26 179.07 0)
@@
 	)
 	(symbol
-		(lib_name "+5V_1")
 		(lib_id "power:+5V")
 		(at 49.53 86.36 90)
@@
 			)
 		)
-		(property "Description" ""
+		(property "Description" "Power symbol creates a global label with name \"+5V\""
 			(at 64.77 59.69 0)
 			(effects
@@
 			)
 		)
-		(property "Description" ""
+		(property "Description" "Power symbol creates a global label with name \"+5V\""
 			(at 146.05 68.58 0)
 			(effects
@@
 		(unit 1)
 		(exclude_from_sim no)
-		(in_bom yes)
+		(in_bom no)
 		(on_board yes)
 		(dnp no)

Commit message: Minor fixes
Parts:
- U1001: LCSC (none) -> C5605
Changed lines of the file:
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@@
 			)
 		)
+		(property "LCSC" "C5605"
+			(at 120.65 140.97 0)
+			(effects
+				(font
+					(size 1.27 1.27)
+				)
+				(hide yes)
+			)
+		)
 		(pin "4"
 		)
@@
 			)
 		)
+		(property "LCSC" "C5605"
+			(at 120.65 127 0)
+			(effects
+				(font
+					(size 1.27 1.27)
+				)
+				(hide yes)
+			)
+		)
 		(pin "4"
 		)
@@
 			)
 		)
+		(property "LCSC" "C5605"
+			(at 120.65 170.18 0)
+			(effects
+				(font
+					(size 1.27 1.27)
+				)
+				(hide yes)
+			)
+		)
 		(pin "4"
 		)
@@
 			)
 		)
+		(property "LCSC" "C5605"
+			(at 120.65 185.42 0)
+			(effects
+				(font
+					(size 1.27 1.27)
+				)
+				(hide yes)
+			)
+		)
 		(pin "4"
 		)
@@
 			)
 		)
+		(property "LCSC" "C5605"
+			(at 120.65 154.94 0)
+			(effects
+				(font
+					(size 1.27 1.27)
+				)
+				(hide yes)
+			)
+		)
 		(pin "4"
 		)
@@
 			)
 		)
+		(property "LCSC" "C5605"
+			(at 68.58 120.65 0)
+			(effects
+				(font
+					(size 1.27 1.27)
+				)
+				(hide yes)
+			)
+		)
 		(pin "4"
 		)
@@
 			(at 48.26 163.83 0)
 			(effects
+				(font
+					(size 1.27 1.27)
+				)
+				(hide yes)
+			)
+		)
+		(property "LCSC" "C5605"
+			(at 48.26 163.83 0)
+			(effects
