File: pcbs/Adder Subtractor/Adder Subtractor.kicad_sch (KiCad schematic)
At the start: 5 parts, among them U1 74HC86, U2 74HC86, U3 74HC283, U4 74HC283

Commit message: Add output buffer
Parts:
- added U5: 74HC245, Package_SO:SOIC-20W_7.5x12.8mm_P1.27mm, symbol 74xx:74HC245
- added U6: 74HC08, Package_SO:SOIC-14_3.9x8.7mm_P1.27mm, symbol 74xx:74LS08
Connections:
- net +5V: now also U5.20 (VCC), U6.14 (VCC)
- net GND: now also U5.1 (A->B), U5.10 (GND), U6.1, U6.10, U6.2, U6.4, U6.5, U6.7 (GND), U6.9
- net Out0: now also U5.18 (B0); no longer J1.A16
- net Out1: now also U5.17 (B1); no longer J1.B16
- net Out2: now also U5.16 (B2); no longer J1.A17
- net Out3: now also U5.15 (B3); no longer J1.B17
- net Out4: now also U5.14 (B4); no longer J1.A18
- net Out5: now also U5.13 (B5); no longer J1.B18
- net Out6: now also U5.12 (B6); no longer J1.A19
- net Out7: now also U5.11 (B7); no longer J1.B19
- net ~{Sub}: now reaches J1.B2
- net ~{Sub}: now also U6.13
- net ~{Add}/Sub renamed ~{Add}
- net ~{Add}: now also U6.12
- new net C0: J1.A16, U5.2 (A0)
- new net C1: J1.B16, U5.3 (A1)
- new net C2: J1.A17, U5.4 (A2)
- new net C3: J1.B17, U5.5 (A3)
- new net C4: J1.A18, U5.6 (A4)
- new net C5: J1.B18, U5.7 (A5)
- new net C6: J1.A19, U5.8 (A6)
- new net C7: J1.B19, U5.9 (A7)
- new net ~{Enable}: U5.19 (CE), U6.11
- no-connect marks 15 -> 17

Commit message: Indicator LEDs
Parts:
- added D1, D2: Blue, LED_SMD:LED_0603_1608Metric, symbol Device:LED
- added R1, R2: 4k7, Resistor_SMD:R_0603_1608Metric, symbol Device:R
Connections:
- net +5V: now also R1.2, R2.2
- net ~{Add}: now also D1.1 (K)
- net ~{Sub}: now also D2.1 (K)
- new net: D2.2 (A), R2.1
- new net: D1.2 (A), R1.1

Commit message: Capacitors for Adder/Subtractor
Parts:
- added C1, C2: C, Capacitor_SMD:C_0603_1608Metric, symbol Device:C
Connections:
- net +5V: now also C1.1, C2.1
- net GND: now also C1.2, C2.2
