File: pcbs/Comparator/Comparator.kicad_pcb (KiCad board)
At the start: 2 copper layers, 8.9 x 64.8 mm, 12 parts, among them U1 74HC85, U2 74HC85, U3 74HC85, U4 74HC85, U5 74HC245

Commit message: Finish routing draft
Parts:
- moved J1 12.7 mm to (50.8, 94.0)
- moved D1 7.34 mm to (100.3, 58.4), turned to 180 degrees
- moved R1 4.09 mm to (100.3, 56.5)
Connections:
- U5 pad 16: /Out_{A=B} -> /Out_{A>B}
- U5 pad 17: /Out_{A<B} -> /Out_{A=B}
- U5 pad 18: /Out_{A>B} -> /Out_{A<B}
Routing:
- net /~{Enable}: track 0.00 -> 177.6 mm, vias 0 -> 3
- net /C1: track 0.00 -> 44.3 mm, vias 0 -> 1
- net /C2: track 0.00 -> 43.4 mm
- net /C0: track 0.00 -> 43.4 mm
- net GND: track 0.00 -> 36.1 mm, vias 0 -> 13
- net /Out_{A>B}: track 0.00 -> 29.0 mm, vias 0 -> 2
- net /Out_{A=B}: track 0.00 -> 25.2 mm, vias 0 -> 2
- net /Out_{A<B}: track 0.00 -> 21.4 mm, vias 0 -> 2
- net +5V: track 12.1 -> 32.6 mm, vias 0 -> 7
- net /A7: track 78.0 -> 87.7 mm, vias 3 -> 4
- net /A3: track 60.6 -> 70.3 mm, vias 3 -> 4
- net /A1: track 68.2 -> 77.9 mm, vias 3 -> 4
- net /A5: track 86.0 -> 95.7 mm, vias 3 -> 4
- net /A6: track 83.4 -> 92.2 mm
- net /A4: track 91.1 -> 99.9 mm
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- added copper zone on B.Cu, net +5V
- added copper zone on F.Cu, net GND
Other:
- board size 8.9 x 64.8 mm -> 50.8 x 104.1 mm
- board text added: "Comparator"
- board text added: "JLCJLCJLCJLC"
- board text added: "RGE2024"
