File: pcbs/Comparator/Comparator.kicad_sch (KiCad schematic)
At the start: 6 parts, among them U1 74HC245, U2 74HC85, U3 74HC85, U4 74HC85, U5 74HC85

Commit message: Starting routing
Parts:
- added C1, C2, C3, C4: C, Capacitor_SMD:C_0603_1608Metric, symbol Device:C
- added D1: Blue, LED_SMD:LED_0603_1608Metric, symbol Device:LED
- added R1: 4k7, Resistor_SMD:R_0603_1608Metric, symbol Device:R
- renumbered U2 to U1, U3 to U2, U4 to U3, U5 to U4, U1 to U5
Connections:
- net +5V: now also C1.1, C2.1, C3.1, C4.1, R1.2
- net B5: now also J1.B13
- net GND: now also C1.2, C2.2, C3.2, C4.2
- net ~{Enable}: now also D1.1 (K)
- new net: D1.2 (A), R1.1

Commit message: Finish routing draft
Connections:
- net Out_{A<B}: now also U5.18 (B0); no longer U5.17 (B1)
- net Out_{A=B}: now also U5.17 (B1); no longer U5.16 (B2)
- net Out_{A>B}: now also U5.16 (B2); no longer U5.18 (B0)
Changed lines of the file:
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@@
 	)
 	(label "Out_{A<B}"
-		(at 269.24 96.52 0)
+		(at 269.24 93.98 0)
 		(fields_autoplaced yes)
 		(effects
@@
 	)
 	(label "Out_{A=B}"
-		(at 269.24 99.06 0)
+		(at 269.24 96.52 0)
 		(fields_autoplaced yes)
 		(effects
@@
 	)
 	(label "Out_{A>B}"
-		(at 269.24 93.98 0)
-		(fields_autoplaced yes)
-		(effects
+		(at 269.24 99.06 0)
+		(fields_autoplaced yes)
+		(effects

Commit message: XOR/NAND board
Parts:
- J1, U1, U2, U3, U4: now left out of the parts list
Changed lines of the file:
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@@
 		(unit 1)
 		(exclude_from_sim no)
-		(in_bom yes)
+		(in_bom no)
 		(on_board yes)
 		(dnp no)
@@
 		(unit 1)
 		(exclude_from_sim no)
-		(in_bom yes)
+		(in_bom no)
 		(on_board yes)
 		(dnp no)
@@
 		(unit 1)
 		(exclude_from_sim no)
-		(in_bom yes)
+		(in_bom no)
 		(on_board yes)
 		(dnp no)
@@
 		(unit 1)
 		(exclude_from_sim no)
-		(in_bom yes)
+		(in_bom no)
 		(on_board yes)
 		(dnp no)
@@
 		(unit 1)
 		(exclude_from_sim no)
-		(in_bom yes)
-		(on_board yes)
-		(dnp no)
+		(in_bom no)
+		(on_board yes)
+		(dnp no)
