File: pcbs/Pi Backplane Connector/inputs.kicad_sch (KiCad schematic)
At the start: 10 parts, among them U4001 74HC165, U4002 74HC165, U4003 74HC165, U4004 74HC165, U4005 74HC165, U4006 74HC165, U4007 74HC165, U4008 74HC165, U4009 74HC165, U4010 74HC165

Commit message: Trying to figure out some routing. Not much success
Connections:
- net In_{0}: no longer names the net of U4009.11 (D0)
- net In_{0}: no longer U4010.11 (D0)
- net In_{10}: no longer names the net of U4008.13 (D2)
- net In_{11}: no longer names the net of U4008.14 (D3)
- net In_{12}: no longer names the net of U4008.3 (D4)
- net In_{13}: no longer names the net of U4008.4 (D5)
- net In_{14}: no longer names the net of U4008.5 (D6)
- net In_{15}: no longer names the net of U4008.6 (D7)
- net In_{16}: no longer names the net of U4007.11 (D0)
- net In_{17}: no longer names the net of U4007.12 (D1)
- net In_{18}: no longer names the net of U4007.13 (D2)
- net In_{19}: no longer names the net of U4007.14 (D3)
- net In_{1}: no longer names the net of U4009.12 (D1)
- net In_{1}: no longer U4010.12 (D1)
- net In_{20}: no longer names the net of U4007.3 (D4)
- net In_{21}: no longer names the net of U4007.4 (D5)
- net In_{22}: no longer names the net of U4007.5 (D6)
- net In_{23}: no longer names the net of U4007.6 (D7)
- net In_{2}: no longer names the net of U4009.13 (D2)
- net In_{2}: no longer U4010.13 (D2)
- net In_{3}: no longer names the net of U4009.14 (D3)
- net In_{3}: no longer U4010.14 (D3)
- net In_{4}: no longer names the net of U4009.3 (D4)
- net In_{4}: no longer U4010.3 (D4)
- net In_{5}: no longer names the net of U4009.4 (D5)
- net In_{5}: no longer U4010.4 (D5)
- net In_{6}: no longer names the net of U4009.5 (D6)
- net In_{6}: no longer U4010.5 (D6)
- net In_{7}: no longer names the net of U4009.6 (D7)
- net In_{7}: no longer U4010.6 (D7)
- net In_{8}: no longer names the net of U4008.11 (D0)
- net In_{9}: no longer names the net of U4008.12 (D1)
Other:
- moved on the sheet: U4001

Commit message: Some routing
Connections:
- net I0: now reaches U4009.11 (D0)
- net I1: now reaches U4009.12 (D1)
- net I2: now reaches U4009.13 (D2)
- net I3: now reaches U4009.14 (D3)
- net I4: now reaches U4009.3 (D4)
- net I5: now reaches U4009.4 (D5)
- net I6: now reaches U4009.5 (D6)
- net I7: now reaches U4009.6 (D7)
- net C8: now reaches U4008.11 (D0)
- net C9: now reaches U4008.12 (D1)
- net C10: now reaches U4008.13 (D2)
- net C11: now reaches U4008.14 (D3)
- net C12: now reaches U4008.3 (D4)
- net C13: now reaches U4008.4 (D5)
- net C14: now reaches U4008.5 (D6)
- net C15: now reaches U4008.6 (D7)
- net B8: now reaches U4006.11 (D0)
- net B9: now reaches U4006.12 (D1)
- net B10: now reaches U4006.13 (D2)
- net B11: now reaches U4006.14 (D3)
- net B12: now reaches U4006.3 (D4)
- net B13: now reaches U4006.4 (D5)
- net B14: now reaches U4006.5 (D6)
- net B15: now reaches U4006.6 (D7)
- net I8: now reaches U4010.11 (D0)
- net I9: now reaches U4010.12 (D1)
- net I10: now reaches U4010.13 (D2)
- net I11: now reaches U4010.14 (D3)
- net I12: now reaches U4010.3 (D4)
- net I13: now reaches U4010.4 (D5)
- net I14: now reaches U4010.5 (D6)
- net I15: now reaches U4010.6 (D7)
- net B0: now reaches U4005.11 (D0)
- net B1: now reaches U4005.12 (D1)
- net B2: now reaches U4005.13 (D2)
- net B3: now reaches U4005.14 (D3)
- net B4: now reaches U4005.3 (D4)
- net B5: now reaches U4005.4 (D5)
- net B6: now reaches U4005.5 (D6)
- net B7: now reaches U4005.6 (D7)
- net C0: now reaches U4007.11 (D0)
- net C1: now reaches U4007.12 (D1)
- net C2: now reaches U4007.13 (D2)
- net C3: now reaches U4007.14 (D3)
- net C4: now reaches U4007.3 (D4)
- net C5: now reaches U4007.4 (D5)
- net C6: now reaches U4007.5 (D6)
- net C7: now reaches U4007.6 (D7)

Commit message: More connections, more routing
Connections:
- net GND: now also U4002.11 (D0), U4002.12 (D1), U4002.13 (D2)
- net Cycle0: now reaches U4002.14 (D3)
- net Cycle1: now reaches U4002.3 (D4)
- net Cycle2: now reaches U4002.4 (D5)
- net Cycle3: now reaches U4002.5 (D6)
- net Cycle4: now reaches U4002.6 (D7)

Commit message: Connections and capacitors
Parts:
- added C4001, C4002, C4003, C4004, C4005, C4006, C4007, C4008, C4009, C4010: 100n, Capacitor_SMD:C_0603_1608Metric, symbol Device:C
Connections:
- net +5V: now also C4001.2, C4002.2, C4003.2, C4004.2, C4005.2, C4006.2, C4007.2, C4008.2, C4009.2, C4010.2
- net GND: now also U4001.11 (D0), U4001.14 (D3), U4001.3 (D4), U4001.4 (D5), U4001.5 (D6), U4001.6 (D7), C4001.1, C4002.1, C4003.1, C4004.1, C4005.1, C4006.1, C4007.1, C4008.1, C4009.1, C4010.1
- net CLOCK: now reaches U4001.12 (D1)
- net RESET: now reaches U4001.13 (D2)
