File: pcbs/Pi Backplane Connector/outputs.kicad_sch (KiCad schematic)
At the start: 10 parts, among them U3001 74HC595, U3002 74HC595, U3003 74HC595, U3004 74HC595, U3005 74HC595, U3006 74HC595, U3007 74HC595, U3008 74HC595, U3009 74HC595, U3010 74HC595

Commit message: Doing some routing
Connections:
- net +5V: now also U3001.16 (VCC), U3002.16 (VCC)
- net GND: now also U3001.8 (GND), U3002.8 (GND), U3005.8 (GND), U3006.8 (GND), U3007.8 (GND), U3008.8 (GND), U3009.8 (GND), U3010.8 (GND)

Commit message: More connections, more routing
Connections:
- net +5V: now also U3001.10 (~{SRCLR}), U3002.10 (~{SRCLR}), U3003.10 (~{SRCLR}), U3004.10 (~{SRCLR}), U3005.10 (~{SRCLR}), U3006.10 (~{SRCLR}), U3007.10 (~{SRCLR}), U3008.10 (~{SRCLR}), U3009.10 (~{SRCLR}), U3010.10 (~{SRCLR})
- net ~{I_{enable}}: now also U3009.13 (~{OE}), U3010.13 (~{OE})
- net SRCLK: now reaches U3002.11 (SRCLK)
- net SRCLK: now also U3001.11 (SRCLK), U3003.11 (SRCLK), U3004.11 (SRCLK), U3005.11 (SRCLK), U3006.11 (SRCLK), U3007.11 (SRCLK), U3008.11 (SRCLK), U3009.11 (SRCLK), U3010.11 (SRCLK)
- net RCLK: now reaches U3002.12 (RCLK)
- net RCLK: now also U3001.12 (RCLK), U3003.12 (RCLK), U3004.12 (RCLK), U3005.12 (RCLK), U3006.12 (RCLK), U3007.12 (RCLK), U3008.12 (RCLK), U3009.12 (RCLK), U3010.12 (RCLK)
- net ~{Enable_{Cycle}}: now reaches U3002.13 (~{OE})
- net Cycle0: now reaches U3002.3 (QD)
- net Cycle1: now reaches U3002.4 (QE)
- net Cycle2: now reaches U3002.5 (QF)
- net Cycle3: now reaches U3002.6 (QG)
- net Cycle4: now reaches U3002.7 (QH)
- net DATA: now reaches U3001.14 (SER)
- no-connect marks 1 -> 4

Commit message: Connections and capacitors
Parts:
- added C3001, C3002, C3003, C3004, C3005, C3006, C3007, C3008, C3009, C3010: 100n, Capacitor_SMD:C_0603_1608Metric, symbol Device:C
- added U3011: 74AHCT125, Package_DIP:DIP-14_W7.62mm_Socket, symbol 74xx:74AHCT125
Connections:
- net +5V: now also C3001.2, C3002.2, C3003.2, C3004.2, C3005.2, C3006.2, C3007.2, C3008.2, C3009.2, C3010.2, U3011.1, U3011.14 (VCC), U3011.4
- net GND: now also U3001.13 (~{OE}), C3001.1, C3002.1, C3003.1, C3004.1, C3005.1, C3006.1, C3007.1, C3008.1, C3009.1, C3010.1, U3011.2, U3011.5, U3011.7 (GND)
- net RST_{out}: now reaches U3001.1 (QB)
- net RST_{out}: now also U3011.12
- net CLK_{out}: now reaches U3001.2 (QC)
- net CLK_{out}: now also U3011.9
- net ~{Enable_{Cycle}} renamed ~{Cycle_{enable}}
- new net CLOCK: U3011.8
- new net RESET: U3011.11
- new net ~{CLOCK_{enable}}: U3011.10
- new net ~{RESET_{enable}}: U3011.13
- no-connect marks 4 -> 12

Commit message: Starting on the connections...
Parts:
- added R3001, R3002, R3003, R3004, R3005, R3006, R3007: 1M, Resistor_SMD:R_0603_1608Metric, symbol Device:R
Connections:
- net +5V: now also R3001.2, R3002.2, R3003.2, R3004.2, R3005.2, R3006.2, R3007.2
- net ~{A_{enable}}: now also R3002.1
- net ~{B_{enable}}: now also R3003.1
- net ~{CLOCK_{enable}}: now also R3007.1
- net ~{C_{enable}}: now also R3004.1
- net ~{Cycle_{enable}}: now also R3001.1
- net ~{I_{enable}}: now also R3005.1
- net ~{RESET_{enable}}: now also R3006.1
