File: pcbs/Pi Backplane Connector/Pi Backplane Connector.kicad_pcb (KiCad board)
At the start: 2 copper layers, 87 parts, among them J1001 Conn_02x20_Odd_Even, J1002 Conn_02x20_Odd_Even, J2001 Raspberry_Pi_2_3, U3001 74HC595, U3002 74HC595, U3003 74HC595, U3004 74HC595, U3005 74HC595, U3006 74HC595, U3007 74HC595, U3008 74HC595, U3009 74HC595, U3010 74HC595, U4001 74HC165, U4002 74HC165, U4003 74HC165, U4004 74HC165, U4005 74HC165, U4006 74HC165, U4007 74HC165, U4008 74HC165, U4009 74HC165, U4010 74HC165

Commit message: Trying to figure out some routing. Not much success
Routing:
- net /A0: track 0.00 -> 137.7 mm
- net /A7: track 0.00 -> 130.8 mm
- net /A6: track 0.00 -> 130.8 mm
- net /A5: track 0.00 -> 130.8 mm
- net /A4: track 0.00 -> 130.8 mm
- net /A3: track 0.00 -> 130.8 mm
- net /A2: track 0.00 -> 130.8 mm
- net /A1: track 0.00 -> 130.8 mm
Changed lines of the file:
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@@
+	)
+	(gr_line
+		(start 292.1 226.06)
+		(end 161.925 226.06)
+		(stroke
+			(width 0.1)
+			(type default)
+		)
+		(layer "F.SilkS")
 	)
 	(gr_line
@@
 	)
 	(gr_line
+		(start 302.26 226.06)
+		(end 292.1 226.06)
+		(stroke
+			(width 0.1)
+			(type default)
+		)
+		(layer "F.SilkS")
+	)
+	(gr_line
 		(start 318.77 121.92)
 		(end 317.5 121.92)
@@
 		)
 	)
+	(segment
+		(start 180.975 91.475)
+		(end 180.975 222.25)
+		(width 0.127)
+		(layer "F.Cu")
+		(net 18)
+	)
+	(segment
+		(start 183.515 91.475)
+		(end 183.515 95.25)
+		(width 0.127)
+		(layer "F.Cu")
+		(net 27)
+	)
+	(segment
+		(start 183.515 95.25)
+		(end 183.515 222.25)
+		(width 0.127)
+		(layer "F.Cu")
+		(net 27)
+	)
+	(segment
+		(start 182.245 88.265)
+		(end 181.61 88.9)
+		(width 0.127)
+		(layer "F.Cu")
+		(net 30)
+	)
+	(segment
+		(start 180.34 88.9)
+		(end 179.705 89.535)
+		(width 0.127)
+		(layer "F.Cu")
+		(net 30)
+	)
+	(segment
+		(start 181.61 88.9)
+		(end 180.34 88.9)
+		(width 0.127)
+		(layer "F.Cu")
+		(net 30)
+	)
+	(segment
+		(start 179.705 95.25)
+		(end 179.705 222.25)
+		(width 0.127)
+		(layer "F.Cu")
+		(net 30)
+	)
+	(segment
+		(start 182.245 86.325)
+		(end 182.245 88.265)
+		(width 0.127)
+		(layer "F.Cu")
+		(net 30)
+	)
+	(segment
+		(start 179.705 89.535)
+		(end 179.705 95.25)
+		(width 0.127)
+		(layer "F.Cu")
+		(net 30)
+	)
+	(segment
+		(start 182.245 91.475)
+		(end 182.245 95.25)
+		(width 0.127)
+		(layer "F.Cu")
+		(net 31)
+	)
+	(segment
+		(start 182.245 109.22)
+		(end 182.245 222.25)
+		(width 0.127)
+		(layer "F.Cu")
+		(net 31)
+	)
+	(segment
+		(start 182.245 95.25)
+		(end 182.245 109.22)
+		(width 0.127)
+		(layer "F.Cu")
+		(net 31)
+	)
+	(segment
+		(start 184.785 139.7)
+		(end 184.785 222.25)
+		(width 0.127)
+		(layer "F.Cu")
+		(net 32)
+	)
+	(segment
+		(start 184.785 91.475)
+		(end 184.785 95.25)
+		(width 0.127)
+		(layer "F.Cu")
+		(net 32)
+	)
+	(segment
+		(start 184.785 95.25)
+		(end 184.785 139.7)
+		(width 0.127)
+		(layer "F.Cu")
+		(net 32)
+	)
+	(segment
+		(start 188.595 95.25)
+		(end 188.595 146.05)
+		(width 0.127)
+		(layer "F.Cu")
+		(net 34)
+	)
+	(segment
+		(start 188.595 91.475)
+		(end 188.595 95.25)
+		(width 0.127)
+		(layer "F.Cu")
+		(net 34)
+	)
+	(segment
+		(start 188.595 146.05)
+		(end 188.595 222.25)
+		(width 0.127)
+		(layer "F.Cu")
+		(net 34)
+	)
+	(segment
+		(start 186.055 91.475)
+		(end 186.055 95.25)
+		(width 0.127)
+		(layer "F.Cu")
+		(net 36)
+	)
+	(segment
+		(start 186.055 95.25)
+		(end 186.055 222.25)
+		(width 0.127)
+		(layer "F.Cu")
+		(net 36)
+	)
+	(segment
+		(start 187.325 95.25)
+		(end 187.325 172.085)
+		(width 0.127)
+		(layer "F.Cu")
+		(net 38)
+	)
+	(segment
+		(start 187.325 172.085)
+		(end 187.325 222.25)
+		(width 0.127)
+		(layer "F.Cu")
+		(net 38)
+	)
+	(segment
+		(start 187.325 91.475)
+		(end 187.325 95.25)
+		(width 0.127)
+		(layer "F.Cu")
+		(net 38)
+	)
 )

Commit message: Some routing
Parts:
- added D1033: White, LED_SMD:LED_0603_1608Metric, F.Cu at (297.2, 177.8)
- added D1034: White, LED_SMD:LED_0603_1608Metric, F.Cu at (315.0, 177.8)
- added D1035: White, LED_SMD:LED_0603_1608Metric, F.Cu at (271.3, 183.2)
- added D1036: White, LED_SMD:LED_0603_1608Metric, F.Cu at (271.3, 185.8)
- added D1037: White, LED_SMD:LED_0603_1608Metric, F.Cu at (271.3, 188.3)
- added D1038: White, LED_SMD:LED_0603_1608Metric, F.Cu at (271.3, 190.9)
- added D1039: White, LED_SMD:LED_0603_1608Metric, F.Cu at (275.4, 178.0)
- added D1040: White, LED_SMD:LED_0603_1608Metric, F.Cu at (275.4, 180.6)
- added D1041: White, LED_SMD:LED_0603_1608Metric, F.Cu at (275.4, 183.2)
- added D1042: White, LED_SMD:LED_0603_1608Metric, F.Cu at (275.4, 185.8)
- added D1043: White, LED_SMD:LED_0603_1608Metric, F.Cu at (275.4, 188.3)
- added D1044: White, LED_SMD:LED_0603_1608Metric, F.Cu at (275.4, 190.9)
- added D1045: White, LED_SMD:LED_0603_1608Metric, F.Cu at (279.4, 178.0)
- added D1046: White, LED_SMD:LED_0603_1608Metric, F.Cu at (279.4, 180.6)
- added D1047: White, LED_SMD:LED_0603_1608Metric, F.Cu at (279.4, 183.2)
- added D1048: White, LED_SMD:LED_0603_1608Metric, F.Cu at (279.4, 185.8)
- added R1033: 4.7k, Resistor_SMD:R_0603_1608Metric, F.Cu at (301.0, 177.8)
- added R1034: 4.7k, Resistor_SMD:R_0603_1608Metric, F.Cu at (311.1, 177.8)
- added R1035: 4.7k, Resistor_SMD:R_0603_1608Metric, F.Cu at (283.5, 183.0)
- added R1036: 4.7k, Resistor_SMD:R_0603_1608Metric, F.Cu at (283.5, 185.5)
- added R1037: 4.7k, Resistor_SMD:R_0603_1608Metric, F.Cu at (283.5, 188.0)
- added R1038: 4.7k, Resistor_SMD:R_0603_1608Metric, F.Cu at (283.5, 190.5)
- added R1039: 4.7k, Resistor_SMD:R_0603_1608Metric, F.Cu at (287.5, 177.9)
- added R1040: 4.7k, Resistor_SMD:R_0603_1608Metric, F.Cu at (287.5, 180.5)
- added R1041: 4.7k, Resistor_SMD:R_0603_1608Metric, F.Cu at (287.5, 183.0)
- added R1042: 4.7k, Resistor_SMD:R_0603_1608Metric, F.Cu at (287.5, 185.5)
- added R1043: 4.7k, Resistor_SMD:R_0603_1608Metric, F.Cu at (287.5, 188.0)
- added R1044: 4.7k, Resistor_SMD:R_0603_1608Metric, F.Cu at (287.5, 190.5)
- added R1045: 4.7k, Resistor_SMD:R_0603_1608Metric, F.Cu at (291.5, 177.9)
- added R1046: 4.7k, Resistor_SMD:R_0603_1608Metric, F.Cu at (291.5, 180.5)
- added R1047: 4.7k, Resistor_SMD:R_0603_1608Metric, F.Cu at (291.5, 183.0)
- added R1048: 4.7k, Resistor_SMD:R_0603_1608Metric, F.Cu at (291.5, 185.5)
- moved J2001 69.2 mm to (102.9, 129.5)
- moved U4010 17.1 mm to (274.3, 233.7)
- moved U4009 15.9 mm to (261.6, 233.7)
- moved U4008 15.2 mm to (248.9, 233.7)
- moved U4007 12.7 mm to (236.2, 233.7)
- moved U4006 0.64 mm to (223.5, 233.7)
Connections:
- J1002 pad 1: /I0 -> /C0
- J1002 pad 10: /I9 -> /C9
- J1002 pad 11: /I10 -> /C10
- J1002 pad 12: /I11 -> /C11
- J1002 pad 13: /I12 -> /C12
- J1002 pad 14: /I13 -> /C13
- J1002 pad 15: /I14 -> /C14
- J1002 pad 16: /I15 -> /C15
- J1002 pad 17: /C0 -> /I0
- J1002 pad 18: /C1 -> /I1
- J1002 pad 19: /C2 -> /I2
- J1002 pad 2: /I1 -> /C1
- J1002 pad 20: /C3 -> /I3
- J1002 pad 21: /C4 -> /I4
- J1002 pad 22: /C5 -> /I5
- J1002 pad 23: /C6 -> /I6
- J1002 pad 24: /C7 -> /I7
- J1002 pad 25: /C8 -> /I8
- J1002 pad 26: /C9 -> /I9
- J1002 pad 27: /C10 -> /I10
- J1002 pad 28: /C11 -> /I11
- J1002 pad 29: /C12 -> /I12
- J1002 pad 3: /I2 -> /C2
- J1002 pad 30: /C13 -> /I13
- J1002 pad 31: /C14 -> /I14
- J1002 pad 32: /C15 -> /I15
- J1002 pad 4: /I3 -> /C3
- J1002 pad 5: /I4 -> /C4
- J1002 pad 6: /I5 -> /C5
- J1002 pad 7: /I6 -> /C6
- J1002 pad 8: /I7 -> /C7
- J1002 pad 9: /I8 -> /C8
- U4005 pad 11: unconnected-(U4005-D0-Pad11) -> /B0
- U4005 pad 12: unconnected-(U4005-D1-Pad12) -> /B1
- U4005 pad 13: unconnected-(U4005-D2-Pad13) -> /B2
- U4005 pad 14: unconnected-(U4005-D3-Pad14) -> /B3
- U4005 pad 3: unconnected-(U4005-D4-Pad3) -> /B4
- U4005 pad 4: unconnected-(U4005-D5-Pad4) -> /B5
- U4005 pad 5: unconnected-(U4005-D6-Pad5) -> /B6
- U4005 pad 6: unconnected-(U4005-D7-Pad6) -> /B7
- U4006 pad 11: unconnected-(U4006-D0-Pad11) -> /B8
- U4006 pad 12: unconnected-(U4006-D1-Pad12) -> /B9
- U4006 pad 13: unconnected-(U4006-D2-Pad13) -> /B10
- U4006 pad 14: unconnected-(U4006-D3-Pad14) -> /B11
- U4006 pad 3: unconnected-(U4006-D4-Pad3) -> /B12
- U4006 pad 4: unconnected-(U4006-D5-Pad4) -> /B13
- U4006 pad 5: unconnected-(U4006-D6-Pad5) -> /B14
- U4006 pad 6: unconnected-(U4006-D7-Pad6) -> /B15
- U4007 pad 11: /Inputs/In_{16} -> /C0
- U4007 pad 12: /Inputs/In_{17} -> /C1
- U4007 pad 13: /Inputs/In_{18} -> /C2
- U4007 pad 14: /Inputs/In_{19} -> /C3
- U4007 pad 3: /Inputs/In_{20} -> /C4
- U4007 pad 4: /Inputs/In_{21} -> /C5
- U4007 pad 5: /Inputs/In_{22} -> /C6
- U4007 pad 6: /Inputs/In_{23} -> /C7
- U4008 pad 11: /Inputs/In_{8} -> /C8
- U4008 pad 12: /Inputs/In_{9} -> /C9
- U4008 pad 13: /Inputs/In_{10} -> /C10
- U4008 pad 14: /Inputs/In_{11} -> /C11
- U4008 pad 3: /Inputs/In_{12} -> /C12
- U4008 pad 4: /Inputs/In_{13} -> /C13
- U4008 pad 5: /Inputs/In_{14} -> /C14
- U4008 pad 6: /Inputs/In_{15} -> /C15
- U4009 pad 11: /Inputs/In_{0} -> /I0
- U4009 pad 12: /Inputs/In_{1} -> /I1
- U4009 pad 13: /Inputs/In_{2} -> /I2
- U4009 pad 14: /Inputs/In_{3} -> /I3
- U4009 pad 3: /Inputs/In_{4} -> /I4
- U4009 pad 4: /Inputs/In_{5} -> /I5
- U4009 pad 5: /Inputs/In_{6} -> /I6
- U4009 pad 6: /Inputs/In_{7} -> /I7
- U4010 pad 11: /Inputs/In_{0} -> /I8
- U4010 pad 12: /Inputs/In_{1} -> /I9
- U4010 pad 13: /Inputs/In_{2} -> /I10
- U4010 pad 14: /Inputs/In_{3} -> /I11
- U4010 pad 3: /Inputs/In_{4} -> /I12
- U4010 pad 4: /Inputs/In_{5} -> /I13
- U4010 pad 5: /Inputs/In_{6} -> /I14
- U4010 pad 6: /Inputs/In_{7} -> /I15
Routing:
- net /A8: track 0.00 -> 273.9 mm, vias 0 -> 3
- net /A9: track 0.00 -> 258.6 mm, vias 0 -> 3
- net /A13: track 0.00 -> 255.6 mm, vias 0 -> 3
- net /A12: track 0.00 -> 253.8 mm, vias 0 -> 3
- net /B0: track 0.00 -> 253.6 mm, vias 0 -> 3
- net /A15: track 0.00 -> 253.0 mm, vias 0 -> 3
- net /A10: track 0.00 -> 252.1 mm, vias 0 -> 3
- net /A11: track 0.00 -> 251.4 mm, vias 0 -> 1
- net /A14: track 0.00 -> 251.3 mm, vias 0 -> 3
- net /B1: track 0.00 -> 245.9 mm, vias 0 -> 3
- net /B5: track 0.00 -> 242.9 mm, vias 0 -> 3
- net /B4: track 0.00 -> 241.1 mm, vias 0 -> 3
- net /B8: track 0.00 -> 240.9 mm, vias 0 -> 3
- net /B7: track 0.00 -> 240.3 mm, vias 0 -> 3
- net /B2: track 0.00 -> 239.4 mm, vias 0 -> 3
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Other:
- board outline added: 254 x 177.8 mm

Commit message: Doing some routing
Parts:
- added D1049: Green, LED_SMD:LED_0603_1608Metric, F.Cu at (297.2, 198.1)
- added D1050: Green, LED_SMD:LED_0603_1608Metric, F.Cu at (315.0, 198.1)
- added D1051: Green, LED_SMD:LED_0603_1608Metric, F.Cu at (297.2, 200.7)
- added D1052: Green, LED_SMD:LED_0603_1608Metric, F.Cu at (315.0, 200.7)
- added D1053: Green, LED_SMD:LED_0603_1608Metric, F.Cu at (297.2, 203.2)
- added D1054: Green, LED_SMD:LED_0603_1608Metric, F.Cu at (315.0, 203.2)
- added D1055: Green, LED_SMD:LED_0603_1608Metric, F.Cu at (297.2, 205.7)
- added D1056: Green, LED_SMD:LED_0603_1608Metric, F.Cu at (315.0, 205.7)
- added D1057: Green, LED_SMD:LED_0603_1608Metric, F.Cu at (297.2, 208.3)
- added D1058: Green, LED_SMD:LED_0603_1608Metric, F.Cu at (315.0, 208.3)
- added D1059: Green, LED_SMD:LED_0603_1608Metric, F.Cu at (297.2, 210.8)
- added D1060: Green, LED_SMD:LED_0603_1608Metric, F.Cu at (315.0, 210.8)
- added D1061: Green, LED_SMD:LED_0603_1608Metric, F.Cu at (297.2, 213.4)
- added D1062: Green, LED_SMD:LED_0603_1608Metric, F.Cu at (315.0, 213.4)
- added D1063: Green, LED_SMD:LED_0603_1608Metric, F.Cu at (297.2, 215.9)
- added D1064: Green, LED_SMD:LED_0603_1608Metric, F.Cu at (315.0, 215.9)
- added R1049: 4.7k, Resistor_SMD:R_0603_1608Metric, F.Cu at (301.0, 198.1)
- added R1050: 4.7k, Resistor_SMD:R_0603_1608Metric, F.Cu at (311.1, 198.1)
- added R1051: 4.7k, Resistor_SMD:R_0603_1608Metric, F.Cu at (301.0, 200.7)
- added R1052: 4.7k, Resistor_SMD:R_0603_1608Metric, F.Cu at (311.1, 200.7)
- added R1053: 4.7k, Resistor_SMD:R_0603_1608Metric, F.Cu at (301.0, 203.2)
- added R1054: 4.7k, Resistor_SMD:R_0603_1608Metric, F.Cu at (311.1, 203.2)
- added R1055: 4.7k, Resistor_SMD:R_0603_1608Metric, F.Cu at (301.0, 205.7)
- added R1056: 4.7k, Resistor_SMD:R_0603_1608Metric, F.Cu at (311.1, 205.7)
- added R1057: 4.7k, Resistor_SMD:R_0603_1608Metric, F.Cu at (301.0, 208.3)
- added R1058: 4.7k, Resistor_SMD:R_0603_1608Metric, F.Cu at (311.1, 208.3)
- added R1059: 4.7k, Resistor_SMD:R_0603_1608Metric, F.Cu at (301.0, 210.8)
- added R1060: 4.7k, Resistor_SMD:R_0603_1608Metric, F.Cu at (311.1, 210.8)
- added R1061: 4.7k, Resistor_SMD:R_0603_1608Metric, F.Cu at (301.0, 213.4)
- added R1062: 4.7k, Resistor_SMD:R_0603_1608Metric, F.Cu at (311.1, 213.4)
- added R1063: 4.7k, Resistor_SMD:R_0603_1608Metric, F.Cu at (301.0, 215.9)
- added R1064: 4.7k, Resistor_SMD:R_0603_1608Metric, F.Cu at (311.1, 215.9)
- moved D1038 44.4 mm to (315.0, 182.9), turned to 180 degrees
- moved D1036 44.0 mm to (315.0, 180.3), turned to 180 degrees
- moved D1040 39.9 mm to (315.0, 185.4), turned to 180 degrees
- moved D1042 39.6 mm to (315.0, 188.0), turned to 180 degrees
- moved D1044 39.6 mm to (315.0, 190.5), turned to 180 degrees
- moved D1046 37.6 mm to (315.0, 193.0), turned to 180 degrees
- moved D1048 36.8 mm to (315.0, 195.6), turned to 180 degrees
- moved R1038 28.7 mm to (311.1, 182.9)
- moved R1036 28.2 mm to (311.1, 180.3)
- moved D1037 26.4 mm to (297.2, 182.9)
- moved D1035 26.0 mm to (297.2, 180.3)
- moved R1040 24.2 mm to (311.1, 185.4)
- moved R1042 23.8 mm to (311.1, 188.0)
- moved R1044 23.7 mm to (311.1, 190.5)
- moved R1046 23.4 mm to (311.1, 193.0)
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Connections:
- U3001 pad 16: unconnected-(U3001-VCC-Pad16) -> +5V
- U3001 pad 8: unconnected-(U3001-GND-Pad8) -> GND
- U3002 pad 16: unconnected-(U3002-VCC-Pad16) -> +5V
- U3002 pad 8: unconnected-(U3002-GND-Pad8) -> GND
- U3005 pad 8: unconnected-(U3005-GND-Pad8) -> GND
- U3006 pad 8: unconnected-(U3006-GND-Pad8) -> GND
- U3007 pad 8: unconnected-(U3007-GND-Pad8) -> GND
- U3008 pad 8: unconnected-(U3008-GND-Pad8) -> GND
- U3009 pad 8: unconnected-(U3009-GND-Pad8) -> GND
- U3010 pad 8: unconnected-(U3010-GND-Pad8) -> GND
Routing:
- net /C0: track 0.00 -> 228.2 mm, vias 0 -> 3
- net /C1: track 0.00 -> 220.5 mm, vias 0 -> 3
- net /C5: track 0.00 -> 217.5 mm, vias 0 -> 3
- net /C8: track 0.00 -> 216.8 mm, vias 0 -> 3
- net /C4: track 0.00 -> 215.7 mm, vias 0 -> 3
- net /C7: track 0.00 -> 214.9 mm, vias 0 -> 3
- net /C2: track 0.00 -> 214.0 mm, vias 0 -> 3
- net /C3: track 0.00 -> 213.3 mm, vias 0 -> 1
- net /C6: track 0.00 -> 213.2 mm, vias 0 -> 3
- net /C9: track 0.00 -> 207.8 mm, vias 0 -> 3
- net /C13: track 0.00 -> 204.8 mm, vias 0 -> 3
- net /C12: track 0.00 -> 203.0 mm, vias 0 -> 3
- net /I0: track 0.00 -> 202.8 mm, vias 0 -> 3
- net /C15: track 0.00 -> 202.2 mm, vias 0 -> 3
- net /C10: track 0.00 -> 201.3 mm, vias 0 -> 3
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
Commit message: More connections, more routing
Parts:
- added D1065: Yellow, LED_SMD:LED_0603_1608Metric, F.Cu at (297.2, 218.4)
- added D1066: Yellow, LED_SMD:LED_0603_1608Metric, F.Cu at (315.0, 218.4)
- added D1067: Yellow, LED_SMD:LED_0603_1608Metric, F.Cu at (297.2, 221.0)
- added D1068: Yellow, LED_SMD:LED_0603_1608Metric, F.Cu at (315.0, 221.0)
- added D1069: Yellow, LED_SMD:LED_0603_1608Metric, F.Cu at (297.2, 223.5)
- added R1065: 4.7k, Resistor_SMD:R_0603_1608Metric, F.Cu at (301.0, 218.4)
- added R1066: 4.7k, Resistor_SMD:R_0603_1608Metric, F.Cu at (311.1, 218.4)
- added R1067: 4.7k, Resistor_SMD:R_0603_1608Metric, F.Cu at (301.0, 221.0)
- added R1068: 4.7k, Resistor_SMD:R_0603_1608Metric, F.Cu at (311.1, 221.0)
- added R1069: 4.7k, Resistor_SMD:R_0603_1608Metric, F.Cu at (301.0, 223.5)
Connections:
- J1002 pad 33: unconnected-(J1002-Pin_33-Pad33) -> /Cycle0
- J1002 pad 34: unconnected-(J1002-Pin_34-Pad34) -> /Cycle1
- J1002 pad 35: unconnected-(J1002-Pin_35-Pad35) -> /Cycle2
- J1002 pad 36: unconnected-(J1002-Pin_36-Pad36) -> /Cycle3
- J1002 pad 37: unconnected-(J1002-Pin_37-Pad37) -> /Cycle4
- U3001 pad 10: unconnected-(U3001-~{SRCLR}-Pad10) -> +5V
- U3001 pad 11: unconnected-(U3001-SRCLK-Pad11) -> /Outputs/SRCLK
- U3001 pad 12: unconnected-(U3001-RCLK-Pad12) -> /Outputs/RCLK
- U3001 pad 14: unconnected-(U3001-SER-Pad14) -> /Outputs/DATA
- U3002 pad 10: unconnected-(U3002-~{SRCLR}-Pad10) -> +5V
- U3002 pad 11: unconnected-(U3002-SRCLK-Pad11) -> /Outputs/SRCLK
- U3002 pad 12: unconnected-(U3002-RCLK-Pad12) -> /Outputs/RCLK
- U3002 pad 13: unconnected-(U3002-~{OE}-Pad13) -> /Outputs/~{Enable_{Cycle}}
- U3002 pad 3: unconnected-(U3002-QD-Pad3) -> /Cycle0
- U3002 pad 4: unconnected-(U3002-QE-Pad4) -> /Cycle1
- U3002 pad 5: unconnected-(U3002-QF-Pad5) -> /Cycle2
- U3002 pad 6: unconnected-(U3002-QG-Pad6) -> /Cycle3
- U3002 pad 7: unconnected-(U3002-QH-Pad7) -> /Cycle4
- U3003 pad 10: unconnected-(U3003-~{SRCLR}-Pad10) -> +5V
- U3003 pad 11: unconnected-(U3003-SRCLK-Pad11) -> /Outputs/SRCLK
- U3003 pad 12: unconnected-(U3003-RCLK-Pad12) -> /Outputs/RCLK
- U3004 pad 10: unconnected-(U3004-~{SRCLR}-Pad10) -> +5V
- U3004 pad 11: unconnected-(U3004-SRCLK-Pad11) -> /Outputs/SRCLK
- U3004 pad 12: unconnected-(U3004-RCLK-Pad12) -> /Outputs/RCLK
- U3005 pad 10: unconnected-(U3005-~{SRCLR}-Pad10) -> +5V
- U3005 pad 11: unconnected-(U3005-SRCLK-Pad11) -> /Outputs/SRCLK
- U3005 pad 12: unconnected-(U3005-RCLK-Pad12) -> /Outputs/RCLK
- U3006 pad 10: unconnected-(U3006-~{SRCLR}-Pad10) -> +5V
- U3006 pad 11: unconnected-(U3006-SRCLK-Pad11) -> /Outputs/SRCLK
- U3006 pad 12: unconnected-(U3006-RCLK-Pad12) -> /Outputs/RCLK
- U3007 pad 10: unconnected-(U3007-~{SRCLR}-Pad10) -> +5V
- U3007 pad 11: unconnected-(U3007-SRCLK-Pad11) -> /Outputs/SRCLK
- U3007 pad 12: unconnected-(U3007-RCLK-Pad12) -> /Outputs/RCLK
- U3008 pad 10: unconnected-(U3008-~{SRCLR}-Pad10) -> +5V
- U3008 pad 11: unconnected-(U3008-SRCLK-Pad11) -> /Outputs/SRCLK
- U3008 pad 12: unconnected-(U3008-RCLK-Pad12) -> /Outputs/RCLK
- U3009 pad 10: unconnected-(U3009-~{SRCLR}-Pad10) -> +5V
- U3009 pad 11: unconnected-(U3009-SRCLK-Pad11) -> /Outputs/SRCLK
- U3009 pad 12: unconnected-(U3009-RCLK-Pad12) -> /Outputs/RCLK
- U3009 pad 13: unconnected-(U3009-~{OE}-Pad13) -> /Outputs/~{I_{enable}}
- U3010 pad 10: unconnected-(U3010-~{SRCLR}-Pad10) -> +5V
- U3010 pad 11: unconnected-(U3010-SRCLK-Pad11) -> /Outputs/SRCLK
- U3010 pad 12: unconnected-(U3010-RCLK-Pad12) -> /Outputs/RCLK
- U3010 pad 13: unconnected-(U3010-~{OE}-Pad13) -> /Outputs/~{I_{enable}}
- U4002 pad 11: unconnected-(U4002-D0-Pad11) -> GND
- U4002 pad 12: unconnected-(U4002-D1-Pad12) -> GND
- U4002 pad 13: unconnected-(U4002-D2-Pad13) -> GND
- U4002 pad 14: unconnected-(U4002-D3-Pad14) -> /Cycle0
- U4002 pad 3: unconnected-(U4002-D4-Pad3) -> /Cycle1
- U4002 pad 4: unconnected-(U4002-D5-Pad4) -> /Cycle2
- U4002 pad 5: unconnected-(U4002-D6-Pad5) -> /Cycle3
- U4002 pad 6: unconnected-(U4002-D7-Pad6) -> /Cycle4
Routing:
- net /Cycle1: track 0.00 -> 282.3 mm, vias 0 -> 3
- net /Cycle3: track 0.00 -> 279.7 mm, vias 0 -> 3
- net /Cycle2: track 0.00 -> 277.9 mm, vias 0 -> 3
- net /Cycle4: track 0.00 -> 275.4 mm, vias 0 -> 3
- net /Cycle0: track 0.00 -> 273.7 mm, vias 0 -> 1
- net /Outputs/SRCLK: track 0.00 -> 161.6 mm, vias 0 -> 10
- net /Outputs/RCLK: track 0.00 -> 154.0 mm, vias 0 -> 10
- net Net-(U3009-QH'): track 0.00 -> 11.4 mm, vias 0 -> 2
- net Net-(U3005-QH'): track 0.00 -> 11.4 mm, vias 0 -> 2
- net Net-(U3007-QH'): track 0.00 -> 11.4 mm, vias 0 -> 2
- net Net-(U3004-QH'): track 0.00 -> 11.4 mm, vias 0 -> 2
- net Net-(U3003-QH'): track 0.00 -> 11.4 mm, vias 0 -> 2
- net /Outputs/Cont1: track 0.00 -> 11.4 mm, vias 0 -> 2
- net Net-(U3008-QH'): track 0.00 -> 11.4 mm, vias 0 -> 2
Other:
- board text added: "C"
- board text added: "C0"
- board text added: "C1"
- board text added: "C14"
- board text added: "C15"
- board text added: "I"
- board text added: "I0"
- board text added: "I1"
- board text added: "I14"
- board text added: "I15"

Commit message: Some more routes
Routing:
- net /Inputs/~{IN_{SELECT}}: track 0.00 -> 247.8 mm, vias 0 -> 10
- net /Inputs/~{IN_{LOAD}}: track 0.00 -> 168.9 mm, vias 0 -> 10
- net /Inputs/IN_{CLK}: track 0.00 -> 157.5 mm, vias 0 -> 10
- net /Outputs/~{I_{enable}}: track 0.00 -> 133.9 mm, vias 0 -> 2
- net /Outputs/~{C_{enable}}: track 0.00 -> 111.1 mm, vias 0 -> 2
- net /Outputs/~{B_{enable}}: track 0.00 -> 88.2 mm, vias 0 -> 2
- net /Outputs/~{A_{enable}}: track 0.00 -> 65.3 mm, vias 0 -> 2
- net +5V: track 0.00 -> 57.1 mm, vias 0 -> 30
- net /Outputs/RCLK: track 154.0 -> 187.0 mm
- net /Outputs/~{Enable_{Cycle}}: track 0.00 -> 31.1 mm, vias 0 -> 1
- net Net-(U4006-DS): track 0.00 -> 29.2 mm, vias 0 -> 2
- net Net-(U4004-DS): track 0.00 -> 29.2 mm, vias 0 -> 2
- net Net-(U4001-DS): track 0.00 -> 29.2 mm, vias 0 -> 2
- net Net-(U4008-DS): track 0.00 -> 29.2 mm, vias 0 -> 2
- net Net-(U4005-DS): track 0.00 -> 29.2 mm, vias 0 -> 2
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Other:
- board size 254 x 177.8 mm -> 254 x 184.2 mm
