File: pcbs/Pi Backplane Connector/Pi Backplane Connector.kicad_pcb (KiCad board)
At the start: 2 copper layers, 254 x 184.2 mm, 161 parts, among them J1001 Conn_02x20_Odd_Even, J1002 Conn_02x20_Odd_Even, J2001 Raspberry_Pi_2_3, U3001 74HC595, U3002 74HC595, U3003 74HC595, U3004 74HC595, U3005 74HC595, U3006 74HC595, U3007 74HC595, U3008 74HC595, U3009 74HC595, U3010 74HC595, U4001 74HC165, U4002 74HC165, U4003 74HC165, U4004 74HC165, U4005 74HC165, U4006 74HC165, U4007 74HC165, U4008 74HC165, U4009 74HC165, U4010 74HC165

Commit message: Connections and capacitors
Parts:
- added C3001: 100n, Capacitor_SMD:C_0603_1608Metric, F.Cu at (153.7, 85.7)
- added C3002: 100n, Capacitor_SMD:C_0603_1608Metric, F.Cu at (166.4, 85.7)
- added C3003: 100n, Capacitor_SMD:C_0603_1608Metric, F.Cu at (179.1, 85.7)
- added C3004: 100n, Capacitor_SMD:C_0603_1608Metric, F.Cu at (191.8, 85.7)
- added C3005: 100n, Capacitor_SMD:C_0603_1608Metric, F.Cu at (204.5, 85.7)
- added C3006: 100n, Capacitor_SMD:C_0603_1608Metric, F.Cu at (217.2, 85.7)
- added C3007: 100n, Capacitor_SMD:C_0603_1608Metric, F.Cu at (229.9, 85.7)
- added C3008: 100n, Capacitor_SMD:C_0603_1608Metric, F.Cu at (242.6, 85.7)
- added C3009: 100n, Capacitor_SMD:C_0603_1608Metric, F.Cu at (255.3, 85.7)
- added C3010: 100n, Capacitor_SMD:C_0603_1608Metric, F.Cu at (268.0, 85.6)
- added C4001: 100n, Capacitor_SMD:C_0603_1608Metric, F.Cu at (153.0, 228.6)
- added C4002: 100n, Capacitor_SMD:C_0603_1608Metric, F.Cu at (165.7, 228.6)
- added C4003: 100n, Capacitor_SMD:C_0603_1608Metric, F.Cu at (178.4, 228.6)
- added C4004: 100n, Capacitor_SMD:C_0603_1608Metric, F.Cu at (191.1, 228.6)
- added C4005: 100n, Capacitor_SMD:C_0603_1608Metric, F.Cu at (203.8, 228.6)
- added C4006: 100n, Capacitor_SMD:C_0603_1608Metric, F.Cu at (216.5, 228.6)
- added C4007: 100n, Capacitor_SMD:C_0603_1608Metric, F.Cu at (229.2, 228.6)
- added C4008: 100n, Capacitor_SMD:C_0603_1608Metric, F.Cu at (241.9, 228.6)
- added C4009: 100n, Capacitor_SMD:C_0603_1608Metric, F.Cu at (254.6, 228.6)
- added C4010: 100n, Capacitor_SMD:C_0603_1608Metric, F.Cu at (267.3, 228.6)
- added D1070: Yellow, LED_SMD:LED_0603_1608Metric, F.Cu at (315.0, 149.9)
- added D1071: Yellow, LED_SMD:LED_0603_1608Metric, F.Cu at (297.2, 149.9)
- added R1070: 4.7k, Resistor_SMD:R_0603_1608Metric, F.Cu at (311.1, 149.9)
- added R1071: 4.7k, Resistor_SMD:R_0603_1608Metric, F.Cu at (301.0, 149.9)
- added U3011: 74AHCT125, Package_DIP:DIP-14_W7.62mm_Socket, F.Cu at (144.8, 142.2)
Connections:
- net /Outputs/~{Enable_{Cycle}} renamed /Outputs/~{Cycle_{enable}}
- J1001 pad 39: unconnected-(J1001-Pin_39-Pad39) -> /RESET
- J1001 pad 40: unconnected-(J1001-Pin_40-Pad40) -> /CLOCK
- U3001 pad 1: unconnected-(U3001-QB-Pad1) -> /Outputs/RST_{out}
- U3001 pad 13: unconnected-(U3001-~{OE}-Pad13) -> GND
- U3001 pad 2: unconnected-(U3001-QC-Pad2) -> /Outputs/CLK_{out}
- U4001 pad 11: unconnected-(U4001-D0-Pad11) -> GND
- U4001 pad 12: unconnected-(U4001-D1-Pad12) -> /CLOCK
- U4001 pad 13: unconnected-(U4001-D2-Pad13) -> /RESET
- U4001 pad 14: unconnected-(U4001-D3-Pad14) -> GND
- U4001 pad 3: unconnected-(U4001-D4-Pad3) -> GND
- U4001 pad 4: unconnected-(U4001-D5-Pad4) -> GND
- U4001 pad 5: unconnected-(U4001-D6-Pad5) -> GND
- U4001 pad 6: unconnected-(U4001-D7-Pad6) -> GND
Routing:
- net /CLOCK: track 0.00 -> 235.5 mm, vias 0 -> 2
- net /RESET: track 0.00 -> 233.7 mm, vias 0 -> 1
- net /Outputs/CLK_{out}: track 0.00 -> 67.5 mm
- net /Outputs/RST_{out}: track 0.00 -> 58.6 mm
- net +5V: track 57.1 -> 98.4 mm
Other:
- board text added: "CLOCK"
- board text added: "~{RESET}"

Commit message: Starting on the connections...
Parts:
- added R3001: 1M, Resistor_SMD:R_0603_1608Metric, F.Cu at (174.6, 74.9)
- added R3002: 1M, Resistor_SMD:R_0603_1608Metric, F.Cu at (200.0, 76.2)
- added R3003: 1M, Resistor_SMD:R_0603_1608Metric, F.Cu at (225.4, 77.5)
- added R3004: 1M, Resistor_SMD:R_0603_1608Metric, F.Cu at (250.8, 78.7)
- added R3005: 1M, Resistor_SMD:R_0603_1608Metric, F.Cu at (276.2, 80.0)
- added R3006: 1M, Resistor_SMD:R_0603_1608Metric, F.Cu at (165.1, 144.8)
- added R3007: 1M, Resistor_SMD:R_0603_1608Metric, F.Cu at (165.1, 152.4)
- added U2001: SN74LVC4245APWR, Package_SO:TSSOP-24_4.4x7.8mm_P0.65mm, F.Cu at (127.0, 132.1)
Routing:
- net /Outputs/~{RESET_{enable}}: track 0.00 -> 11.9 mm, vias 0 -> 1
- net /Outputs/~{CLOCK_{enable}}: track 0.00 -> 11.9 mm, vias 0 -> 1
- net +5V: track 98.4 -> 107.3 mm, vias 30 -> 37
- net /Outputs/~{Cycle_{enable}}: track 31.1 -> 32.8 mm
- net /Outputs/~{C_{enable}}: track 111.1 -> 112.8 mm
- net /Outputs/~{B_{enable}}: track 88.2 -> 89.9 mm
- net /Outputs/~{I_{enable}}: track 133.9 -> 135.6 mm
- net /Outputs/~{A_{enable}}: track 65.3 -> 67.0 mm

Commit message: Thinking about Pi connections
Parts:
- added C2001: 100n, Capacitor_SMD:C_0603_1608Metric, F.Cu at (127.0, 139.7)
- added C2002: 100n, Capacitor_SMD:C_0603_1608Metric, F.Cu at (127.0, 154.9)
- added C2003: 100n, Capacitor_SMD:C_0603_1608Metric, F.Cu at (127.0, 170.2)
- added R2001: 1M, Resistor_SMD:R_0603_1608Metric, F.Cu at (101.6, 210.8)
- added R2002: 1M, Resistor_SMD:R_0603_1608Metric, F.Cu at (101.6, 227.3)
- added R2003: 1M, Resistor_SMD:R_0603_1608Metric, F.Cu at (101.6, 229.9)
- added R2004: 1M, Resistor_SMD:R_0603_1608Metric, F.Cu at (101.6, 214.6)
- added R2005: 1M, Resistor_SMD:R_0603_1608Metric, F.Cu at (101.6, 222.2)
- added R2006: 1M, Resistor_SMD:R_0603_1608Metric, F.Cu at (101.6, 224.8)
- added R2007: 1M, Resistor_SMD:R_0603_1608Metric, F.Cu at (101.6, 184.2)
- added R2008: 1M, Resistor_SMD:R_0603_1608Metric, F.Cu at (101.6, 188.0)
- added R2009: 1M, Resistor_SMD:R_0603_1608Metric, F.Cu at (101.6, 191.8)
- added R2010: 1M, Resistor_SMD:R_0603_1608Metric, F.Cu at (101.6, 195.6)
- added R2011: 1M, Resistor_SMD:R_0603_1608Metric, F.Cu at (101.6, 199.4)
- added R2012: 1M, Resistor_SMD:R_0603_1608Metric, F.Cu at (101.6, 203.2)
- added R2013: 1M, Resistor_SMD:R_0603_1608Metric, F.Cu at (101.6, 207.0)
- added U2001: SN74LVC4245APWR, Package_SO:TSSOP-24_4.4x7.8mm_P0.65mm, F.Cu at (121.9, 162.6)
- added U2002: SN74LVC4245APWR, Package_SO:TSSOP-24_4.4x7.8mm_P0.65mm, F.Cu at (121.9, 147.3)
- moved U2003 5.08 mm to (121.9, 132.1)
- renumbered U2001 to U2003
Connections:
- J2001 pad 19: unconnected-(J2001-MOSI0/GPIO10-Pad19) -> /Pi Control/COPI0
- J2001 pad 23: unconnected-(J2001-SCLK0/GPIO11-Pad23) -> /Pi Control/SCLK0
- J2001 pad 24: unconnected-(J2001-~{CE0}/GPIO8-Pad24) -> /Pi Control/~{PE0}
- J2001 pad 26: unconnected-(J2001-~{CE1}/GPIO7-Pad26) -> /Pi Control/~{PE1}
- J2001 pad 27: unconnected-(J2001-ID_SD/GPIO0-Pad27) -> /Pi Control/Ins
- J2001 pad 28: unconnected-(J2001-ID_SC/GPIO1-Pad28) -> /Pi Control/Abus
- J2001 pad 29: unconnected-(J2001-GCLK1/GPIO5-Pad29) -> /Pi Control/ResetWire
- J2001 pad 3: unconnected-(J2001-SDA/GPIO2-Pad3) -> /Pi Control/Bbus
- J2001 pad 31: unconnected-(J2001-GCLK2/GPIO6-Pad31) -> /Pi Control/ClockWire
- J2001 pad 35: unconnected-(J2001-GPIO19/MISO1-Pad35) -> /Pi Control/CIPO1
- J2001 pad 40: unconnected-(J2001-GPIO21/SCLK1-Pad40) -> /Pi Control/SCLK1
- J2001 pad 5: unconnected-(J2001-SCL/GPIO3-Pad5) -> /Pi Control/Cbus
- J2001 pad 7: unconnected-(J2001-GCLK0/GPIO4-Pad7) -> /Pi Control/CYCLEbus
- U2003 pad 10: unconnected-(U2001-A8-Pad10) -> /Outputs/SRCLK
- U2003 pad 14: unconnected-(U2001-B8-Pad14) -> /Pi Control/SCLK0
- U2003 pad 15: unconnected-(U2001-B7-Pad15) -> /Pi Control/COPI0
- U2003 pad 16: unconnected-(U2001-B6-Pad16) -> /Pi Control/~{PE0}
- U2003 pad 17: unconnected-(U2001-B5-Pad17) -> GND
- U2003 pad 18: unconnected-(U2001-B4-Pad18) -> GND
- U2003 pad 19: unconnected-(U2001-B3-Pad19) -> /Pi Control/~{PE1}
- U2003 pad 2: +5V -> GND
- U2003 pad 20: unconnected-(U2001-B2-Pad20) -> /Pi Control/~{LOAD_1}
- U2003 pad 21: unconnected-(U2001-B1-Pad21) -> /Pi Control/SCLK1
- U2003 pad 3: unconnected-(U2001-A1-Pad3) -> /Inputs/IN_{CLK}
- U2003 pad 4: unconnected-(U2001-A2-Pad4) -> /Inputs/~{IN_{LOAD}}
- U2003 pad 5: unconnected-(U2001-A3-Pad5) -> /Outputs/RCLK
- U2003 pad 8: unconnected-(U2001-A6-Pad8) -> /Inputs/~{IN_{SELECT}}
- U2003 pad 9: unconnected-(U2001-A7-Pad9) -> /Outputs/DATA
Routing:
- net /Inputs/~{IN_{SELECT}}: track 247.8 -> 350.9 mm
- net /Inputs/~{IN_{LOAD}}: track 168.9 -> 269.5 mm
- net /Inputs/IN_{CLK}: track 157.5 -> 255.5 mm
- net /Inputs/IN_{DATA}: track 19.9 -> 98.9 mm
- net /Outputs/~{Cycle_{enable}}: track 32.8 -> 106.1 mm
- net /Outputs/~{A_{enable}}: track 67.0 -> 137.8 mm
- net /Outputs/~{B_{enable}}: track 89.9 -> 158.1 mm
- net /Outputs/~{C_{enable}}: track 112.8 -> 178.4 mm
- net /Outputs/DATA: track 0.00 -> 63.7 mm, vias 0 -> 1
- net /Outputs/~{I_{enable}}: track 135.6 -> 198.8 mm
- net /Outputs/RCLK: track 187.0 -> 247.6 mm
- net /Outputs/SRCLK: track 161.6 -> 219.6 mm
