File: pcbs/Pi Backplane Connector/picontrol.kicad_sch (KiCad schematic)
At the start: 1 part, among them J2001 Raspberry_Pi_2_3

Commit message: Starting on the connections...
Parts:
- added U2001: SN74LVC4245APWR, Package_SO:TSSOP-24_4.4x7.8mm_P0.65mm, symbol 7400_Extras:74LVC4245
Connections:
- net +3.3V: now also U2001.23 (V_{CCB}), U2001.24 (V_{CCB})
- net +5V: now also U2001.1 (V_{CCA}), U2001.2 (AB/~{BA})
- net GND: now also U2001.11 (GND), U2001.12 (GND), U2001.13 (GND), U2001.22 (~{OE})
Other:
- moved on the sheet: J2001

Commit message: Thinking about Pi connections
Parts:
- added C2001, C2002, C2003: 100n, Capacitor_SMD:C_0603_1608Metric, symbol Device:C
- added R2001, R2002, R2003, R2004, R2005, R2006, R2007, R2008, R2009, R2010, R2011, R2012, R2013: 1M, Resistor_SMD:R_0603_1608Metric, symbol Device:R
- added U2001, U2002: SN74LVC4245APWR, Package_SO:TSSOP-24_4.4x7.8mm_P0.65mm, symbol 7400_Extras:74LVC4245
- renumbered U2001 to U2003
Connections:
- net +3.3V: now also U2001.23 (V_{CCB}), U2001.24 (V_{CCB}), U2002.23 (V_{CCB}), U2002.24 (V_{CCB})
- net +5V: now also C2001.2, C2002.2, C2003.2, R2001.2, R2002.2, R2003.2, R2007.2, R2008.2, R2009.2, R2010.2, R2011.2, R2012.2, R2013.2, U2001.1 (V_{CCA}), U2001.2 (AB/~{BA}), U2002.1 (V_{CCA}); no longer U2003.2 (AB/~{BA})
- net GND: now also U2003.17 (B5), U2003.18 (B4), U2003.2 (AB/~{BA}), C2001.1, C2002.1, C2003.1, R2004.2, R2005.2, R2006.2, U2001.10 (A8), U2001.11 (GND), U2001.12 (GND), U2001.13 (GND), U2001.22 (~{OE}), U2001.4 (A2), U2001.5 (A3), U2001.6 (A4), U2001.7 (A5), U2001.8 (A6), U2001.9 (A7), U2002.11 (GND), U2002.12 (GND), U2002.13 (GND), U2002.14 (B8), U2002.2 (AB/~{BA}), U2002.22 (~{OE})
- net CLK_OUT: now reaches U2003.10 (A8)
- net SCLK0: now reaches U2003.14 (B8)
- net SCLK0: now also J2001.23 (SCLK0/GPIO11), R2005.1
- net COPI0: now reaches U2003.15 (B7)
- net COPI0: now also J2001.19 (MOSI0/GPIO10), R2004.1
- net ~{PE0}: now reaches U2003.16 (B6)
- net ~{PE0}: now also J2001.24 (~{CE0}/GPIO8), R2001.1
- net ~{PE1}: now reaches U2003.19 (B3)
- net ~{PE1}: now also J2001.26 (~{CE1}/GPIO7), R2003.1
- net ~{LOAD_1}: now reaches U2003.20 (B2)
- net ~{LOAD_1}: now also R2002.1
- net SCLK1: now reaches U2003.21 (B1)
- net SCLK1: now also J2001.40 (GPIO21/SCLK1), R2006.1
- net CLK_IN: now reaches U2003.3 (A1)
- net ~{IN_{ld}}: now reaches U2003.4 (A2)
- net ~{IN_{en}}: now reaches U2003.5 (A3)
- net ~{OUT_{en}}: now reaches U2003.8 (A6)
- net DATA_OUT: now reaches U2003.9 (A7)
- net Ins: now reaches J2001.27 (ID_SD/GPIO0)
- net Ins: now also R2007.1, U2002.21 (B1)
- net Abus: now reaches J2001.28 (ID_SC/GPIO1)
- net Abus: now also R2008.1, U2002.20 (B2)
- net ResetWire: now reaches J2001.29 (GCLK1/GPIO5)
- net ResetWire: now also R2012.1, U2002.16 (B6)
- net Bbus: now reaches J2001.3 (SDA/GPIO2)
- net Bbus: now also R2009.1, U2002.19 (B3)
- net ClockWire: now reaches J2001.31 (GCLK2/GPIO6)
- net ClockWire: now also R2013.1, U2002.15 (B7)
- net CIPO1: now reaches J2001.35 (GPIO19/MISO1)
- net CIPO1: now also U2001.21 (B1)
- net Cbus: now reaches J2001.5 (SCL/GPIO3)
- net Cbus: now also R2010.1, U2002.18 (B4)
- net CYCLEbus: now reaches J2001.7 (GCLK0/GPIO4)
- net CYCLEbus: now also R2011.1, U2002.17 (B5)
- new net IN_DATA: U2001.3 (A1)
- new net ~{A_{en}}: U2002.4 (A2)
- new net ~{B_{en}}: U2002.5 (A3)
- new net ~{CLOCK_{en}}: U2002.9 (A7)
- new net ~{CYCLE_{en}}: U2002.7 (A5)
- new net ~{C_{en}}: U2002.6 (A4)
- new net ~{I_{en}}: U2002.3 (A1)
- new net ~{RESET_{en}}: U2002.8 (A6)
- no-connect marks 0 -> 12

Commit message: Don't destroy the Pi
Connections:
- net +3.3V: now also R2001.2, R2002.2, R2003.2, R2007.2, R2008.2, R2009.2, R2010.2, R2011.2, R2012.2, R2013.2
- net +5V: no longer R2001.2, R2002.2, R2003.2, R2007.2, R2008.2, R2009.2, R2010.2, R2011.2, R2012.2, R2013.2

Commit message: Doing some routing
Connections:
- net Abus: now also J2001.8 (GPIO14/TXD), U2003.20 (B2); no longer J2001.28 (ID_SC/GPIO1), U2002.20 (B2)
- net Bbus: now also U2003.19 (B3); no longer U2002.19 (B3)
- net CLK_IN: now also U2002.3 (A1); no longer U2003.3 (A1)
- net CYCLEbus: now also J2001.10 (GPIO15/RXD), U2003.21 (B1); no longer J2001.7 (GCLK0/GPIO4), U2002.17 (B5)
- net Cbus: now also U2003.18 (B4); no longer U2002.18 (B4)
- net ClockWire: no longer J2001.31 (GCLK2/GPIO6)
- net GND: no longer U2003.17 (B5), U2003.18 (B4)
- net Ins: now also J2001.7 (GCLK0/GPIO4), U2003.17 (B5); no longer J2001.27 (ID_SD/GPIO0), U2002.21 (B1)
- net ResetWire: no longer J2001.29 (GCLK1/GPIO5)
- net SCLK1: now also U2002.21 (B1); no longer U2003.21 (B1)
- net ~{A_{en}}: now also U2003.4 (A2); no longer U2002.4 (A2)
- net ~{B_{en}}: now also U2003.5 (A3); no longer U2002.5 (A3)
- net ~{CYCLE_{en}}: now also U2003.3 (A1); no longer U2002.7 (A5)
- net ~{C_{en}}: now also U2003.6 (A4); no longer U2002.6 (A4)
- net ~{IN_{en}}: now also U2002.5 (A3); no longer U2003.5 (A3)
- net ~{IN_{ld}}: now also U2002.4 (A2); no longer U2003.4 (A2)
- net ~{I_{en}}: now also U2003.7 (A5); no longer U2002.3 (A1)
- net ~{LOAD_1}: now also J2001.32 (PWM0/GPIO12), U2002.20 (B2); no longer U2003.20 (B2)
- net ~{PE1}: now also U2002.19 (B3); no longer U2003.19 (B3)
- no-connect marks 12 -> 10

Commit message: Completing initial wire-up
Connections:
- net ClockWire: now also J2001.11 (GPIO17), U2002.16 (B6); no longer U2002.15 (B7)
- net ResetWire: now also J2001.12 (GPIO18/PWM0), U2002.15 (B7); no longer U2002.16 (B6)
- net ~{CLOCK_{en}}: now also U2002.8 (A6); no longer U2002.9 (A7)
- net ~{RESET_{en}}: now also U2002.9 (A7); no longer U2002.8 (A6)
Changed lines of the file:
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@@
 	)
 	(label "ResetWire"
-		(at 113.03 110.49 180)
+		(at 113.03 113.03 180)
 		(fields_autoplaced yes)
 		(effects
@@
 	)
 	(label "ResetWire"
-		(at 87.63 58.42 0)
-		(fields_autoplaced yes)
-		(effects
-			(font
-				(size 1.27 1.27)
-			)
-			(justify left bottom)
+		(at 22.86 52.07 180)
+		(fields_autoplaced yes)
+		(effects
+			(font
+				(size 1.27 1.27)
+			)
+			(justify right bottom)
 		)
 	)
 	(label "ClockWire"
-		(at 92.71 62.23 180)
+		(at 22.86 49.53 180)
 		(fields_autoplaced yes)
 		(effects
@@
 	)
 	(label "ClockWire"
-		(at 113.03 113.03 180)
+		(at 113.03 110.49 180)
 		(fields_autoplaced yes)
 		(effects
@@
 	(hierarchical_label "~{CLOCK_{en}}"
 		(shape output)
-		(at 154.94 113.03 0)
+		(at 154.94 110.49 0)
 		(fields_autoplaced yes)
 		(effects
@@
 	(hierarchical_label "~{RESET_{en}}"
 		(shape output)
-		(at 154.94 110.49 0)
-		(fields_autoplaced yes)
-		(effects
+		(at 154.94 113.03 0)
+		(fields_autoplaced yes)
+		(effects

Commit message: Double checking
Connections:
- net GND: now also U2002.17 (B5), U2002.18 (B4)
- no-connect marks 10 -> 24
Changed lines of the file:
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@@
+	)
+	(junction
+		(at 118.11 105.41)
+		(diameter 0)
+		(color 0 0 0 0)
 	)
 	(junction
@@
 	)
 	(no_connect
+		(at 66.04 41.91)
+	)
+	(no_connect
+		(at 25.4 69.85)
+	)
+	(no_connect
+		(at 154.94 105.41)
+	)
+	(no_connect
+		(at 25.4 80.01)
+	)
+	(no_connect
+		(at 25.4 46.99)
+	)
+	(no_connect
+		(at 154.94 107.95)
+	)
+	(no_connect
+		(at 66.04 57.15)
+	)
+	(no_connect
+		(at 25.4 67.31)
+	)
+	(no_connect
+		(at 66.04 39.37)
+	)
+	(no_connect
 		(at 121.92 170.18)
 	)
@@
 	)
 	(no_connect
+		(at 25.4 72.39)
+	)
+	(no_connect
+		(at 25.4 77.47)
+	)
+	(no_connect
 		(at 121.92 162.56)
 	)
@@
 	)
 	(no_connect
+		(at 66.04 82.55)
+	)
+	(no_connect
 		(at 66.04 69.85)
 	)
@@
 	)
 	(no_connect
+		(at 25.4 74.93)
+	)
+	(no_connect
 		(at 121.92 172.72)
 	)
@@
 	)
 	(no_connect
+		(at 66.04 59.69)
+	)
+	(no_connect
 		(at 121.92 165.1)
 	)
@@
 	(wire
 		(pts
-			(xy 113.03 107.95) (xy 123.19 107.95)
-		)
-		(stroke
-			(width 0)
-			(type default)
-		)
-	)
-	(wire
-		(pts
 			(xy 137.16 64.77) (xy 140.97 64.77)
 		)
@@
 	(wire
 		(pts
+			(xy 118.11 105.41) (xy 123.19 105.41)
+		)
+		(stroke
+			(width 0)
+			(type default)
+		)
+	)
+	(wire
+		(pts
 			(xy 148.59 83.82) (xy 151.13 83.82)
 		)
@@
 	(wire
 		(pts
+			(xy 118.11 107.95) (xy 123.19 107.95)
+		)
+		(stroke
+			(width 0)
+			(type default)
+		)
+	)
+	(wire
+		(pts
 			(xy 198.12 114.3) (xy 200.66 114.3)
 		)
@@
 	(wire
 		(pts
+			(xy 118.11 105.41) (xy 118.11 107.95)
+		)
+		(stroke
+			(width 0)
+			(type default)
+		)
+	)
+	(wire
+		(pts
 			(xy 66.04 54.61) (xy 68.58 54.61)
 		)
@@
 	(wire
 		(pts
-			(xy 113.03 105.41) (xy 123.19 105.41)
+			(xy 113.03 105.41) (xy 118.11 105.41)
 		)
 		(stroke
@@
 					(unit 1)
 				)
+			)
+		)
+	)
+	(symbol
+		(lib_id "power:GND")
+		(at 113.03 105.41 270)
+		(unit 1)
+		(exclude_from_sim no)
+		(in_bom yes)
+		(on_board yes)
+		(dnp no)
+		(fields_autoplaced yes)
+		(property "Reference" "#PWR02004"
+			(at 106.68 105.41 0)
+			(effects
+				(font
+					(size 1.27 1.27)
+				)
+				(hide yes)
+			)
+		)
+		(property "Value" "GND"
+			(at 109.22 105.4099 90)
+			(effects
+				(font
+					(size 1.27 1.27)
+				)
+				(justify right)
+			)
+		)
+		(property "Footprint" ""
+			(at 113.03 105.41 0)
+			(effects
+				(font
+					(size 1.27 1.27)
+				)
+				(hide yes)
+			)
+		)
+		(property "Datasheet" ""
+			(at 113.03 105.41 0)
+			(effects
+				(font
+					(size 1.27 1.27)
+				)
+				(hide yes)
+			)
+		)
+		(property "Description" "Power symbol creates a global label with name \"GND\" , ground"
+			(at 113.03 105.41 0)
+			(effects
+				(font
+					(size 1.27 1.27)
+				)
+				(hide yes)
+			)
+		)
+		(pin "1"
+		)
+		(instances
+			(project ""
+				(path "/84ab2617-954b-4ceb-a5e3-268c9e11a862/f2d6763d-0b70-425b-969c-e85d688f63f8"
+					(reference "#PWR02004")
+					(unit 1)
+				)
