File: pcbs/ALU Carrier/xornand.kicad_sch (KiCad schematic)
At the start: 0 parts

Commit message: Roughing out
Parts:
- added J5001, J5002: ~, BoardEdgeConnectors:TE-5530843-4-Mount, symbol BoardEdgeConnectors:TE-5530843-4
Connections:
- new net +5V: J5001.B1, J5002.B1
- new net A0: J5001.A2
- new net A1: J5001.B2
- new net A10: J5002.A3
- new net A11: J5002.B3
- new net A12: J5002.A4
- new net A13: J5002.B4
- new net A14: J5002.A5
- new net A15: J5002.B5
- new net A2: J5001.A3
- new net A3: J5001.B3
- new net A4: J5001.A4
- new net A5: J5001.B4
- new net A6: J5001.A5
- new net A7: J5001.B5
- new net A8: J5002.A2
- new net A9: J5002.B2
- new net B0: J5001.A8
- new net B1: J5001.B8
- new net B10: J5002.A9
- new net B11: J5002.B9
- new net B12: J5002.A10
- new net B13: J5002.B10
- new net B14: J5002.A11
- new net B15: J5002.B11
- new net B2: J5001.A9
- new net B3: J5001.B9
- new net B4: J5001.A10
- new net B5: J5001.B10
- new net B6: J5001.A11
- new net B7: J5001.B11
- new net B8: J5002.A8
- new net B9: J5002.B8
- new net GND: J5001.A22, J5002.A22
- new net Out0: J5001.A17
- new net Out1: J5001.B17
- new net Out10: J5002.A18
- new net Out11: J5002.B18
- new net Out12: J5002.A19
- new net Out13: J5002.B19
- new net Out14: J5002.A20
- new net Out15: J5002.B20
- new net Out2: J5001.A18
- new net Out3: J5001.B18
- new net Out4: J5001.A19
- new net Out5: J5001.B19
- new net Out6: J5001.A20
- new net Out7: J5001.B20
- new net Out8: J5002.A17
- new net Out9: J5002.B17
- new net ~{NAND}: J5001.A14, J5002.A14
- new net ~{XOR}: J5001.B14, J5002.B14
- no-connect marks 0 -> 32
