File: pcbs/ALU Carrier/ALU Carrier.kicad_pcb (KiCad board)
At the start: 2 copper layers, 65 parts, among them J1001 Conn_02x20_Odd_Even, J1002 Conn_02x20_Odd_Even, U2001 74HC138, U6001 74HC14, U7001 74HC14, U7002 74HC08, U8001 74HC245, U8002 74HC245

Commit message: Routing, routing, routing
Parts:
- moved R8017 210.2 mm to (69.8, 97.2)
- moved D8017 200.3 mm to (66.7, 102.4), turned to -90 degrees
- moved R8016 81.0 mm to (243.8, 231.1), turned to 180 degrees
- moved D8013 78.5 mm to (240.0, 223.5), turned to 180 degrees
- moved D8014 78.4 mm to (240.0, 226.1), turned to 180 degrees
- moved D8015 78.4 mm to (240.0, 228.6), turned to 180 degrees
- moved D8016 78.3 mm to (240.0, 231.1), turned to 180 degrees
- moved R8001 70.4 mm to (273.2, 217.1), turned to 180 degrees
- moved R8013 70.0 mm to (265.2, 217.1), turned to 180 degrees
- moved R8007 69.7 mm to (269.2, 217.1), turned to 180 degrees
- moved R8012 66.4 mm to (252.9, 224.8), turned to 180 degrees
- moved R8002 65.5 mm to (273.2, 214.6), turned to 180 degrees
- moved R8014 65.0 mm to (265.2, 214.6), turned to 180 degrees
- moved R8008 64.7 mm to (269.2, 214.6), turned to 180 degrees
- moved D8007 62.7 mm to (240.0, 208.3), turned to 180 degrees
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Connections:
- U8001 pad 11: unconnected-(U8001-B7-Pad11) -> /Adder Subtractor/Out7
- U8001 pad 12: unconnected-(U8001-B6-Pad12) -> /Adder Subtractor/Out6
- U8001 pad 13: unconnected-(U8001-B5-Pad13) -> /Adder Subtractor/Out5
- U8001 pad 14: unconnected-(U8001-B4-Pad14) -> /Adder Subtractor/Out4
- U8001 pad 15: unconnected-(U8001-B3-Pad15) -> /Adder Subtractor/Out3
- U8001 pad 16: unconnected-(U8001-B2-Pad16) -> /Adder Subtractor/Out2
- U8001 pad 17: unconnected-(U8001-B1-Pad17) -> /Adder Subtractor/Out1
- U8001 pad 18: unconnected-(U8001-B0-Pad18) -> /Adder Subtractor/Out0
- U8001 pad 2: unconnected-(U8001-A0-Pad2) -> /C0
- U8001 pad 3: unconnected-(U8001-A1-Pad3) -> /C1
- U8001 pad 4: unconnected-(U8001-A2-Pad4) -> /C2
- U8001 pad 5: unconnected-(U8001-A3-Pad5) -> /C3
- U8001 pad 6: unconnected-(U8001-A4-Pad6) -> /C4
- U8001 pad 7: unconnected-(U8001-A5-Pad7) -> /C5
- U8001 pad 8: unconnected-(U8001-A6-Pad8) -> /C6
- U8001 pad 9: unconnected-(U8001-A7-Pad9) -> /C7
- U8002 pad 11: unconnected-(U8002-B7-Pad11) -> /Adder Subtractor/Out15
- U8002 pad 12: unconnected-(U8002-B6-Pad12) -> /Adder Subtractor/Out14
- U8002 pad 13: unconnected-(U8002-B5-Pad13) -> /Adder Subtractor/Out13
- U8002 pad 14: unconnected-(U8002-B4-Pad14) -> /Adder Subtractor/Out12
- U8002 pad 15: unconnected-(U8002-B3-Pad15) -> /Adder Subtractor/Out11
- U8002 pad 16: unconnected-(U8002-B2-Pad16) -> /Adder Subtractor/Out10
- U8002 pad 17: unconnected-(U8002-B1-Pad17) -> /Adder Subtractor/Out9
- U8002 pad 18: unconnected-(U8002-B0-Pad18) -> /Adder Subtractor/Out8
- U8002 pad 2: unconnected-(U8002-A0-Pad2) -> /C8
- U8002 pad 3: unconnected-(U8002-A1-Pad3) -> /C9
- U8002 pad 4: unconnected-(U8002-A2-Pad4) -> /C10
- U8002 pad 5: unconnected-(U8002-A3-Pad5) -> /C11
- U8002 pad 6: unconnected-(U8002-A4-Pad6) -> /C12
- U8002 pad 7: unconnected-(U8002-A5-Pad7) -> /C13
- U8002 pad 8: unconnected-(U8002-A6-Pad8) -> /C14
- U8002 pad 9: unconnected-(U8002-A7-Pad9) -> /C15
Routing:
- net /Adder Subtractor/Out15: track 20.8 -> 365.3 mm, vias 0 -> 5
- net /Adder Subtractor/Out13: track 27.2 -> 368.5 mm, vias 0 -> 5
- net /Adder Subtractor/Out11: track 33.5 -> 371.7 mm, vias 0 -> 5
- net /Adder Subtractor/Out9: track 39.9 -> 376.1 mm, vias 0 -> 5
- net /Adder Subtractor/Out1: track 65.3 -> 354.8 mm, vias 0 -> 5
- net /Adder Subtractor/Out5: track 52.6 -> 337.4 mm, vias 0 -> 4
- net /Adder Subtractor/Out7: track 46.2 -> 320.3 mm, vias 0 -> 4
- net /Adder Subtractor/Out3: track 58.9 -> 333.0 mm, vias 0 -> 4
- net /Adder Subtractor/Out14: track 49.3 -> 322.8 mm, vias 0 -> 4
- net /Adder Subtractor/Out12: track 62.0 -> 327.2 mm, vias 0 -> 4
- net /Adder Subtractor/Out10: track 74.7 -> 331.7 mm, vias 0 -> 4
- net /Adder Subtractor/Out8: track 87.4 -> 336.1 mm, vias 0 -> 4
- net /Adder Subtractor/Out6: track 74.7 -> 310.7 mm, vias 0 -> 4
- net /Adder Subtractor/Out2: track 100.1 -> 330.7 mm, vias 0 -> 5
- net /Adder Subtractor/Out4: track 87.4 -> 312.6 mm, vias 0 -> 4
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
Commit message: Working towards the connectors
Parts:
- moved U7001 75.7 mm to (62.8, 47.6)
- moved U7002 75.0 mm to (73.0, 48.3)
- moved D8017 72.8 mm to (76.8, 30.3)
- moved R8017 72.8 mm to (80.0, 25.1)
- moved U2001 51.5 mm to (61.0, 64.8)
- moved R2001 50.1 mm to (73.7, 67.3), turned to 180 degrees
- moved R2002 50.1 mm to (73.7, 69.8), turned to 180 degrees
- moved R2003 50.0 mm to (73.7, 72.4), turned to 180 degrees
- moved R2004 50.0 mm to (73.7, 74.9), turned to 180 degrees
- moved R2005 50.0 mm to (73.7, 77.5), turned to 180 degrees
- moved R2006 50.0 mm to (73.7, 80.0), turned to 180 degrees
- moved R2007 49.9 mm to (73.7, 82.5), turned to 180 degrees
- moved R2008 49.9 mm to (73.7, 85.1), turned to 180 degrees
- moved D2008 46.7 mm to (77.5, 85.1)
- moved D2007 46.6 mm to (77.5, 82.5)
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Connections:
- U6001 pad 1: /B3 -> GND
- U6001 pad 12: unconnected-(U6001-Pad12) -> /Barrel Shifter/B3_inv
- U6001 pad 13: GND -> /B3
- U6001 pad 2: /Barrel Shifter/B3_inv -> unconnected-(U6001-Pad2)
- U7001 pad 1: /Enabler/Cycle2 -> GND
- U7001 pad 10: unconnected-(U7001-Pad10) -> Net-(U7001-Pad10)
- U7001 pad 11: GND -> /Enabler/Cycle3
- U7001 pad 12: unconnected-(U7001-Pad12) -> Net-(U7001-Pad12)
- U7001 pad 13: GND -> /Enabler/Cycle2
- U7001 pad 2: Net-(U7001-Pad2) -> unconnected-(U7001-Pad2)
- U7001 pad 3: /Enabler/Cycle3 -> GND
- U7001 pad 4: Net-(U7001-Pad4) -> unconnected-(U7001-Pad4)
- U7002 pad 1: Net-(U7001-Pad2) -> Net-(U7001-Pad12)
- U7002 pad 2: Net-(U7001-Pad4) -> Net-(U7001-Pad10)
- U8001 pad 1: unconnected-(U8001-A->B-Pad1) -> GND
- U8002 pad 1: unconnected-(U8002-A->B-Pad1) -> GND
Routing:
- net /A11: track 190.5 -> 384.2 mm, vias 0 -> 5
- net /A12: track 206.4 -> 392.5 mm, vias 0 -> 5
- net /B0: track 306.8 -> 487.6 mm, vias 0 -> 5
- net /Barrel Shifter/~{Shift}: track 75.5 -> 250.7 mm, vias 0 -> 2
- net /B1: track 320.7 -> 481.4 mm, vias 0 -> 5
- net /Adder Subtractor/~{ADD}: track 51.9 -> 211.2 mm, vias 0 -> 2
- net /Adder Subtractor/~{SUB}: track 18.3 -> 172.6 mm, vias 0 -> 2
- net /A1: track 245.2 -> 384.9 mm, vias 0 -> 5
- net /A0: track 252.1 -> 388.7 mm, vias 0 -> 5
- net /A2: track 266.1 -> 398.2 mm, vias 0 -> 5
- net /Enabler/~{Enable}: track 0.00 -> 127.9 mm, vias 0 -> 3
- net /A4: track 280.1 -> 407.7 mm, vias 0 -> 5
- net /A3: track 266.7 -> 394.4 mm, vias 0 -> 5
- net /A6: track 294.1 -> 417.2 mm, vias 0 -> 5
- net /B2: track 328.3 -> 451.5 mm, vias 0 -> 5
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