File: pcbs/ALU Carrier/output.kicad_sch (KiCad schematic)
At the start: 36 parts, among them U8001 74HC245, U8002 74HC245

Commit message: Routing, routing, routing
Connections:
- net Out0: now also U8001.18 (B0)
- net Out1: now also U8001.17 (B1)
- net Out10: now also U8002.16 (B2)
- net Out11: now also U8002.15 (B3)
- net Out12: now also U8002.14 (B4)
- net Out13: now also U8002.13 (B5)
- net Out14: now also U8002.12 (B6)
- net Out15: now also U8002.11 (B7)
- net Out2: now also U8001.16 (B2)
- net Out3: now also U8001.15 (B3)
- net Out4: now also U8001.14 (B4)
- net Out5: now also U8001.13 (B5)
- net Out6: now also U8001.12 (B6)
- net Out7: now also U8001.11 (B7)
- net Out8: now also U8002.18 (B0)
- net Out9: now also U8002.17 (B1)
- net C8: now reaches U8002.2 (A0)
- net C9: now reaches U8002.3 (A1)
- net C10: now reaches U8002.4 (A2)
- net C11: now reaches U8002.5 (A3)
- net C12: now reaches U8002.6 (A4)
- net C13: now reaches U8002.7 (A5)
- net C14: now reaches U8002.8 (A6)
- net C15: now reaches U8002.9 (A7)
- net C0: now reaches U8001.2 (A0)
- net C1: now reaches U8001.3 (A1)
- net C2: now reaches U8001.4 (A2)
- net C3: now reaches U8001.5 (A3)
- net C4: now reaches U8001.6 (A4)
- net C5: now reaches U8001.7 (A5)
- net C6: now reaches U8001.8 (A6)
- net C7: now reaches U8001.9 (A7)

Commit message: Working towards the connectors
Connections:
- net GND: now also U8001.1 (A->B), U8002.1 (A->B)
Changed lines of the file:
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@@
 	(wire
 		(pts
+			(xy 50.8 63.5) (xy 63.5 63.5)
+		)
+		(stroke
+			(width 0)
+			(type default)
+		)
+	)
+	(wire
+		(pts
 			(xy 119.38 173.99) (xy 127 173.99)
 		)
@@
 	(wire
 		(pts
+			(xy 139.7 63.5) (xy 152.4 63.5)
+		)
+		(stroke
+			(width 0)
+			(type default)
+		)
+	)
+	(wire
+		(pts
 			(xy 134.62 173.99) (xy 139.7 173.99)
 		)
@@
 	(label "Out6"
 		(at 88.9 55.88 0)
+		(fields_autoplaced yes)
 		(effects
 			(font
@@
 	(label "C6"
 		(at 40.64 55.88 0)
+		(fields_autoplaced yes)
 		(effects
 			(font
@@
 	(label "Out7"
 		(at 88.9 58.42 0)
+		(fields_autoplaced yes)
 		(effects
 			(font
@@
 	(label "Out13"
 		(at 177.8 53.34 0)
+		(fields_autoplaced yes)
 		(effects
 			(font
@@
 	(label "Out9"
 		(at 177.8 43.18 0)
+		(fields_autoplaced yes)
 		(effects
 			(font
@@
 	(label "Out10"
 		(at 177.8 45.72 0)
+		(fields_autoplaced yes)
 		(effects
 			(font
@@
 	(label "C15"
 		(at 129.54 58.42 0)
+		(fields_autoplaced yes)
 		(effects
 			(font
@@
 	(label "C14"
 		(at 129.54 55.88 0)
+		(fields_autoplaced yes)
 		(effects
 			(font
@@
 	(label "Out15"
 		(at 177.8 58.42 0)
+		(fields_autoplaced yes)
 		(effects
 			(font
@@
 	(label "C0"
 		(at 40.64 40.64 0)
+		(fields_autoplaced yes)
 		(effects
 			(font
@@
 	(label "Out0"
 		(at 88.9 40.64 0)
+		(fields_autoplaced yes)
 		(effects
 			(font
@@
 	(label "Out3"
 		(at 88.9 48.26 0)
+		(fields_autoplaced yes)
 		(effects
 			(font
@@
 	(label "Out8"
 		(at 177.8 40.64 0)
+		(fields_autoplaced yes)
 		(effects
 			(font
@@
 	(label "C3"
 		(at 40.64 48.26 0)
+		(fields_autoplaced yes)
 		(effects
 			(font
@@
 	(label "Out2"
 		(at 88.9 45.72 0)
+		(fields_autoplaced yes)
 		(effects
 			(font
@@
 	(label "C7"
 		(at 40.64 58.42 0)
+		(fields_autoplaced yes)
 		(effects
 			(font
@@
 	(label "C5"
 		(at 40.64 53.34 0)
+		(fields_autoplaced yes)
 		(effects
 			(font
@@
 	(label "C2"
 		(at 40.64 45.72 0)
+		(fields_autoplaced yes)
 		(effects
 			(font
@@
 	(label "C11"
 		(at 129.54 48.26 0)
+		(fields_autoplaced yes)
 		(effects
 			(font
@@
 	(label "Out14"
 		(at 177.8 55.88 0)
+		(fields_autoplaced yes)
 		(effects
 			(font
@@
 	(label "Out12"
 		(at 177.8 50.8 0)
+		(fields_autoplaced yes)
 		(effects
 			(font
@@
 	(label "C12"
 		(at 129.54 50.8 0)
+		(fields_autoplaced yes)
 		(effects
 			(font
@@
 	(label "C10"
 		(at 129.54 45.72 0)
+		(fields_autoplaced yes)
 		(effects
 			(font
@@
 	(label "C1"
 		(at 40.64 43.18 0)
+		(fields_autoplaced yes)
 		(effects
 			(font
@@
 	(label "C13"
 		(at 129.54 53.34 0)
+		(fields_autoplaced yes)
 		(effects
 			(font
@@
 	(label "Out11"
 		(at 177.8 48.26 0)
+		(fields_autoplaced yes)
 		(effects
 			(font
@@
 	(label "C9"
 		(at 129.54 43.18 0)
+		(fields_autoplaced yes)
 		(effects
 			(font
@@
 	(label "Out5"
 		(at 88.9 53.34 0)
+		(fields_autoplaced yes)
 		(effects
 			(font
@@
 	(label "C4"
 		(at 40.64 50.8 0)
+		(fields_autoplaced yes)
 		(effects
 			(font
@@
 	(label "C8"
 		(at 129.54 40.64 0)
+		(fields_autoplaced yes)
 		(effects
 			(font
@@
 	(label "Out4"
 		(at 88.9 50.8 0)
+		(fields_autoplaced yes)
 		(effects
 			(font
@@
 	(label "Out1"
 		(at 88.9 43.18 0)
+		(fields_autoplaced yes)
 		(effects
 			(font
@@
 	)
 	(symbol
+		(lib_id "power:GND")
+		(at 50.8 63.5 270)
+		(unit 1)
+		(exclude_from_sim no)
+		(in_bom yes)
+		(on_board yes)
+		(dnp no)
+		(fields_autoplaced yes)
+		(property "Reference" "#PWR08008"
+			(at 44.45 63.5 0)
+			(effects
+				(font
+					(size 1.27 1.27)
+				)
+				(hide yes)
+			)
+		)
+		(property "Value" "GND"
+			(at 46.99 63.4999 90)
+			(effects
+				(font
+					(size 1.27 1.27)
+				)
+				(justify right)
+			)
+		)
+		(property "Footprint" ""
+			(at 50.8 63.5 0)
+			(effects
+				(font
+					(size 1.27 1.27)
+				)
+				(hide yes)
+			)
+		)
+		(property "Datasheet" ""
+			(at 50.8 63.5 0)
+			(effects
+				(font
+					(size 1.27 1.27)
+				)
+				(hide yes)
+			)
+		)
+		(property "Description" "Power symbol creates a global label with name \"GND\" , ground"
+			(at 50.8 63.5 0)
+			(effects
+				(font
+					(size 1.27 1.27)
+				)
+				(hide yes)
+			)
+		)
+		(pin "1"
+		)
+		(instances
+			(project ""
+				(path "/2be9e5f9-941e-4c29-a733-4c8d2e8b8610/08238967-dc73-4239-b057-bfde33a1b185"
+					(reference "#PWR08008")
+					(unit 1)
+				)
+			)
+		)
+	)
+	(symbol
 		(lib_id "Device:R")
 		(at 143.51 153.67 270)
@@
 					(unit 1)
 				)
+			)
+		)
+	)
+	(symbol
+		(lib_id "power:GND")
+		(at 139.7 63.5 270)
+		(unit 1)
+		(exclude_from_sim no)
+		(in_bom yes)
+		(on_board yes)
+		(dnp no)
+		(fields_autoplaced yes)
+		(property "Reference" "#PWR08009"
+			(at 133.35 63.5 0)
+			(effects
+				(font
+					(size 1.27 1.27)
+				)
+				(hide yes)
+			)
+		)
+		(property "Value" "GND"
+			(at 135.89 63.4999 90)
+			(effects
+				(font
+					(size 1.27 1.27)
+				)
+				(justify right)
+			)
+		)
+		(property "Footprint" ""
+			(at 139.7 63.5 0)
+			(effects
+				(font
+					(size 1.27 1.27)
+				)
+				(hide yes)
+			)
+		)
+		(property "Datasheet" ""
+			(at 139.7 63.5 0)
+			(effects
+				(font
+					(size 1.27 1.27)
+				)
+				(hide yes)
+			)
+		)
+		(property "Description" "Power symbol creates a global label with name \"GND\" , ground"
+			(at 139.7 63.5 0)
+			(effects
+				(font
+					(size 1.27 1.27)
+				)
+				(hide yes)
+			)
+		)
+		(pin "1"
+		)
+		(instances
+			(project "ALU Carrier"
+				(path "/2be9e5f9-941e-4c29-a733-4c8d2e8b8610/08238967-dc73-4239-b057-bfde33a1b185"
+					(reference "#PWR08009")
+					(unit 1)
+				)
