File: pcbs/ALU Carrier/addsub.kicad_sch (KiCad schematic)
At the start: 2 parts

Commit message: Thinking some more
Connections:
- no-connect marks 28 -> 29
Changed lines of the file:
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@@
+	)
+	(no_connect
+		(at 167.64 119.38)
 	)
 	(no_connect
