File: pcbs/Register File Carrier/enabler.kicad_sch (KiCad schematic)
At the start: 23 parts, among them U3001 74HC14, U3002 74HC08, U3003 74HC138, U3004 74HC08

Commit message: [PCB] Register File Carrier r01 (#21)
Update the Register File Carrier to get the 'enable' logic correct. Had constructed an 'Active High' when 'Active Low' was required.

Also should address #20 , standardising on a single part.
Parts:
- U3003: now left out of the parts list
Connections:
- net GND: now also U3001.1
- net ~{Enable}: now also U3002.8; no longer U3001.2
- no-connect marks 5 -> 6
Other:
- moved on the sheet: U3001A
Changed lines of the file:
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@@
 	(generator_version "8.0")
 	(paper "A4")
+	(title_block
+		(rev "1")
+	)
 	(junction
 		(at 215.9 66.04)
@@
 	)
 	(junction
+		(at 255.27 137.16)
+		(diameter 0)
+		(color 0 0 0 0)
+	)
+	(junction
 		(at 44.45 160.02)
 		(diameter 0)
@@
 	)
 	(junction
+		(at 149.86 55.88)
+		(diameter 0)
+		(color 0 0 0 0)
+	)
+	(junction
 		(at 22.86 128.27)
 		(diameter 0)
@@
 	)
 	(junction
-		(at 149.86 55.88)
-		(diameter 0)
-		(color 0 0 0 0)
-	)
-	(junction
 		(at 203.2 66.04)
 		(diameter 0)
@@
 	)
 	(no_connect
+		(at 275.59 121.92)
+	)
+	(no_connect
 		(at 40.64 109.22)
 	)
@@
 	(wire
 		(pts
-			(xy 147.32 55.88) (xy 149.86 55.88)
-		)
-		(stroke
-			(width 0)
-			(type default)
-		)
-	)
-	(wire
-		(pts
 			(xy 254 41.91) (xy 254 44.45)
 		)
@@
 	(wire
 		(pts
-			(xy 128.27 55.88) (xy 132.08 55.88)
-		)
-		(stroke
-			(width 0)
-			(type default)
-		)
-	)
-	(wire
-		(pts
 			(xy 57.15 83.82) (xy 67.31 83.82)
 		)
@@
 	(wire
 		(pts
+			(xy 255.27 121.92) (xy 260.35 121.92)
+		)
+		(stroke
+			(width 0)
+			(type default)
+		)
+	)
+	(wire
+		(pts
 			(xy 80.01 100.33) (xy 80.01 132.08)
 		)
@@
 	(wire
 		(pts
+			(xy 255.27 137.16) (xy 255.27 121.92)
+		)
+		(stroke
+			(width 0)
+			(type default)
+		)
+	)
+	(wire
+		(pts
 			(xy 130.81 119.38) (xy 133.35 119.38)
 		)
@@
 		(pts
 			(xy 228.6 41.91) (xy 228.6 44.45)
+		)
+		(stroke
+			(width 0)
+			(type default)
+		)
+	)
+	(wire
+		(pts
+			(xy 128.27 55.88) (xy 149.86 55.88)
 		)
 		(stroke
@@
 		(unit 1)
 		(exclude_from_sim no)
-		(in_bom yes)
+		(in_bom no)
 		(on_board yes)
 		(dnp no)
@@
 	(symbol
 		(lib_id "74xx:74HC14")
-		(at 139.7 55.88 0)
+		(at 267.97 121.92 0)
 		(unit 1)
 		(exclude_from_sim no)
@@
 		(fields_autoplaced yes)
 		(property "Reference" "U3001"
-			(at 139.7 46.99 0)
+			(at 267.97 113.03 0)
 			(effects
 				(font
@@
 		)
 		(property "Value" "74HC14"
-			(at 139.7 49.53 0)
+			(at 267.97 115.57 0)
 			(effects
 				(font
@@
 		)
 		(property "Footprint" "Package_SO:SOIC-14_3.9x8.7mm_P1.27mm"
-			(at 139.7 55.88 0)
+			(at 267.97 121.92 0)
 			(effects
 				(font
@@
 		)
 		(property "Datasheet" "https://www.lcsc.com/datasheet/lcsc_datasheet_2407241044_Nexperia-74HC14D-653_C5605.pdf"
-			(at 139.7 55.88 0)
+			(at 267.97 121.92 0)
 			(effects
 				(font
@@
 		)
 		(property "Description" "Hex inverter schmitt trigger"
-			(at 139.7 55.88 0)
+			(at 267.97 121.92 0)
 			(effects
 				(font
@@
 		)
 		(property "LCSC" "C5605"
-			(at 139.7 55.88 0)
-			(effects
-				(font
+			(at 267.97 121.92 0)
+			(effects
+				(font
