File: pcbs/Program Counter/BufferLR.kicad_sch (KiCad schematic)
At the start: 2 parts, among them U5001 74HC245, U5002 74HC245

Commit message: Some more LEDs and silkscreening
Parts:
- added D5001: Blue, LED_SMD:LED_0603_1608Metric, symbol Device:LED
- added R5001: 4k7, Resistor_SMD:R_0603_1608Metric, symbol Device:R
Connections:
- net +5V: now also D5001.2 (A)
- net ~{Enable}: now also R5001.1
- new net: D5001.1 (K), R5001.2
