File: pcbs/Program Counter/Program Counter.kicad_sch (KiCad schematic)
At the start: 2 parts, among them J1001 Conn_02x20_Odd_Even, J1002 Conn_02x20_Odd_Even

Commit message: Resizing sheet
Other:
- title: (none) -> Program Counter
Changed lines of the file:
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@@
 	(generator "eeschema")
 	(generator_version "8.0")
-	(paper "A4")
+	(paper "A3")
+	(title_block
+		(title "Program Counter")
+	)
 	(junction
 		(at 43.18 39.37)

Commit message: Starting to think about connections
Parts:
- added J1003, J1004: ~, BoardEdgeConnectors:TE-5530843-4-Mount, symbol BoardEdgeConnectors:TE-5530843-4
Connections:
- net +5V: now also J1003.B1, J1004.B1
- net Cycle4: now also J1003.B11
- net GND: now also J1003.A22, J1003.B20, J1004.A22, J1004.B20
- net Ao0 renamed A0
- net Ao1 renamed A1
- net Ao10 renamed A10
- net Ao11 renamed A11
- net Ao12 renamed A12
- net Ao13 renamed A13
- net Ao14 renamed A14
- net Ao15 renamed A15
- net Ao2 renamed A2
- net Ao3 renamed A3
- net Ao4 renamed A4
- net Ao5 renamed A5
- net Ao6 renamed A6
- net Ao7 renamed A7
- net Ao8 renamed A8
- net Ao9 renamed A9
- net Bo0 renamed B0
- net Bo1 renamed B1
- net Bo10 renamed B10
- net Bo11 renamed B11
- net Bo12 renamed B12
- net Bo13 renamed B13
- net Bo14 renamed B14
- net Bo15 renamed B15
- net Bo2 renamed B2
- net Bo3 renamed B3
- net Bo4 renamed B4
- net Bo5 renamed B5
- net Bo6 renamed B6
- net Bo7 renamed B7
- net Bo8 renamed B8
- net Bo9 renamed B9
- new net Inc.Out0: J1004.A2
- new net Inc.Out1: J1004.B2
- new net Inc.Out10: J1004.A7
- new net Inc.Out11: J1004.B7
- new net Inc.Out12: J1004.A8
- new net Inc.Out13: J1004.B8
- new net Inc.Out14: J1004.A9
- new net Inc.Out15: J1004.B9
- new net Inc.Out2: J1004.A3
- new net Inc.Out3: J1004.B3
- new net Inc.Out4: J1004.A4
- new net Inc.Out5: J1004.B4
- new net Inc.Out6: J1004.A5
- new net Inc.Out7: J1004.B5
- new net Inc.Out8: J1004.A6
- new net Inc.Out9: J1004.B6
- new net Increment0: J1004.A10
- new net Increment1: J1004.B10
- new net Increment2: J1004.A11
- new net Increment3: J1004.B11
- new net PC.In0: J1003.A2
- new net PC.In1: J1003.B2
- new net PC.In10: J1003.A7
- new net PC.In11: J1003.B7
- new net PC.In12: J1003.A8
- new net PC.In13: J1003.B8
- new net PC.In14: J1003.A9
- new net PC.In15: J1003.B9
- new net PC.In2: J1003.A3
- new net PC.In3: J1003.B3
- new net PC.In4: J1003.A4
- new net PC.In5: J1003.B4
- new net PC.In6: J1003.A5
- new net PC.In7: J1003.B5
- new net PC.In8: J1003.A6
- new net PC.In9: J1003.B6
- new net PC.Out0: J1003.A12, J1004.A12
- new net PC.Out1: J1003.B12, J1004.B12
- new net PC.Out10: J1003.A17, J1004.A17
- new net PC.Out11: J1003.B17, J1004.B17
- new net PC.Out12: J1003.A18, J1004.A18
- new net PC.Out13: J1003.B18, J1004.B18
- new net PC.Out14: J1003.A19, J1004.A19
- new net PC.Out15: J1003.B19, J1004.B19
- new net PC.Out2: J1003.A13, J1004.A13
- new net PC.Out3: J1003.B13, J1004.B13
- new net PC.Out4: J1003.A14, J1004.A14
- new net PC.Out5: J1003.B14, J1004.B14
- new net PC.Out6: J1003.A15, J1004.A15
- new net PC.Out7: J1003.B15, J1004.B15
- new net PC.Out8: J1003.A16, J1004.A16
- new net PC.Out9: J1003.B16, J1004.B16
- new net ~{RESET}: J1003.B10
- no-connect marks 5 -> 20
Other:
- added sheet BranchZero Buffer (BufferLR.kicad_sch)
- added sheet Increment Buffer (BufferRL.kicad_sch)
- added sheet Instruction Cycle Buffer (BufferRL.kicad_sch)
- added sheet LoadPC Buffer (BufferRL.kicad_sch)

Commit message: Some preliminary routing
Connections:
- no-connect marks 20 -> 17
Changed lines of the file:
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@@
-	)
-	(no_connect
-		(at 260.35 96.52)
 	)
 	(no_connect
@@
 	)
 	(no_connect
-		(at 289.56 96.52)
-	)
-	(no_connect
-		(at 260.35 93.98)
-	)
-	(no_connect

Commit message: Thinking about more circuitry
Other:
- added sheet Enabler (enabler.kicad_sch)
Changed lines of the file:
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@@
 		)
 	)
+	(bus
+		(pts
+			(xy 76.2 175.26) (xy 86.36 175.26)
+		)
+		(stroke
+			(width 0)
+			(type default)
+		)
+	)
 	(wire
 		(pts
@@
 		)
 	)
+	(bus
+		(pts
+			(xy 76.2 171.45) (xy 86.36 171.45)
+		)
+		(stroke
+			(width 0)
+			(type default)
+		)
+	)
 	(wire
 		(pts
@@
 		)
 	)
+	(label "Cycle[0..4]"
+		(at 76.2 175.26 180)
+		(fields_autoplaced yes)
+		(effects
+			(font
+				(size 1.27 1.27)
+			)
+			(justify right bottom)
+		)
+	)
 	(label "A4"
 		(at 26.67 46.99 180)
@@
 		)
 	)
+	(label "I[0..3]"
+		(at 76.2 171.45 180)
+		(fields_autoplaced yes)
+		(effects
+			(font
+				(size 1.27 1.27)
+			)
+			(justify right bottom)
+		)
+	)
 	(label "PC.Out14"
 		(at 149.86 115.57 180)
@@
 				)
 			)
+		)
+	)
+	(sheet
+		(at 86.36 167.64)
+		(size 39.37 25.4)
+		(fields_autoplaced yes)
+		(stroke
+			(width 0.1524)
+			(type solid)
+		)
+		(fill
+			(color 0 0 0 0.0000)
+		)
+		(property "Sheetname" "Enabler"
+			(at 86.36 166.9284 0)
+			(effects
+				(font
+					(size 1.27 1.27)
+				)
+				(justify left bottom)
+			)
+		)
+		(property "Sheetfile" "enabler.kicad_sch"
+			(at 86.36 193.6246 0)
+			(effects
+				(font
+					(size 1.27 1.27)
+				)
+				(justify left top)
+			)
+		)
+		(pin "~{ExecCycle}" output
+			(at 125.73 173.99 0)
+			(effects
+				(font
+					(size 1.27 1.27)
+				)
+				(justify right)
+			)
+		)
+		(pin "I[0..3]" input
+			(at 86.36 171.45 180)
+			(effects
+				(font
+					(size 1.27 1.27)
+				)
+				(justify left)
+			)
+		)
+		(pin "~{Halt}" output
+			(at 125.73 177.8 0)
+			(effects
+				(font
+					(size 1.27 1.27)
+				)
+				(justify right)
+			)
+		)
+		(pin "~{LoadPC}" output
+			(at 125.73 181.61 0)
+			(effects
+				(font
+					(size 1.27 1.27)
+				)
+				(justify right)
+			)
+		)
+		(pin "Cycle[0..4]" input
+			(at 86.36 175.26 180)
+			(effects
+				(font
+					(size 1.27 1.27)
+				)
+				(justify left)
+			)
+		)
+		(pin "~{InstrCycle}" output
+			(at 125.73 185.42 0)
+			(effects
+				(font
+					(size 1.27 1.27)
+				)
+				(justify right)
+			)
+		)
+		(instances
+			(project "Program Counter"
+				(path "/6d6da32b-3371-451c-a9b1-ca4368fb7dac"
+					(page "6")
+				)
+			)

Commit message: More schematic, more layout
Connections:
- net Cycle4: no longer J1003.B11
- new net ClockPC: J1003.B11
Other:
- sheet Enabler ports: added B[0..15], CLK_{PC}, ~{DoBranch}, ~{NormalUpdate}; removed none

Commit message: Routing.... should be silkscreen and final adjustments next
Connections:
- net RESET is gone; now on net ~{RESET}: J1001.39 (Pin_39)
- no-connect marks 17 -> 33
Other:
- sheet Enabler ports: added none; removed ~{ExecCycle}
Changed lines of the file:
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@@
 	)
 	(no_connect
+		(at 26.67 139.7)
+	)
+	(no_connect
 		(at 41.91 85.09)
 	)
 	(no_connect
+		(at 26.67 137.16)
+	)
+	(no_connect
+		(at 260.35 93.98)
+	)
+	(no_connect
+		(at 44.45 132.08)
+	)
+	(no_connect
 		(at 29.21 85.09)
 	)
@@
 	)
 	(no_connect
+		(at 44.45 137.16)
+	)
+	(no_connect
+		(at 44.45 142.24)
+	)
+	(no_connect
 		(at 153.67 69.85)
 	)
 	(no_connect
+		(at 44.45 139.7)
+	)
+	(no_connect
 		(at 264.16 71.12)
 	)
@@
 	)
 	(no_connect
+		(at 26.67 129.54)
+	)
+	(no_connect
 		(at 264.16 119.38)
 	)
 	(no_connect
+		(at 44.45 87.63)
+	)
+	(no_connect
 		(at 153.67 118.11)
 	)
 	(no_connect
+		(at 260.35 96.52)
+	)
+	(no_connect
+		(at 26.67 134.62)
+	)
+	(no_connect
+		(at 289.56 96.52)
+	)
+	(no_connect
 		(at 173.99 123.19)
 	)
 	(no_connect
+		(at 44.45 134.62)
+	)
+	(no_connect
+		(at 44.45 129.54)
+	)
+	(no_connect
+		(at 26.67 142.24)
+	)
+	(no_connect
+		(at 26.67 132.08)
+	)
+	(no_connect
 		(at 153.67 120.65)
 	)
@@
 		)
 	)
-	(label "RESET"
+	(label "~{RESET}"
 		(at 26.67 87.63 180)
 		(fields_autoplaced yes)
@@
 			)
 		)
-		(pin "~{ExecCycle}" output
-			(at 125.73 173.99 0)
-			(effects
-				(font
-					(size 1.27 1.27)
-				)
-				(justify right)
-			)
-		)

Commit message: Prepping for final check
Parts:
- added H1001, H1002, H1003, H1004: MountingHole, MountingHole:MountingHole_2.7mm_M2.5_ISO7380, symbol Mechanical:MountingHole

Commit message: Think I had something backwards.... will recheck after
Connections:
- net Increment0 is gone; now on net GND: J1004.A10
- net Increment2 is gone; now on net GND: J1004.A11
- net Increment3 is gone; now on net GND: J1004.B11
- no-connect marks 33 -> 30
Changed lines of the file:
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@@
 	)
 	(no_connect
-		(at 260.35 93.98)
-	)
-	(no_connect
 		(at 44.45 132.08)
 	)
@@
 	)
 	(no_connect
-		(at 260.35 96.52)
-	)
-	(no_connect
 		(at 26.67 134.62)
 	)
 	(no_connect
-		(at 289.56 96.52)
-	)
-	(no_connect
 		(at 173.99 123.19)
 	)
@@
 	(wire
 		(pts
-			(xy 284.48 96.52) (xy 289.56 96.52)
+			(xy 284.48 96.52) (xy 307.34 96.52)
 		)
 		(stroke
@@
 	(wire
 		(pts
+			(xy 245.11 93.98) (xy 264.16 93.98)
+		)
+		(stroke
+			(width 0)
+			(type default)
+		)
+	)
+	(wire
+		(pts
+			(xy 245.11 96.52) (xy 264.16 96.52)
+		)
+		(stroke
+			(width 0)
+			(type default)
+		)
+	)
+	(wire
+		(pts
 			(xy 27.94 152.4) (xy 29.21 152.4)
 		)
@@
 	(wire
 		(pts
-			(xy 260.35 93.98) (xy 264.16 93.98)
-		)
-		(stroke
-			(width 0)
-			(type default)
-		)
-	)
-	(wire
-		(pts
 			(xy 26.67 111.76) (xy 29.21 111.76)
 		)
@@
 		)
 	)
-	(wire
-		(pts
-			(xy 260.35 96.52) (xy 264.16 96.52)
-		)
-		(stroke
-			(width 0)
-			(type default)
-		)
-	)
 	(bus
 		(pts
@@
 		)
 	)
-	(label "Increment2"
-		(at 260.35 96.52 180)
-		(fields_autoplaced yes)
-		(effects
-			(font
-				(size 1.27 1.27)
-			)
-			(justify right bottom)
-		)
-	)
 	(label "~{InstrCycle}"
 		(at 196.85 146.05 180)
@@
 		)
 	)
-	(label "Increment0"
-		(at 260.35 93.98 180)
-		(fields_autoplaced yes)
-		(effects
-			(font
-				(size 1.27 1.27)
-			)
-			(justify right bottom)
-		)
-	)
 	(label "~{DoBranch}"
 		(at 196.85 198.12 180)
@@
 		)
 	)
-	(label "Increment3"
-		(at 289.56 96.52 0)
-		(fields_autoplaced yes)
-		(effects
-			(font
-				(size 1.27 1.27)
-			)
-			(justify left bottom)
-		)
-	)
 	(label "B4"
 		(at 26.67 67.31 180)
@@
 	)
 	(symbol
+		(lib_id "power:GND")
+		(at 245.11 96.52 0)
+		(unit 1)
+		(exclude_from_sim no)
+		(in_bom yes)
+		(on_board yes)
+		(dnp no)
+		(fields_autoplaced yes)
+		(property "Reference" "#PWR01011"
+			(at 245.11 102.87 0)
+			(effects
+				(font
+					(size 1.27 1.27)
+				)
+				(hide yes)
+			)
+		)
+		(property "Value" "GND"
+			(at 245.11 101.6 0)
+			(effects
+				(font
+					(size 1.27 1.27)
+				)
+			)
+		)
+		(property "Footprint" ""
+			(at 245.11 96.52 0)
+			(effects
+				(font
+					(size 1.27 1.27)
+				)
+				(hide yes)
+			)
+		)
+		(property "Datasheet" ""
+			(at 245.11 96.52 0)
+			(effects
+				(font
+					(size 1.27 1.27)
+				)
+				(hide yes)
+			)
+		)
+		(property "Description" "Power symbol creates a global label with name \"GND\" , ground"
+			(at 245.11 96.52 0)
+			(effects
+				(font
+					(size 1.27 1.27)
+				)
+				(hide yes)
+			)
+		)
+		(pin "1"
+		)
+		(instances
+			(project ""
+				(path "/6d6da32b-3371-451c-a9b1-ca4368fb7dac"
+					(reference "#PWR01011")
+					(unit 1)
+				)
+			)
+		)
+	)
+	(symbol
 		(lib_id "Connector_Generic:Conn_02x20_Odd_Even")
 		(at 34.29 62.23 0)
@@
 	(symbol
 		(lib_id "power:GND")
+		(at 245.11 93.98 180)
+		(unit 1)
+		(exclude_from_sim no)
+		(in_bom yes)
+		(on_board yes)
+		(dnp no)
+		(fields_autoplaced yes)
+		(property "Reference" "#PWR01012"
+			(at 245.11 87.63 0)
+			(effects
+				(font
+					(size 1.27 1.27)
+				)
+				(hide yes)
+			)
+		)
+		(property "Value" "GND"
+			(at 245.11 88.9 0)
+			(effects
+				(font
+					(size 1.27 1.27)
+				)
+			)
+		)
+		(property "Footprint" ""
+			(at 245.11 93.98 0)
+			(effects
+				(font
+					(size 1.27 1.27)
+				)
+				(hide yes)
+			)
+		)
+		(property "Datasheet" ""
+			(at 245.11 93.98 0)
+			(effects
+				(font
+					(size 1.27 1.27)
+				)
+				(hide yes)
+			)
+		)
+		(property "Description" "Power symbol creates a global label with name \"GND\" , ground"
+			(at 245.11 93.98 0)
+			(effects
+				(font
+					(size 1.27 1.27)
+				)
+				(hide yes)
+			)
+		)
+		(pin "1"
+		)
+		(instances
+			(project ""
+				(path "/6d6da32b-3371-451c-a9b1-ca4368fb7dac"
+					(reference "#PWR01012")
+					(unit 1)
+				)
+			)
+		)
+	)
+	(symbol
+		(lib_id "power:GND")
 		(at 44.45 152.4 90)
 		(unit 1)
@@
 					(unit 1)
 				)
+			)
+		)
+	)
+	(symbol
+		(lib_id "power:GND")
+		(at 307.34 96.52 0)
+		(unit 1)
+		(exclude_from_sim no)
+		(in_bom yes)
+		(on_board yes)
+		(dnp no)
+		(fields_autoplaced yes)
+		(property "Reference" "#PWR01013"
+			(at 307.34 102.87 0)
+			(effects
+				(font
+					(size 1.27 1.27)
+				)
+				(hide yes)
+			)
+		)
+		(property "Value" "GND"
+			(at 307.34 101.6 0)
+			(effects
+				(font
+					(size 1.27 1.27)
+				)
+			)
+		)
+		(property "Footprint" ""
+			(at 307.34 96.52 0)
+			(effects
+				(font
+					(size 1.27 1.27)
+				)
+				(hide yes)
+			)
+		)
+		(property "Datasheet" ""
+			(at 307.34 96.52 0)
+			(effects
+				(font
+					(size 1.27 1.27)
+				)
+				(hide yes)
+			)
+		)
+		(property "Description" "Power symbol creates a global label with name \"GND\" , ground"
+			(at 307.34 96.52 0)
+			(effects
+				(font
+					(size 1.27 1.27)
+				)
+				(hide yes)
+			)
+		)
+		(pin "1"
+		)
+		(instances
+			(project ""
+				(path "/6d6da32b-3371-451c-a9b1-ca4368fb7dac"
+					(reference "#PWR01013")
+					(unit 1)
+				)
