File: pcbs/Program Counter/enabler.kicad_sch (KiCad schematic)
At the start: 23 parts, among them U6001 74HC14, U6002 74HC08, U6003 74HC08, U6004 74HC138

Commit message: More schematic, more layout
Parts:
- added U6005: 74HC14, Package_SO:SOIC-14_3.9x8.7mm_P1.27mm, symbol 74xx:74HC14
Connections:
- net +5V: now also U6005.14 (VCC)
- net Cycle4: now also U6003.4, U6003.5
- net GND: now also U6002.10, U6002.4, U6002.5, U6002.9, U6005.11, U6005.13, U6005.7 (GND), U6005.9; no longer U6003.4, U6003.5
- net ~{BranchZero}: now also U6005.3
- net CLK_{PC}: now reaches U6003.6
- net at U6002.8: no longer U6002.5
- net ~{DoBranch}: now reaches U6002.11
- net ~{DoBranch}: now also U6005.5; no longer U6002.4
- net at U6002.12: now also U6005.4
- net at U6002.13: now also U6005.2
- new net B Bus Check/B_{Any}: U6005.1
- new net ~{NormalUpdate}: U6005.6
- no-connect marks 6 -> 8
Other:
- added sheet B Bus Check (bbuscheck.kicad_sch)
- moved on the sheet: D6001, R6001, U6001B, U6002A, U6002B, U6002C, U6002D, U6003B, U6004

Commit message: Roughing out the control logic routing
Parts:
- removed U6002: 74HC08, Package_SO:SOIC-14_3.9x8.7mm_P1.27mm, symbol 74xx:74LS08
- added D6010: Blue, LED_SMD:LED_0603_1608Metric, symbol Device:LED
- added R6010: 4k7, Resistor_SMD:R_0603_1608Metric, symbol Device:R
- renumbered U6003 to U6002, U6005 to U6003
Connections:
- net +5V: now also D6010.2 (A)
- net CLK_{PC}: now also U6001.8; no longer U6002.6
- net Cycle0: now also U6001.1; no longer U6001.5
- net Cycle1: now also U6001.3; no longer U6001.1
- net Cycle2: now also U6001.5; no longer U6001.11
- net Cycle3: now also U6001.13; no longer U6001.9
- net Cycle4: now also U6001.11; no longer U6001.13, U6002.4, U6002.5
- net GND: now also U6003.5; no longer U6001.3, U6003.9
- net ~{DoBranch}: now also U6002.6, U6003.9; no longer U6003.5
- net ~{InstrCycle}: now also R6010.1
- net ~{NormalUpdate}: now also U6003.8; no longer U6003.6
- net at U6001.12: now also U6002.12; no longer U6002.10
- net at U6001.10: now also U6001.9, U6002.10; no longer U6002.12
- net at U6002.13: now also U6001.6; no longer U6001.8
- net at U6002.1: now also U6001.4; no longer U6001.6
- net at U6003.4: now also U6002.5
- net at U6003.2: now also U6002.4
- new net: D6010.1 (K), R6010.2
Other:
- moved on the sheet: U6001A, U6001B, U6001C, U6001D, U6001E, U6001F, U6002B, U6003C, U6003D

Commit message: Routing.... should be silkscreen and final adjustments next
Parts:
- added D6011: Blue, LED_SMD:LED_0603_1608Metric, symbol Device:LED
- added R6011: 4k7, Resistor_SMD:R_0603_1608Metric, symbol Device:R
Connections:
- net +5V: now also D6011.2 (A)
- net ~{B_{any}}: now reaches U6002.4, U6003.2
- net ~{B_{any}}: now also R6011.1
- new net: D6011.1 (K), R6011.2
- no-connect marks 8 -> 3

Commit message: Think I had something backwards.... will recheck after
Connections:
- net ~{DoBranch}: now also U6003.8; no longer U6002.6, U6003.9
- net ~{NormalUpdate}: now also U6002.6, U6003.9; no longer U6003.8
Changed lines of the file:
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@@
-	)
-	(junction
-		(at 104.14 182.88)
-		(diameter 0)
-		(color 0 0 0 0)
 	)
 	(junction
@@
 	(wire
 		(pts
-			(xy 104.14 182.88) (xy 128.27 182.88)
-		)
-		(stroke
-			(width 0)
-			(type default)
-		)
-	)
-	(wire
-		(pts
 			(xy 57.15 209.55) (xy 57.15 210.82)
 		)
@@
 	(wire
 		(pts
-			(xy 80.01 182.88) (xy 104.14 182.88)
+			(xy 80.01 182.88) (xy 128.27 182.88)
 		)
 		(stroke
@@
 		(pts
 			(xy 92.71 88.9) (xy 102.87 88.9)
-		)
-		(stroke
-			(width 0)
-			(type default)
-		)
-	)
-	(wire
-		(pts
-			(xy 104.14 182.88) (xy 104.14 185.42)
 		)
 		(stroke
@@
 	(hierarchical_label "~{NormalUpdate}"
 		(shape output)
-		(at 350.52 143.51 0)
+		(at 350.52 160.02 0)
 		(fields_autoplaced yes)
 		(effects
@@
 	(hierarchical_label "~{DoBranch}"
 		(shape output)
-		(at 350.52 160.02 0)
-		(fields_autoplaced yes)
-		(effects
+		(at 350.52 143.51 0)
+		(fields_autoplaced yes)
+		(effects
