File: pcbs/SlothPU Backplane/SlothPU Backplane.kicad_sch (KiCad schematic)
At the start: 17 parts, among them J1001 Conn_02x20_Odd_Even, J1002 Conn_02x20_Odd_Even, J1003 Conn_02x20_Odd_Even, J1004 Conn_02x20_Odd_Even, J1005 Conn_02x20_Odd_Even, J1006 Conn_02x20_Odd_Even, J1007 Conn_02x20_Odd_Even, J1008 Conn_02x20_Odd_Even, J1009 Conn_02x20_Odd_Even, J1010 Conn_02x20_Odd_Even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

Commit message: Routing
Parts:
- removed J1005, J1006, J1009, J1010: Conn_02x20_Odd_Even, Connector_PinHeader_2.54mm:PinHeader_2x20_P2.54mm_Vertical, symbol Connector_Generic:Conn_02x20_Odd_Even
- added J1010: Barrel_Jack_Switch, Connector_BarrelJack:BarrelJack_Horizontal, symbol Connector:Barrel_Jack_Switch
- renumbered J1007 to J1005, J1008 to J1006, J1011 to J1007, J1012 to J1008, J1013 to J1009
Connections:
- net +5V: now also J1010.1
- net GND: now also J1010.2
- no-connect marks 31 -> 22
Other:
- moved on the sheet: J1005, J1006, J1007, J1008, J1009

Commit message: Refinements
Parts:
- added C1001, C1002: 10u, Capacitor_THT:CP_Radial_D4.0mm_P1.50mm, symbol Device:C_Polarized_Small
Connections:
- net +5V: now also C1001.1, C1002.1
- net GND: now also C1001.2, C1002.2
