File: pcbs/SlothPU Backplane/SlothPU Backplane.kicad_pcb (KiCad board)
At the start: 2 copper layers, 17 parts, among them J1001 Conn_02x20_Odd_Even, J1002 Conn_02x20_Odd_Even, J1003 Conn_02x20_Odd_Even, J1004 Conn_02x20_Odd_Even, J1005 Conn_02x20_Odd_Even, J1006 Conn_02x20_Odd_Even, J1007 Conn_02x20_Odd_Even, J1008 Conn_02x20_Odd_Even, J1009 Conn_02x20_Odd_Even, J1010 Conn_02x20_Odd_Even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

Commit message: Routing
Parts:
- removed the J1005 at (355.6, 63.5)
- removed the J1006 at (279.4, 63.5)
- removed the J1009 at (358.1, 215.9)
- J1010: value Conn_02x20_Odd_Even -> Barrel_Jack_Switch; footprint Connector_PinHeader_2.54mm:PinHeader_2x20_P2.54mm_Vertical -> Connector_BarrelJack:BarrelJack_Horizontal
- moved H1004 265.2 mm to (218.4, 231.1)
- moved H1002 205.7 mm to (218.4, 50.8)
- moved H1003 177.5 mm to (50.8, 231.1)
- moved J1007 165.1 mm to (215.9, 74.9)
- moved J1008 165.1 mm to (215.9, 151.1)
- moved J1010 102.8 mm to (213.4, 137.2), turned to 180 degrees
- moved J1009 93.9 mm to (55.9, 138.4)
- moved H1001 38.4 mm to (50.8, 50.8)
- moved J1005 12.8 mm to (191.8, 228.6)
- moved J1006 12.8 mm to (115.6, 228.6)
- moved J1003 12.7 mm to (190.5, 50.8)
- moved J1004 12.7 mm to (114.3, 50.8)
- renumbered J1007 to J1005, J1008 to J1006, J1011 to J1007, J1012 to J1008, J1013 to J1009
Connections:
- J1010 pad 1: /C0 -> +5V
- J1010 pad 2: /C1 -> GND
- J1010 pad 3: /C2 -> unconnected-(J1010-Pad3)
Routing:
- net /I8: track 0.00 -> 344.0 mm, vias 0 -> 1
- net /I6: track 0.00 -> 344.0 mm, vias 0 -> 1
- net /I4: track 0.00 -> 344.0 mm, vias 0 -> 1
- net /I2: track 0.00 -> 344.0 mm, vias 0 -> 1
- net /I14: track 0.00 -> 344.0 mm, vias 0 -> 1
- net /I13: track 0.00 -> 344.0 mm, vias 0 -> 1
- net /I12: track 0.00 -> 344.0 mm, vias 0 -> 1
- net /I10: track 0.00 -> 344.0 mm, vias 0 -> 1
- net /I0: track 0.00 -> 344.0 mm, vias 0 -> 1
- net /C8: track 0.00 -> 344.0 mm, vias 0 -> 1
- net /C6: track 0.00 -> 344.0 mm, vias 0 -> 1
- net /C14: track 0.00 -> 344.0 mm, vias 0 -> 1
- net /C10: track 0.00 -> 344.0 mm, vias 0 -> 1
- net /B8: track 0.00 -> 344.0 mm, vias 0 -> 1
- net /B6: track 0.00 -> 344.0 mm, vias 0 -> 1
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- added copper zone on B.Cu, net +5V
- added copper zone on F.Cu, net GND
Other:
- board outline added: 182.9 x 195.6 mm

Commit message: Adding silkscreen
Other:
- board text added: "+5V"
- board text added: "GND"
- board text added: "SlothPU16 Backplane"
Changed lines of the file:
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@@
 		(tags "Power Jack")
 		(property "Reference" "J1010"
-			(at -8.45 5.75 360)
+			(at -8.45 5.75 0)
 			(layer "F.SilkS")
 			(effects
@@
 		)
 		(property "Value" "Barrel_Jack_Switch"
-			(at -6.2 -5.5 360)
+			(at -6.2 -5.5 0)
 			(layer "F.Fab")
 			(effects
@@
 		)
 		(fp_text user "${REFERENCE}"
-			(at -3 -2.95 360)
+			(at -3 -2.95 0)
 			(layer "F.Fab")
 			(effects
@@
 		(layer "Edge.Cuts")
 	)
+	(gr_text "+5V"
+		(at 190.5 48.895 -90)
+		(layer "F.SilkS")
+		(effects
+			(font
+				(size 1.2192 1.2192)
+				(thickness 0.1524)
+			)
+			(justify right)
+		)
+	)
+	(gr_text "+5V"
+		(at 55.245 76.2 0)
+		(layer "F.SilkS")
+		(effects
+			(font
+				(size 1.2192 1.2192)
+				(thickness 0.1524)
+			)
+			(justify left)
+		)
+	)
+	(gr_text "+5V"
+		(at 191.77 226.695 -90)
+		(layer "F.SilkS")
+		(effects
+			(font
+				(size 1.2192 1.2192)
+				(thickness 0.1524)
+			)
+			(justify right)
+		)
+	)
+	(gr_text "+5V"
+		(at 213.995 74.93 0)
+		(layer "F.SilkS")
+		(effects
+			(font
+				(size 1.2192 1.2192)
+				(thickness 0.1524)
+			)
+			(justify right)
+		)
+	)
+	(gr_text "+5V"
+		(at 220.345 74.93 0)
+		(layer "F.SilkS")
+		(effects
+			(font
+				(size 1.2192 1.2192)
+				(thickness 0.1524)
+			)
+			(justify left)
+		)
+	)
+	(gr_text "SlothPU16 Backplane"
+		(at 107.315 121.92 0)
+		(layer "F.SilkS")
+		(effects
+			(font
+				(size 3.2512 3.2512)
+				(thickness 0.4064)
+			)
+			(justify left bottom)
+		)
+	)
+	(gr_text "+5V"
+		(at 190.5 55.245 -90)
+		(layer "F.SilkS")
+		(effects
+			(font
+				(size 1.2192 1.2192)
+				(thickness 0.1524)
+			)
+			(justify left)
+		)
+	)
+	(gr_text "GND"
+		(at 55.245 200.66 0)
+		(layer "F.SilkS")
+		(effects
+			(font
+				(size 1.2192 1.2192)
+				(thickness 0.1524)
+			)
+			(justify left)
+		)
+	)
+	(gr_text "GND"
+		(at 66.04 55.245 -90)
+		(layer "F.SilkS")
+		(effects
+			(font
+				(size 1.2192 1.2192)
+				(thickness 0.1524)
+			)
+			(justify left)
+		)
+	)
+	(gr_text "GND"
+		(at 67.31 233.045 -90)
+		(layer "F.SilkS")
+		(effects
+			(font
+				(size 1.2192 1.2192)
+				(thickness 0.1524)
+			)
+			(justify left)
+		)
+	)
+	(gr_text "GND"
+		(at 220.345 199.39 0)
+		(layer "F.SilkS")
+		(effects
+			(font
+				(size 1.2192 1.2192)
+				(thickness 0.1524)
+			)
+			(justify left)
+		)
+	)
+	(gr_text "GND"
+		(at 213.995 199.39 0)
+		(layer "F.SilkS")
+		(effects
+			(font
+				(size 1.2192 1.2192)
+				(thickness 0.1524)
+			)
+			(justify right)
+		)
+	)
+	(gr_text "GND"
+		(at 66.04 48.895 -90)
+		(layer "F.SilkS")
+		(effects
+			(font
+				(size 1.2192 1.2192)
+				(thickness 0.1524)
+			)
+			(justify right)
+		)
+	)
+	(gr_text "+5V"
+		(at 191.77 233.045 -90)
+		(layer "F.SilkS")
+		(effects
+			(font
+				(size 1.2192 1.2192)
+				(thickness 0.1524)
+			)
+			(justify left)
+		)
+	)
+	(gr_text "+5V"
+		(at 48.895 76.2 0)
+		(layer "F.SilkS")
+		(effects
+			(font
+				(size 1.2192 1.2192)
+				(thickness 0.1524)
+			)
+			(justify right)
+		)
+	)
+	(gr_text "GND"
+		(at 48.895 200.66 0)
+		(layer "F.SilkS")
+		(effects
+			(font
+				(size 1.2192 1.2192)
+				(thickness 0.1524)
+			)
+			(justify right)
+		)
+	)
+	(gr_text "GND"
+		(at 67.31 226.695 -90)
+		(layer "F.SilkS")
+		(effects
+			(font
+				(size 1.2192 1.2192)
+				(thickness 0.1524)
+			)
+			(justify right)
+		)
+	)
 	(segment

Commit message: Refinements
Parts:
- added C1001: 10u, Capacitor_THT:CP_Radial_D4.0mm_P1.50mm, F.Cu at (120.7, 137.2)
- added C1002: 10u, Capacitor_THT:CP_Radial_D4.0mm_P1.50mm, F.Cu at (134.6, 137.2)
Other:
- board text added: "RGE2025"

Commit message: Add s/n marker
Other:
- board text added: "JLCJLCJLCJLC"
Changed lines of the file:
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@@
+		)
+	)
+	(gr_text "JLCJLCJLCJLC"
+		(at 218.44 212.725 90)
+		(layer "B.SilkS")
+		(effects
+			(font
+				(size 1.2192 1.2192)
+				(thickness 0.1016)
+			)
+			(justify left bottom mirror)
 		)
 	)
